File: pcb/sensors_o2_temp.sch (KiCad schematic (older format))
At the start: 19 parts

Commit message: fixed library
Parts:
- U?: symbol RespiraWorks:INA333AIDGKR -> Ventilator-rescue:INA333AIDGKR-RespiraWorks
Changed lines of the file:
@@
 $EndSheet
 $Comp
-L RespiraWorks:+3.3V_Sns #PWR?
+L Ventilator-rescue:+3.3V_Sns-RespiraWorks #PWR?
 U 1 1 60107496
 P 3000 1100
@@
 Connection ~ 3450 1250
 $Comp
-L RespiraWorks:+3.3V_Sns #PWR?
+L Ventilator-rescue:+3.3V_Sns-RespiraWorks #PWR?
 U 1 1 6011C562
 P 3000 1800
@@
 Connection ~ 3450 1950
 $Comp
-L RespiraWorks:+3.3V_Sns #PWR?
+L Ventilator-rescue:+3.3V_Sns-RespiraWorks #PWR?
 U 1 1 6011C9C4
 P 3000 2500
@@
 Connection ~ 3450 2650
 $Comp
-L RespiraWorks:+3.3V_Sns #PWR?
+L Ventilator-rescue:+3.3V_Sns-RespiraWorks #PWR?
 U 1 1 6011CE53
 P 3000 3200
@@
 Connection ~ 3450 3350
 $Comp
-L RespiraWorks:+3.3V_Sns #PWR?
+L Ventilator-rescue:+3.3V_Sns-RespiraWorks #PWR?
 U 1 1 6011D298
 P 3000 3900
@@
 Oxy_Level
 $Comp
-L RespiraWorks:INA333AIDGKR U?
+L Ventilator-rescue:INA333AIDGKR-RespiraWorks U?
 U 1 1 60132AA0
 P 5400 5950
@@
 NoConn ~ 1700 5850
 $Comp
-L RespiraWorks:+3.3V_Sns #PWR?
+L Ventilator-rescue:+3.3V_Sns-RespiraWorks #PWR?
 U 1 1 60148A3F
 P 5400 5100
@@
 Connection ~ 5400 5100
 $Comp
-L RespiraWorks:+3.3V_Sns #PWR?
+L Ventilator-rescue:+3.3V_Sns-RespiraWorks #PWR?
 U 1 1 60148D99
 P 2700 5450

Commit message: Un-fucked library references
Fixed bad paths in sym/fp-lib-table
Deleted "rescue" library
Removed references to rescue library
Parts:
- U?: symbol Ventilator-rescue:INA333AIDGKR-RespiraWorks -> RespiraWorks:INA333AIDGKR
Changed lines of the file:
@@
 $EndSheet
 $Comp
-L Ventilator-rescue:+3.3V_Sns-RespiraWorks #PWR?
+L RespiraWorks:+3.3V_Sns #PWR?
 U 1 1 60107496
 P 3000 1100
@@
 Connection ~ 3450 1250
 $Comp
-L Ventilator-rescue:+3.3V_Sns-RespiraWorks #PWR?
+L RespiraWorks:+3.3V_Sns #PWR?
 U 1 1 6011C562
 P 3000 1800
@@
 Connection ~ 3450 1950
 $Comp
-L Ventilator-rescue:+3.3V_Sns-RespiraWorks #PWR?
+L RespiraWorks:+3.3V_Sns #PWR?
 U 1 1 6011C9C4
 P 3000 2500
@@
 Connection ~ 3450 2650
 $Comp
-L Ventilator-rescue:+3.3V_Sns-RespiraWorks #PWR?
+L RespiraWorks:+3.3V_Sns #PWR?
 U 1 1 6011CE53
 P 3000 3200
@@
 Connection ~ 3450 3350
 $Comp
-L Ventilator-rescue:+3.3V_Sns-RespiraWorks #PWR?
+L RespiraWorks:+3.3V_Sns #PWR?
 U 1 1 6011D298
 P 3000 3900
@@
 Oxy_Level
 $Comp
-L Ventilator-rescue:INA333AIDGKR-RespiraWorks U?
+L RespiraWorks:INA333AIDGKR U?
 U 1 1 60132AA0
 P 5400 5950
@@
 NoConn ~ 1700 5850
 $Comp
-L Ventilator-rescue:+3.3V_Sns-RespiraWorks #PWR?
+L RespiraWorks:+3.3V_Sns #PWR?
 U 1 1 60148A3F
 P 5400 5100
@@
 Connection ~ 5400 5100
 $Comp
-L Ventilator-rescue:+3.3V_Sns-RespiraWorks #PWR?
+L RespiraWorks:+3.3V_Sns #PWR?
 U 1 1 60148D99
 P 2700 5450

Commit message: prior stash
Parts:
- removed C?: 100nF 100V X7R, RespiraWorks_Std:C_0603_1608Metric, symbol Device:C
- removed C?: 1uF 10V X7R, RespiraWorks_Std:C_0603_1608Metric, symbol Device:C
- removed J?: Molex Micro-Fit, RespiraWorks_Std:Molex_Micro-Fit_3.0_43650-0315_1x03_P3.00mm_Vertical, symbol Connector_Generic:Conn_01x03
- removed R?: 2.05K 1%, RespiraWorks_Std:R_0603_1608Metric, symbol Device:R
- removed R? (x7): 10K 1%, RespiraWorks_Std:R_0603_1608Metric, symbol Device:R
- removed R?: 1.5K 1%, RespiraWorks_Std:R_0603_1608Metric, symbol Device:R
- removed R?: DNP, RespiraWorks_Std:R_0603_1608Metric, symbol Device:R
- removed TP?: Stepper1_Temp, RespiraWorks_Std:TestPoint_Pad_2.0x2.0mm, symbol Connector:TestPoint
- removed TP?: Stepper2_Temp, RespiraWorks_Std:TestPoint_Pad_2.0x2.0mm, symbol Connector:TestPoint
- removed TP?: Blower_Temp, RespiraWorks_Std:TestPoint_Pad_2.0x2.0mm, symbol Connector:TestPoint
- removed TP?: Batt_Temp, RespiraWorks_Std:TestPoint_Pad_2.0x2.0mm, symbol Connector:TestPoint
- removed TP?: Spare_Temp, RespiraWorks_Std:TestPoint_Pad_2.0x2.0mm, symbol Connector:TestPoint
- removed U?: INA333AIDGKR, RespiraWorks_Std:VSSOP-8_3.0x3.0mm_P0.65mm, symbol RespiraWorks:INA333AIDGKR
Connections:
- no-connect marks 1 -> 0
Other:
- note removed: "Gain = 49.8\nSensor output = approx. 0.0006V/%FiO2\n0 to 3.3V output = 0V (0% FiO2) to 3.0V (100% FiO2)\nMust be calibrated in software - this is just a general range - galvanic sensors drift!"
- note removed: "LPF fc = 106 Hz"
- note removed: "Optionally holds output low (10K or so)\nin case INA333 fails or its supply voltage\ndisappears"
- note removed: "Rg"
- note removed: "Rg = 100K/(Gain - 1)"
- note removed: "Series input protection:\n200 pA max. input bias for INA333\n= 2 µV max. offset << 25 µV of\nINA333's own input offset"
- note removed: "Teledyne R-24\nor equivalent"

Commit message: combined schs
Parts:
- added C?: 100nF 100V X7R, RespiraWorks_Std:C_0603_1608Metric, symbol Device:C
- added C?: 1uF 10V X7R, RespiraWorks_Std:C_0603_1608Metric, symbol Device:C
- added J?: Molex Micro-Fit, RespiraWorks_Std:Molex_Micro-Fit_3.0_43650-0315_1x03_P3.00mm_Vertical, symbol Connector_Generic:Conn_01x03
- added R?: 2.05K 1%, RespiraWorks_Std:R_0603_1608Metric, symbol Device:R
- added R? (x7): 10K 1%, RespiraWorks_Std:R_0603_1608Metric, symbol Device:R
- added R?: 1.5K 1%, RespiraWorks_Std:R_0603_1608Metric, symbol Device:R
- added R?: DNP, RespiraWorks_Std:R_0603_1608Metric, symbol Device:R
- added TP?: Stepper1_Temp, RespiraWorks_Std:TestPoint_Pad_2.0x2.0mm, symbol Connector:TestPoint
- added TP?: Stepper2_Temp, RespiraWorks_Std:TestPoint_Pad_2.0x2.0mm, symbol Connector:TestPoint
- added TP?: Blower_Temp, RespiraWorks_Std:TestPoint_Pad_2.0x2.0mm, symbol Connector:TestPoint
- added TP?: Batt_Temp, RespiraWorks_Std:TestPoint_Pad_2.0x2.0mm, symbol Connector:TestPoint
- added TP?: Spare_Temp, RespiraWorks_Std:TestPoint_Pad_2.0x2.0mm, symbol Connector:TestPoint
- added U?: INA333AIDGKR, RespiraWorks_Std:VSSOP-8_3.0x3.0mm_P0.65mm, symbol RespiraWorks:INA333AIDGKR
Connections:
- new net: R?.2, U?.1 (R1)
- new net: R?.2, U?.2 (-)
- new net: R?.2, U?.3 (+)
- new net: R?.1, R?.1, U?.6
- new net: R?.1, U?.8 (R1)
- new net: J?.3 (Pin_3), R?.1, R?.1, R?.1, R?.2
- new net: J?.1 (Pin_1), R?.1, R?.1, R?.2, R?.2
- new net +3.3V_Sns: C?.2, R?.2, R?.2, U?.7 (V+)
- new net Batt_Temp: TP?.1
- new net Blower_Temp: TP?.1
- new net GND: C?.1, C?.1, R?.1, R?.1, R?.2, U?.4 (V-), U?.5 (REF)
- new net Oxy_Level: C?.2, R?.2
- new net Spare_Temp: TP?.1
- new net Stepper1_Temp: TP?.1
- new net Stepper2_Temp: TP?.1
- no-connect marks 0 -> 1
Other:
- note added: "Gain = 49.8\nSensor output = approx. 0.0006V/%FiO2\n0 to 3.3V output = 0V (0% FiO2) to 3.0V (100% FiO2)\nMust be calibrated in software - this is just a general range - galvanic sensors drift!"
- note added: "LPF fc = 106 Hz"
- note added: "Optionally holds output low (10K or so)\nin case INA333 fails or its supply voltage\ndisappears"
- note added: "Rg"
- note added: "Rg = 100K/(Gain - 1)"
- note added: "Series input protection:\n200 pA max. input bias for INA333\n= 2 µV max. offset << 25 µV of\nINA333's own input offset"
- note added: "Teledyne R-24\nor equivalent"
