File: pcb/battery_charger.sch (KiCad schematic (older format))
At the start: 49 parts

Commit message: added the 12V buck for main VSYS
Other:
- note added: "Design notes:\n- 6.3A max current, 19V input\n- Inductor selection: Isat 9.1A, 3.3uH\n- Wurth 7443330330 or Bourns SRP1038A-3R3M (OPL alt: MWSA1004-3R3MT)\n- Voltage will range from 12V to 16.8V for 4s Li-Ion battery\n- 11.5 to 13.0V for SLA (lead acid)\n- N-CH FET: CSD17304Q3 (OPL) or BSZ050N03LSGATMA1 (OPL)\n- P-CH FET: CSD25402Q3A (OPL) or CSD25404Q3T (OPL)\n"
- note removed: "Design notes:\n- 6.3A max current, 19V input\n- Inductor selection: Isat 9.1A, 3.3uH\n- Wurth 7443330330 or Bourns SRP1038A-3R3M (OPL alt: MWSA1004-3R3MT)\n- Voltage will range from 10.8V to 12.6V for 3s Li-Ion battery\n- 11.5 to 13.0V for SLA (lead acid)\n- N-CH FET: CSD17304Q3 (OPL) or BSZ050N03LSGATMA1 (OPL)\n- P-CH FET: CSD25402Q3A (OPL) or CSD25404Q3T (OPL)\n"
Changed lines of the file:
@@
 SDA
 Text Notes 4600 1550 0    50   ~ 0
-Design notes:\n- 6.3A max current, 19V input\n- Inductor selection: Isat 9.1A, 3.3uH\n- Wurth 7443330330 or Bourns SRP1038A-3R3M (OPL alt: MWSA1004-3R3MT)\n- Voltage will range from 10.8V to 12.6V for 3s Li-Ion battery\n- 11.5 to 13.0V for SLA (lead acid)\n- N-CH FET: CSD17304Q3 (OPL) or BSZ050N03LSGATMA1 (OPL)\n- P-CH FET: CSD25402Q3A (OPL) or CSD25404Q3T (OPL)\n
+Design notes:\n- 6.3A max current, 19V input\n- Inductor selection: Isat 9.1A, 3.3uH\n- Wurth 7443330330 or Bourns SRP1038A-3R3M (OPL alt: MWSA1004-3R3MT)\n- Voltage will range from 12V to 16.8V for 4s Li-Ion battery\n- 11.5 to 13.0V for SLA (lead acid)\n- N-CH FET: CSD17304Q3 (OPL) or BSZ050N03LSGATMA1 (OPL)\n- P-CH FET: CSD25402Q3A (OPL) or CSD25404Q3T (OPL)\n
 $Comp
 L RespiraWorks_Std:SRP1038A-3R3M L?
@@
 	1    0    0    -1
 $EndComp
-Text HLabel 7850 5000 2    50   Input ~ 0
+Text HLabel 7850 5000 2    50   Output ~ 0
 PSYS
-Text HLabel 8350 4800 2    50   Input ~ 0
+Text HLabel 8350 4800 2    50   Output ~ 0
 IBAT
-Text HLabel 9500 4700 2    50   Input ~ 0
+Text HLabel 9500 4700 2    50   Output ~ 0
 IADPT
 Wire Wire Line
@@
 Wire Wire Line
 	7150 4500 9000 4500
-Text HLabel 9000 4500 2    50   Input ~ 0
+Text HLabel 9000 4500 2    50   Output ~ 0
 ACOK
 Wire Wire Line
@@
 Wire Wire Line
 	3950 4000 5300 4000
-Text HLabel 10500 2000 2    50   Input ~ 0
+Text HLabel 10500 2000 2    50   Output ~ 0
 VLINK
 Wire Wire Line
@@
 	7800 3200 8850 3200
 Connection ~ 7800 3200
-Text HLabel 8850 3200 2    50   Input ~ 0
+Text HLabel 8850 3200 2    50   BiDi ~ 0
 BAT_P
 Wire Wire Line

Commit message: charger and buck are in, commit before starting on balancer/fuel gauge
Parts:
- added C?: 100pF, Capacitor_SMD:C_0603_1608Metric, symbol Device:C
- added C?: 0.01uF, Capacitor_SMD:C_0603_1608Metric, symbol Device:C
- added R? (x2): 316k, Resistor_SMD:R_0603_1608Metric, symbol Device:R
- added R? (x2): 100k, Resistor_SMD:R_0603_1608Metric, symbol Device:R
- added R?: 0, Resistor_SMD:R_0603_1608Metric, symbol Device:R
- added R?: 3M, Resistor_SMD:R_0603_1608Metric, symbol Device:R
- C?: value 100pF -> 0.01uF
Connections:
- wire segments 133 -> 150
Other:
- note added: "Optional: R between CMPIN and\nCMPOUT sets hysteresis"
- note added: "Threshold here is 1.2V, max of 7V\nnBATPRES asserted when BAT_P over 9.6V\nReused ILIM resistor values to reduce BOM."
- note added: "V_ilim = 20*IPDM*Rac\nV_ilim = 1.29V -> 6.45A"
- note removed: "V_ilim = 3.57V > ILIM = 6400mA\nShort ILIM_HIZ to GND to shut off all power"
- moved on the sheet: C?
Changed lines of the file:
@@
 $EndComp
 Connection ~ 1800 4200
-Text Notes 3800 6600 0    50   ~ 0
-V_ilim = 3.57V > ILIM = 6400mA\nShort ILIM_HIZ to GND to shut off all power
+Text Notes 2500 5400 0    50   ~ 0
+V_ilim = 20*IPDM*Rac\nV_ilim = 1.29V -> 6.45A
 $Comp
 L Device:R R?
@@
 L Device:C C?
 U 1 1 60580F39
-P 8000 5250
+P 4100 5450
 AR Path="/601A64F8/60580F39" Ref="C?"  Part="1"
 AR Path="/601A64F8/60567144/60580F39" Ref="C?"  Part="1"
-F 0 "C?" H 8115 5296 50  0000 L CNN
-F 1 "100pF" H 8115 5205 50  0000 L CNN
-F 2 "Capacitor_SMD:C_0603_1608Metric" H 8038 5100 50  0001 C CNN
-F 3 "~" H 8000 5250 50  0001 C CNN
-	1    8000 5250
+F 0 "C?" H 4215 5496 50  0000 L CNN
+F 1 "0.01uF" H 4215 5405 50  0000 L CNN
+F 2 "Capacitor_SMD:C_0603_1608Metric" H 4138 5300 50  0001 C CNN
+F 3 "~" H 4100 5450 50  0001 C CNN
+	1    4100 5450
 	1    0    0    -1
 $EndComp
@@
 Wire Wire Line
 	7800 2000 8300 2000
-Text Label 4150 5100 0    50   ~ 0
+Text Label 3900 5000 0    50   ~ 0
 REGN
 Wire Wire Line
@@
 Text HLabel 1250 2000 0    50   Input ~ 0
 VIN_ADP
+$Comp
+L Device:R R?
+U 1 1 60332888
+P 3850 5150
+AR Path="/601A64F8/60332888" Ref="R?"  Part="1"
+AR Path="/601A64F8/60567144/60332888" Ref="R?"  Part="1"
+F 0 "R?" H 3600 5200 50  0000 L CNN
+F 1 "316k" H 3600 5100 50  0000 L CNN
+F 2 "Resistor_SMD:R_0603_1608Metric" V 3780 5150 50  0001 C CNN
+F 3 "~" H 3850 5150 50  0001 C CNN
+	1    3850 5150
+	1    0    0    -1
+$EndComp
+$Comp
+L Device:R R?
+U 1 1 6033CD9E
+P 3850 5450
+AR Path="/601A64F8/6033CD9E" Ref="R?"  Part="1"
+AR Path="/601A64F8/60567144/6033CD9E" Ref="R?"  Part="1"
+F 0 "R?" H 3600 5500 50  0000 L CNN
+F 1 "100k" H 3600 5400 50  0000 L CNN
+F 2 "Resistor_SMD:R_0603_1608Metric" V 3780 5450 50  0001 C CNN
+F 3 "~" H 3850 5450 50  0001 C CNN
+	1    3850 5450
+	1    0    0    -1
+$EndComp
+$Comp
+L power:GND #PWR?
+U 1 1 60341EC1
+P 3850 5600
+AR Path="/601A64F8/60341EC1" Ref="#PWR?"  Part="1"
+AR Path="/601A64F8/60567144/60341EC1" Ref="#PWR?"  Part="1"
+F 0 "#PWR?" H 3850 5350 50  0001 C CNN
+F 1 "GND" H 3855 5427 50  0000 C CNN
+F 2 "" H 3850 5600 50  0001 C CNN
+F 3 "" H 3850 5600 50  0001 C CNN
+	1    3850 5600
+	1    0    0    -1
+$EndComp
+Wire Wire Line
+	5300 5300 4100 5300
+Connection ~ 3850 5300
+Wire Wire Line
+	3850 5000 4150 5000
+Wire Wire Line
+	4150 5000 4150 5100
+Connection ~ 4100 5300
+Wire Wire Line
+	4100 5300 3850 5300
+Wire Wire Line
+	4100 5600 3850 5600
+Connection ~ 3850 5600
+$Comp
+L Device:C C?
+U 1 1 6035868D
+P 8000 5250
+AR Path="/601A64F8/6035868D" Ref="C?"  Part="1"
+AR Path="/601A64F8/60567144/6035868D" Ref="C?"  Part="1"
+F 0 "C?" H 8115 5296 50  0000 L CNN
+F 1 "100pF" H 8115 5205 50  0000 L CNN
+F 2 "Capacitor_SMD:C_0603_1608Metric" H 8038 5100 50  0001 C CNN
+F 3 "~" H 8000 5250 50  0001 C CNN
+	1    8000 5250
+	1    0    0    -1
+$EndComp
+$Comp
+L Device:R R?
+U 1 1 6035E290
+P 5000 5900
+AR Path="/601A64F8/6035E290" Ref="R?"  Part="1"
+AR Path="/601A64F8/60567144/6035E290" Ref="R?"  Part="1"
+F 0 "R?" V 5050 6100 50  0000 L CNN
+F 1 "0" V 5050 5650 50  0000 L CNN
+F 2 "Resistor_SMD:R_0603_1608Metric" V 4930 5900 50  0001 C CNN
+F 3 "~" H 5000 5900 50  0001 C CNN
+	1    5000 5900
+	0    -1   -1   0
+$EndComp
+Wire Wire Line
+	5300 5900 5150 5900
+Wire Wire Line
+	4850 5900 4650 5900
+Wire Wire Line
+	4650 5900 4650 5700
+Wire Wire Line
+	4650 5700 5150 5700
+Wire Wire Line
+	5300 5500 4850 5500
+Wire Wire Line
+	4550 5500 4550 6350
+$Comp
+L Device:R R?
+U 1 1 60376C83
+P 4250 6200
+AR Path="/601A64F8/60376C83" Ref="R?"  Part="1"
+AR Path="/601A64F8/60567144/60376C83" Ref="R?"  Part="1"
+F 0 "R?" H 4000 6250 50  0000 L CNN
+F 1 "316k" H 4000 6150 50  0000 L CNN
+F 2 "Resistor_SMD:R_0603_1608Metric" V 4180 6200 50  0001 C CNN
+F 3 "~" H 4250 6200 50  0001 C CNN
+	1    4250 6200
+	1    0    0    -1
+$EndComp
+$Comp
+L Device:R R?
+U 1 1 60376C89
+P 4250 6500
+AR Path="/601A64F8/60376C89" Ref="R?"  Part="1"
+AR Path="/601A64F8/60567144/60376C89" Ref="R?"  Part="1"
+F 0 "R?" H 4000 6550 50  0000 L CNN
+F 1 "100k" H 4000 6450 50  0000 L CNN
+F 2 "Resistor_SMD:R_0603_1608Metric" V 4180 6500 50  0001 C CNN
+F 3 "~" H 4250 6500 50  0001 C CNN
+	1    4250 6500
+	1    0    0    -1
+$EndComp
+Wire Wire Line
+	4550 6350 4250 6350
+Connection ~ 4250 6350
+$Comp
+L power:GND #PWR?
+U 1 1 60384778
+P 4250 6650
+AR Path="/601A64F8/60384778" Ref="#PWR?"  Part="1"
+AR Path="/601A64F8/60567144/60384778" Ref="#PWR?"  Part="1"
+F 0 "#PWR?" H 4250 6400 50  0001 C CNN
+F 1 "GND" H 4255 6477 50  0000 C CNN
+F 2 "" H 4250 6650 50  0001 C CNN
+F 3 "" H 4250 6650 50  0001 C CNN
+	1    4250 6650
+	-1   0    0    -1
+$EndComp
+Text Label 8350 3200 0    50   ~ 0
+BAT_P
+Text Label 4000 6050 0    50   ~ 0
+BAT_P
+Wire Wire Line
+	4250 6050 4000 6050
+Text Notes 2200 6450 0    50   ~ 0
+Threshold here is 1.2V, max of 7V\nnBATPRES asserted when BAT_P over 9.6V\nReused ILIM resistor values to reduce BOM.
+$Comp
+L Device:R R?
+U 1 1 603A873E
+P 5000 5600
+AR Path="/601A64F8/603A873E" Ref="R?"  Part="1"
+AR Path="/601A64F8/60567144/603A873E" Ref="R?"  Part="1"
+F 0 "R?" V 5050 5800 50  0000 L CNN
+F 1 "3M" V 5050 5350 50  0000 L CNN
+F 2 "Resistor_SMD:R_0603_1608Metric" V 4930 5600 50  0001 C CNN
+F 3 "~" H 5000 5600 50  0001 C CNN
+F 4 "DNP" V 5000 5600 50  0000 C CNN "DNP"
+	1    5000 5600
+	0    -1   -1   0
+$EndComp
+Wire Wire Line
+	4850 5600 4850 5500
+Connection ~ 4850 5500
+Wire Wire Line
+	4850 5500 4550 5500
+Wire Wire Line
+	5150 5600 5150 5700
+Connection ~ 5150 5700
+Wire Wire Line
+	5150 5700 5300 5700
+Text Notes 4750 6250 0    50   ~ 0
+Optional: R between CMPIN and\nCMPOUT sets hysteresis
+$Comp
+L Device:C C?
+U 1 1 603BD7CB
+P 4550 6500
+AR Path="/601A64F8/603BD7CB" Ref="C?"  Part="1"
+AR Path="/601A64F8/60567144/603BD7CB" Ref="C?"  Part="1"
+F 0 "C?" H 4665 6546 50  0000 L CNN
+F 1 "0.01uF" H 4665 6455 50  0000 L CNN
+F 2 "Capacitor_SMD:C_0603_1608Metric" H 4588 6350 50  0001 C CNN
+F 3 "~" H 4550 6500 50  0001 C CNN
+	1    4550 6500
+	1    0    0    -1
+$EndComp
+$Comp
+L power:GND #PWR?
+U 1 1 603C4110
+P 4550 6650
+AR Path="/601A64F8/603C4110" Ref="#PWR?"  Part="1"
+AR Path="/601A64F8/60567144/603C4110" Ref="#PWR?"  Part="1"
+F 0 "#PWR?" H 4550 6400 50  0001 C CNN
+F 1 "GND" H 4555 6477 50  0000 C CNN
+F 2 "" H 4550 6650 50  0001 C CNN
+F 3 "" H 4550 6650 50  0001 C CNN
+	1    4550 6650
+	-1   0    0    -1
+$EndComp
+Connection ~ 4550 6350
 $EndSCHEMATC

Commit message: added battery balancer/fuel gauge
Connections:
- net labels added: PACK_P
- net labels removed: BAT_P
Changed lines of the file:
@@
 	3050 4900 2600 4900
 Text Label 2600 4550 0    50   ~ 0
-BAT_P
+PACK_P
 Text Label 2600 4900 0    50   ~ 0
 VIN_ADP
@@
 Connection ~ 7800 3200
 Text HLabel 8850 3200 2    50   BiDi ~ 0
-BAT_P
+PACK_P
 Wire Wire Line
 	1800 2000 1250 2000
@@
 $EndComp
 Text Label 8350 3200 0    50   ~ 0
-BAT_P
+PACK_P
 Text Label 4000 6050 0    50   ~ 0
-BAT_P
+PACK_P
 Wire Wire Line
 	4250 6050 4000 6050

Commit message: clean up, add part numbers to parts, added design comments
Parts:
- removed D? (x2): D_Schottky, symbol Device:D_Schottky
- removed R?: 169k, Resistor_SMD:R_0603_1608Metric, symbol Device:R
- added D?: BAT54C, Package_TO_SOT_SMD:SOT-23, symbol Diode:BAT54C
- added R?: 10k, Resistor_SMD:R_0603_1608Metric, symbol Device:R
- R? (x2): footprint Capacitor_SMD:C_1206_3216Metric -> RespiraWorks_Std:R_1206_3216Metric
- R?: value 169k -> 30.1k
Connections:
- wire segments 150 -> 146
Other:
- note added: "Design notes:\n- 6.3A max current, 20V input\n- Inductor selection: Isat 9.1A, 3.3uH\n- Wurth 7443330330 or Bourns SRP1038A-3R3M (OPL alt: MWSA1004-3R3MT)\n- Voltage will range from 12V to 16.8V for 4s Li-Ion battery\n- 11.5 to 13.0V for SLA (lead acid)\n- N-CH FET: CSD17304Q3 (OPL) or BSZ050N03LSGATMA1 (OPL)\n- P-CH FET: CSD25402Q3A (OPL) or CSD25404Q3T (OPL)\n"
- note added: "Optional: R between CMPIN and\nCMPOUT sets hysteresis\n(not req'd when comparator \npolarity set to LOW)"
- note added: "PMON default is 1uA/W\nIBAT and IADT are voltage outputs\n"
- note added: "Threshold here is 2.3V, max of 7V\nnBATPRES asserted when BAT_P over 9.6V\nReused ILIM resistor values to reduce BOM."
- note removed: "Design notes:\n- 6.3A max current, 19V input\n- Inductor selection: Isat 9.1A, 3.3uH\n- Wurth 7443330330 or Bourns SRP1038A-3R3M (OPL alt: MWSA1004-3R3MT)\n- Voltage will range from 12V to 16.8V for 4s Li-Ion battery\n- 11.5 to 13.0V for SLA (lead acid)\n- N-CH FET: CSD17304Q3 (OPL) or BSZ050N03LSGATMA1 (OPL)\n- P-CH FET: CSD25402Q3A (OPL) or CSD25404Q3T (OPL)\n"
- note removed: "Optional: R between CMPIN and\nCMPOUT sets hysteresis"
- note removed: "Threshold here is 1.2V, max of 7V\nnBATPRES asserted when BAT_P over 9.6V\nReused ILIM resistor values to reduce BOM."
- moved on the sheet: C?, R?

Commit message: WIP implement comments from review
Parts:
- added C?: 1uF, Capacitor_SMD:C_0603_1608Metric, symbol Device:C
- added R?: 10, RespiraWorks_Std:R_0603_1608Metric, symbol Device:R
- C? (x3): value 0.033uF -> 0.1uF
- C? (x2): footprint Capacitor_SMD:C_0805_2012Metric -> (none)
- R?: value 68k -> 442k
Connections:
- wire segments 146 -> 148
Other:
- note added: "Design notes:\n- 6.3A max current, 17-20V input, approx 120W\n- Inductor selection: Isat 9.1A, 3.3uH\n- Wurth 7443330330 or Bourns SRP1038A-3R3M (OPL alt: MWSA1004-3R3MT)\n- Voltage will range from 12V to 16.8V for 4s Li-Ion battery\n- 11.5 to 13.0V for SLA (lead acid)\n- N-CH FET: CSD17304Q3 (OPL) or BSZ050N03LSGATMA1 (OPL)\n- P-CH FET: CSD25402Q3A (OPL) or CSD25404Q3T (OPL)\n"
- note added: "V_ilim = 20*IPDM*Rac\nV_ilim = 1.29V -> 6.45A\nNote this is adapter current"
- note removed: "Design notes:\n- 6.3A max current, 20V input\n- Inductor selection: Isat 9.1A, 3.3uH\n- Wurth 7443330330 or Bourns SRP1038A-3R3M (OPL alt: MWSA1004-3R3MT)\n- Voltage will range from 12V to 16.8V for 4s Li-Ion battery\n- 11.5 to 13.0V for SLA (lead acid)\n- N-CH FET: CSD17304Q3 (OPL) or BSZ050N03LSGATMA1 (OPL)\n- P-CH FET: CSD25402Q3A (OPL) or CSD25404Q3T (OPL)\n"
- note removed: "V_ilim = 20*IPDM*Rac\nV_ilim = 1.29V -> 6.45A"

Commit message: WIP implement PR comments
Parts:
- C?: DNP (none) -> DNP
Changed lines of the file:
@@
 F 2 "Capacitor_SMD:C_0603_1608Metric" H 1988 2300 50  0001 C CNN
 F 3 "~" H 1950 2450 50  0001 C CNN
+F 4 "DNP" V 1600 2450 50  0000 C CNN "DNP"
 	1    1950 2450
 	0    -1   -1   0

Commit message: updated footprints to reference to RW library
Parts:
- removed C? (x2): 33uF, symbol Device:CP
- added C? (x2): 33uF, RespiraWorks_Std:CP_Elec_6.3x7.7, symbol Device:CP
- C? (x18): footprint Capacitor_SMD:C_0603_1608Metric -> RespiraWorks_Std:C_0603_1608Metric
- C? (x10): footprint Capacitor_SMD:C_0805_2012Metric -> RespiraWorks_Std:C_0805_2012Metric
- D?: footprint Package_TO_SOT_SMD:SOT-23 -> RespiraWorks_Std:SOT-23
- Q? (x5): footprint Package_SON:VSON-8_3.3x3.3mm_P0.65mm_NexFET -> RespiraWorks_Std:VSON-8_3.3x3.3mm_P0.65mm_NexFET
- R? (x17): footprint Resistor_SMD:R_0603_1608Metric -> RespiraWorks_Std:R_0603_1608Metric
- U?: footprint Package_DFN_QFN:QFN-28-1EP_4x4mm_P0.4mm_EP2.6x2.6mm_ThermalVias -> RespiraWorks_Std:QFN-28-1EP_4x4mm_P0.4mm_EP2.6x2.6mm_ThermalVias

Commit message: inductor footprint assignments
Parts:
- L?: footprint (none) -> RespiraWorks:L_Bourns-SRP1038; Manufacturer (none) -> Bourns; Manufacturer PN (none) -> SRP1038A-3R3M
Changed lines of the file:
@@
 F 0 "L?" H 6050 2190 50  0000 C CNN
 F 1 "SRP1038A-3R3M" H 6050 2099 50  0000 C CNN
-F 2 "" V 6050 2000 50  0001 C CNN
+F 2 "RespiraWorks:L_Bourns-SRP1038" V 6050 2000 50  0001 C CNN
 F 3 "https://www.bourns.com/docs/Product-Datasheets/SRP1038A.pdf" V 6050 2000 50  0001 C CNN
+F 4 "Bourns" H 6050 2000 50  0001 C CNN "Manufacturer"
+F 5 "SRP1038A-3R3M" H 6050 2000 50  0001 C CNN "Manufacturer PN"
 	1    6050 2000
 	1    0    0    -1
