File: pcb/battery_charger.sch (KiCad schematic (older format))
At the start: 58 parts

Commit message: BOM
More BOM consolidation with bulk capacitors + changed tantalum stepper caps to aluminum, added bulk cap to PSol driver
Made stepper's 3.3V power naming consistent with others (3.3V->3V3)
Slightly increased current limit on PSOL/heater driver
Changed 3906 transistors to 2907 to better support +5V_Batt current
Parts:
- removed D?: BAT54C, RespiraWorks_Std:SOT-23, symbol Diode:BAT54C
- added D? (x2): BAT54J, RespiraWorks_Std:D_SOD-323F, symbol Diode:BAT54J
- C? (x2): Dielectric (none) -> Aluminum
- C?: value 150pF -> 100pF
- C? (x2): footprint RespiraWorks_Std:C_0805_2012Metric -> RespiraWorks_Std:C_1210_3225Metric; Dielectric X5R -> X7S; Manufacturer (none) -> Murata; Manufacturer PN (none) -> GRM32EC72A106KE05L; Voltage 35V -> 100V
- C? (x8): footprint RespiraWorks_Std:C_0805_2012Metric -> RespiraWorks_Std:C_1210_3225Metric; Dielectric (none) -> X7S; Manufacturer (none) -> Murata; Manufacturer PN (none) -> GRM32EC72A106KE05L; Voltage 25V -> 100V
- R? (x4): footprint RespiraWorks_std:R_0603_1608Metric -> RespiraWorks_Std:R_0603_1608Metric
Connections:
- wire segments 146 -> 147
Changed lines of the file:
@@
 F 0 "R?" V 3750 3300 50  0000 L CNN
 F 1 "0" V 3750 3800 50  0000 L CNN
-F 2 "RespiraWorks_std:R_0603_1608Metric" V 3730 3600 50  0001 C CNN
+F 2 "RespiraWorks_Std:R_0603_1608Metric" V 3730 3600 50  0001 C CNN
 F 3 "~" H 3800 3600 50  0001 C CNN
 	1    3800 3600
@@
 AR Path="/6041384A/60567144/60580ED6" Ref="C?"  Part="1"
 F 0 "C?" V 4500 2550 50  0000 C CNN
-F 1 "150pF" V 4800 2600 50  0000 C CNN
+F 1 "100pF" V 4800 2600 50  0000 C CNN
 F 2 "RespiraWorks_Std:C_0603_1608Metric" H 4688 2450 50  0001 C CNN
 F 3 "~" H 4650 2600 50  0001 C CNN
@@
 F 0 "R?" V 3850 3600 50  0000 L CNN
 F 1 "0" V 3850 3150 50  0000 L CNN
-F 2 "RespiraWorks_std:R_0603_1608Metric" V 3730 3400 50  0001 C CNN
+F 2 "RespiraWorks_Std:R_0603_1608Metric" V 3730 3400 50  0001 C CNN
 F 3 "~" H 3800 3400 50  0001 C CNN
 	1    3800 3400
@@
 F 0 "C?" H 4000 2050 50  0000 L CNN
 F 1 "10uF" H 4000 1950 50  0000 L CNN
-F 2 "RespiraWorks_Std:C_0805_2012Metric" H 3988 2000 50  0001 C CNN
+F 2 "RespiraWorks_Std:C_1210_3225Metric" H 3988 2000 50  0001 C CNN
 F 3 "~" H 3950 2150 50  0001 C CNN
-F 4 "35V" H 4000 1850 50  0000 L CNN "Voltage"
-F 5 "X5R" H 3950 2150 50  0001 C CNN "Dielectric"
+F 4 "100V" H 4000 1850 50  0000 L CNN "Voltage"
+F 5 "X7S" H 3950 2150 50  0001 C CNN "Dielectric"
+F 6 "Murata" H 3950 2150 50  0001 C CNN "Manufacturer"
+F 7 "GRM32EC72A106KE05L" H 3950 2150 50  0001 C CNN "Manufacturer PN"
 	1    3950 2150
 	1    0    0    -1
@@
 F 0 "C?" H 9850 1200 50  0000 L CNN
 F 1 "10uF" H 9850 1100 50  0000 L CNN
-F 2 "RespiraWorks_Std:C_0805_2012Metric" H 9838 1150 50  0001 C CNN
+F 2 "RespiraWorks_Std:C_1210_3225Metric" H 9838 1150 50  0001 C CNN
 F 3 "~" H 9800 1300 50  0001 C CNN
-F 4 "25V" H 9850 1000 50  0000 L CNN "Voltage"
+F 4 "100V" H 9850 1000 50  0000 L CNN "Voltage"
+F 5 "X7S" H 9800 1300 50  0001 C CNN "Dielectric"
+F 6 "Murata" H 9800 1300 50  0001 C CNN "Manufacturer"
+F 7 "GRM32EC72A106KE05L" H 9800 1300 50  0001 C CNN "Manufacturer PN"
 	1    9800 1300
 	1    0    0    -1
@@
 F 0 "C?" H 9550 1200 50  0000 L CNN
 F 1 "10uF" H 9550 1100 50  0000 L CNN
-F 2 "RespiraWorks_Std:C_0805_2012Metric" H 9538 1150 50  0001 C CNN
+F 2 "RespiraWorks_Std:C_1210_3225Metric" H 9538 1150 50  0001 C CNN
 F 3 "~" H 9500 1300 50  0001 C CNN
-F 4 "25V" H 9550 1000 50  0000 L CNN "Voltage"
+F 4 "100V" H 9550 1000 50  0000 L CNN "Voltage"
+F 5 "X7S" H 9500 1300 50  0001 C CNN "Dielectric"
+F 6 "Murata" H 9500 1300 50  0001 C CNN "Manufacturer"
+F 7 "GRM32EC72A106KE05L" H 9500 1300 50  0001 C CNN "Manufacturer PN"
 	1    9500 1300
 	1    0    0    -1
@@
 F 0 "C?" H 9250 1200 50  0000 L CNN
 F 1 "10uF" H 9250 1100 50  0000 L CNN
-F 2 "RespiraWorks_Std:C_0805_2012Metric" H 9238 1150 50  0001 C CNN
+F 2 "RespiraWorks_Std:C_1210_3225Metric" H 9238 1150 50  0001 C CNN
 F 3 "~" H 9200 1300 50  0001 C CNN
-F 4 "25V" H 9250 1000 50  0000 L CNN "Voltage"
+F 4 "100V" H 9250 1000 50  0000 L CNN "Voltage"
+F 5 "X7S" H 9200 1300 50  0001 C CNN "Dielectric"
+F 6 "Murata" H 9200 1300 50  0001 C CNN "Manufacturer"
+F 7 "GRM32EC72A106KE05L" H 9200 1300 50  0001 C CNN "Manufacturer PN"
 	1    9200 1300
 	1    0    0    -1
@@
 F 0 "C?" H 8950 1200 50  0000 L CNN
 F 1 "10uF" H 8950 1100 50  0000 L CNN
-F 2 "RespiraWorks_Std:C_0805_2012Metric" H 8938 1150 50  0001 C CNN
+F 2 "RespiraWorks_Std:C_1210_3225Metric" H 8938 1150 50  0001 C CNN
 F 3 "~" H 8900 1300 50  0001 C CNN
-F 4 "25V" H 8950 1000 50  0000 L CNN "Voltage"
+F 4 "100V" H 8950 1000 50  0000 L CNN "Voltage"
+F 5 "X7S" H 8900 1300 50  0001 C CNN "Dielectric"
+F 6 "Murata" H 8900 1300 50  0001 C CNN "Manufacturer"
+F 7 "GRM32EC72A106KE05L" H 8900 1300 50  0001 C CNN "Manufacturer PN"
 	1    8900 1300
 	1    0    0    -1
@@
 F 0 "C?" H 8650 1200 50  0000 L CNN
 F 1 "10uF" H 8650 1100 50  0000 L CNN
-F 2 "RespiraWorks_Std:C_0805_2012Metric" H 8638 1150 50  0001 C CNN
+F 2 "RespiraWorks_Std:C_1210_3225Metric" H 8638 1150 50  0001 C CNN
 F 3 "~" H 8600 1300 50  0001 C CNN
-F 4 "25V" H 8650 1000 50  0000 L CNN "Voltage"
+F 4 "100V" H 8650 1000 50  0000 L CNN "Voltage"
+F 5 "X7S" H 8600 1300 50  0001 C CNN "Dielectric"
+F 6 "Murata" H 8600 1300 50  0001 C CNN "Manufacturer"
+F 7 "GRM32EC72A106KE05L" H 8600 1300 50  0001 C CNN "Manufacturer PN"
 	1    8600 1300
 	1    0    0    -1
@@
 F 0 "C?" H 9550 2050 50  0000 L CNN
 F 1 "10uF" H 9550 1950 50  0000 L CNN
-F 2 "RespiraWorks_Std:C_0805_2012Metric" H 9538 2000 50  0001 C CNN
+F 2 "RespiraWorks_Std:C_1210_3225Metric" H 9538 2000 50  0001 C CNN
 F 3 "~" H 9500 2150 50  0001 C CNN
-F 4 "25V" H 9550 1850 50  0000 L CNN "Voltage"
+F 4 "100V" H 9550 1850 50  0000 L CNN "Voltage"
+F 5 "X7S" H 9500 2150 50  0001 C CNN "Dielectric"
+F 6 "Murata" H 9500 2150 50  0001 C CNN "Manufacturer"
+F 7 "GRM32EC72A106KE05L" H 9500 2150 50  0001 C CNN "Manufacturer PN"
 	1    9500 2150
 	1    0    0    -1
@@
 F 0 "C?" H 9250 2050 50  0000 L CNN
 F 1 "10uF" H 9250 1950 50  0000 L CNN
-F 2 "RespiraWorks_Std:C_0805_2012Metric" H 9238 2000 50  0001 C CNN
+F 2 "RespiraWorks_Std:C_1210_3225Metric" H 9238 2000 50  0001 C CNN
 F 3 "~" H 9200 2150 50  0001 C CNN
-F 4 "25V" H 9250 1850 50  0000 L CNN "Voltage"
+F 4 "100V" H 9250 1850 50  0000 L CNN "Voltage"
+F 5 "X7S" H 9200 2150 50  0001 C CNN "Dielectric"
+F 6 "Murata" H 9200 2150 50  0001 C CNN "Manufacturer"
+F 7 "GRM32EC72A106KE05L" H 9200 2150 50  0001 C CNN "Manufacturer PN"
 	1    9200 2150
 	1    0    0    -1
@@
 F 0 "C?" H 8950 2050 50  0000 L CNN
 F 1 "10uF" H 8950 1950 50  0000 L CNN
-F 2 "RespiraWorks_Std:C_0805_2012Metric" H 8938 2000 50  0001 C CNN
+F 2 "RespiraWorks_Std:C_1210_3225Metric" H 8938 2000 50  0001 C CNN
 F 3 "~" H 8900 2150 50  0001 C CNN
-F 4 "25V" H 8950 1850 50  0000 L CNN "Voltage"
+F 4 "100V" H 8950 1850 50  0000 L CNN "Voltage"
+F 5 "X7S" H 8900 2150 50  0001 C CNN "Dielectric"
+F 6 "Murata" H 8900 2150 50  0001 C CNN "Manufacturer"
+F 7 "GRM32EC72A106KE05L" H 8900 2150 50  0001 C CNN "Manufacturer PN"
 	1    8900 2150
 	1    0    0    -1
@@
 F 0 "R?" V 7250 3200 50  0000 L CNN
 F 1 "0" V 7250 2750 50  0000 L CNN
-F 2 "RespiraWorks_std:R_0603_1608Metric" V 7130 3000 50  0001 C CNN
+F 2 "RespiraWorks_Std:R_0603_1608Metric" V 7130 3000 50  0001 C CNN
 F 3 "~" H 7200 3000 50  0001 C CNN
 	1    7200 3000
@@
 F 0 "R?" V 5050 6100 50  0000 L CNN
 F 1 "0" V 5050 5650 50  0000 L CNN
-F 2 "RespiraWorks_std:R_0603_1608Metric" V 4930 5900 50  0001 C CNN
+F 2 "RespiraWorks_Std:R_0603_1608Metric" V 4930 5900 50  0001 C CNN
 F 3 "~" H 5000 5900 50  0001 C CNN
 	1    5000 5900
@@
 Wire Wire Line
 	3900 5500 4850 5500
-$Comp
-L Diode:BAT54C D?
-U 1 1 6027BBEA
-P 2850 4650
-AR Path="/5FCD4B8E/603C510C/60567144/6027BBEA" Ref="D?"  Part="1"
-AR Path="/6041384A/60567144/6027BBEA" Ref="D?"  Part="1"
-F 0 "D?" V 2804 4738 50  0000 L CNN
-F 1 "BAT54C" V 2895 4738 50  0000 L CNN
-F 2 "RespiraWorks_Std:SOT-23" H 2925 4775 50  0001 L CNN
-F 3 "http://www.diodes.com/_files/datasheets/ds11005.pdf" H 2770 4650 50  0001 C CNN
-	1    2850 4650
-	0    -1   1    0
-$EndComp
 Wire Wire Line
 	3050 4500 3050 4650
@@
 F 5 "Panasonic" H 9800 2150 50  0001 C CNN "Manufacturer"
 F 6 "EEE-FK1H330XP" H 9800 2150 50  0001 C CNN "Manufacturer PN"
+F 7 "Aluminum" H 9800 2150 50  0001 C CNN "Dielectric"
 	1    9800 2150
 	1    0    0    -1
@@
 F 5 "Panasonic" H 10100 2150 50  0001 C CNN "Manufacturer"
 F 6 "EEE-FK1H330XP" H 10100 2150 50  0001 C CNN "Manufacturer PN"
+F 7 "Aluminum" H 10100 2150 50  0001 C CNN "Dielectric"
 	1    10100 2150
 	1    0    0    -1
@@
 F 0 "C?" H 3700 2050 50  0000 L CNN
 F 1 "10uF" H 3700 1950 50  0000 L CNN
-F 2 "RespiraWorks_Std:C_0805_2012Metric" H 3688 2000 50  0001 C CNN
+F 2 "RespiraWorks_Std:C_1210_3225Metric" H 3688 2000 50  0001 C CNN
 F 3 "~" H 3650 2150 50  0001 C CNN
-F 4 "35V" H 3700 1850 50  0000 L CNN "Voltage"
-F 5 "X5R" H 3650 2150 50  0001 C CNN "Dielectric"
+F 4 "100V" H 3700 1850 50  0000 L CNN "Voltage"
+F 5 "X7S" H 3650 2150 50  0001 C CNN "Dielectric"
+F 6 "Murata" H 3650 2150 50  0001 C CNN "Manufacturer"
+F 7 "GRM32EC72A106KE05L" H 3650 2150 50  0001 C CNN "Manufacturer PN"
 	1    3650 2150
 	1    0    0    -1
@@
 Text Notes 6950 5400 0    50   ~ 0
 5.4V nominal
+$Comp
+L Diode:BAT54J D?
+U 1 1 60756F63
+P 2850 4800
+AR Path="/6041384A/60567D6E/60756F63" Ref="D?"  Part="1"
+AR Path="/6041384A/60567144/60756F63" Ref="D?"  Part="1"
+F 0 "D?" H 2850 4900 50  0000 C CNN
+F 1 "BAT54J" V 2850 4600 50  0000 C CNN
+F 2 "RespiraWorks_Std:D_SOD-323F" H 2850 4625 50  0001 C CNN
+F 3 "https://assets.nexperia.com/documents/data-sheet/BAT54J.pdf" H 2850 4800 50  0001 C CNN
+	1    2850 4800
+	0    1    1    0
+$EndComp
+$Comp
+L Diode:BAT54J D?
+U 1 1 6075D700
+P 2850 4500
+AR Path="/6041384A/60567D6E/6075D700" Ref="D?"  Part="1"
+AR Path="/6041384A/60567144/6075D700" Ref="D?"  Part="1"
+F 0 "D?" H 2850 4600 50  0000 C CNN
+F 1 "BAT54J" V 2850 4300 50  0000 C CNN
+F 2 "RespiraWorks_Std:D_SOD-323F" H 2850 4325 50  0001 C CNN
+F 3 "https://assets.nexperia.com/documents/data-sheet/BAT54J.pdf" H 2850 4500 50  0001 C CNN
+	1    2850 4500
+	0    1    -1   0
+$EndComp
+Wire Wire Line
+	2850 4650 3050 4650
+Connection ~ 2850 4650
 $EndSCHEMATC

Commit message: BOM, fixes
Finished assigning parts, footprints except generic resistors
Added series resistors for logic signals received by UI computer to protect against UI computer power-down
Added tolerance notes on main schem
Replaced PSol fuse with PTC
Enlarged PSol driver bypass resistors to 0 ohm
Changed PSol unpopulated current-limiting resistor to divider
Parts:
- C? (x2): Dielectric (none) -> X7R; Manufacturer (none) -> Kemet; Manufacturer PN (none) -> C0805C105K5RACTU; Voltage (none) -> 50V
- C? (x3): Dielectric (none) -> NP0; Manufacturer (none) -> Kemet; Manufacturer PN (none) -> C0603C101J5GACTU; Voltage (none) -> 50V
- C? (x2): Dielectric (none) -> NP0; Manufacturer (none) -> Murata; Manufacturer PN (none) -> GRM1885C1H103JA01D; Voltage (none) -> 50V
- C? (x2): Dielectric (none) -> X7R; Manufacturer (none) -> Kemet; Manufacturer PN (none) -> C0603C473K5RACTU; Voltage (none) -> 50V
- C? (x6): Dielectric (none) -> X7R; Manufacturer (none) -> Kemet; Manufacturer PN (none) -> C0603C104K5RACTU; Voltage (none) -> 50V
- C?: Dielectric (none) -> NP0; Manufacturer (none) -> Kemet; Manufacturer PN (none) -> C0603C101J5GACTU
- C?: Dielectric (none) -> NP0; Manufacturer (none) -> Murata; Manufacturer PN (none) -> GRM1885C1H103JA01D; Voltage 25V -> 50V
- D? (x2): Manufacturer (none) -> Nexperia; Manufacturer PN (none) -> BAT54J,115
- Q? (x4): Manufacturer TI -> Texas Instruments
- R? (x2): Manufacturer (none) -> Vishay; Manufacturer PN (none) -> WSL1206R0100FEA
Changed lines of the file:
@@
 F 2 "RespiraWorks_Std:C_0603_1608Metric" H 5288 2000 50  0001 C CNN
 F 3 "~" H 5250 2150 50  0001 C CNN
+F 4 "X7R" H 5250 2150 50  0001 C CNN "Dielectric"
+F 5 "Kemet" H 5250 2150 50  0001 C CNN "Manufacturer"
+F 6 "C0603C473K5RACTU" H 5250 2150 50  0001 C CNN "Manufacturer PN"
+F 7 "50V" H 5250 2150 50  0001 C CNN "Voltage"
 	1    5250 2150
 	1    0    0    -1
@@
 F 2 "RespiraWorks_Std:C_0603_1608Metric" H 3438 2650 50  0001 C CNN
 F 3 "~" H 3400 2800 50  0001 C CNN
+F 4 "X7R" H 3400 2800 50  0001 C CNN "Dielectric"
+F 5 "Kemet" H 3400 2800 50  0001 C CNN "Manufacturer"
+F 6 "C0603C104K5RACTU" H 3400 2800 50  0001 C CNN "Manufacturer PN"
+F 7 "50V" H 3400 2800 50  0001 C CNN "Voltage"
 	1    3400 2800
 	1    0    0    -1
@@
 F 2 "RespiraWorks_Std:C_0603_1608Metric" H 3138 2650 50  0001 C CNN
 F 3 "~" H 3100 2800 50  0001 C CNN
+F 4 "X7R" H 3100 2800 50  0001 C CNN "Dielectric"
+F 5 "Kemet" H 3100 2800 50  0001 C CNN "Manufacturer"
+F 6 "C0603C104K5RACTU" H 3100 2800 50  0001 C CNN "Manufacturer PN"
+F 7 "50V" H 3100 2800 50  0001 C CNN "Voltage"
 	1    3100 2800
 	1    0    0    -1
@@
 F 2 "RespiraWorks_Std:C_0603_1608Metric" H 7188 5750 50  0001 C CNN
 F 3 "~" H 7150 5900 50  0001 C CNN
+F 4 "X7R" H 7150 5900 50  0001 C CNN "Dielectric"
+F 5 "Kemet" H 7150 5900 50  0001 C CNN "Manufacturer"
+F 6 "C0805C105K5RACTU" H 7150 5900 50  0001 C CNN "Manufacturer PN"
+F 7 "50V" H 7150 5900 50  0001 C CNN "Voltage"
 	1    7150 5900
 	1    0    0    -1
@@
 F 3 "~" H 4650 2600 50  0001 C CNN
 F 4 "50V" V 4900 2550 50  0000 C CNN "Voltage"
+F 5 "NP0" H 4650 2600 50  0001 C CNN "Dielectric"
+F 6 "Kemet" H 4650 2600 50  0001 C CNN "Manufacturer"
+F 7 "C0603C101J5GACTU" H 4650 2600 50  0001 C CNN "Manufacturer PN"
 	1    4650 2600
 	0    1    1    0
@@
 F 2 "RespiraWorks_Std:R_1206_3216Metric" V 3180 2000 50  0001 C CNN
 F 3 "~" H 3250 2000 50  0001 C CNN
+F 4 "Vishay" H 3250 2000 50  0001 C CNN "Manufacturer"
+F 5 "WSL1206R0100FEA" H 3250 2000 50  0001 C CNN "Manufacturer PN"
 	1    3250 2000
 	0    1    1    0
@@
 F 2 "RespiraWorks_Std:C_0603_1608Metric" H 8988 4700 50  0001 C CNN
 F 3 "~" H 8950 4850 50  0001 C CNN
+F 4 "NP0" H 8950 4850 50  0001 C CNN "Dielectric"
+F 5 "Kemet" H 8950 4850 50  0001 C CNN "Manufacturer"
+F 6 "C0603C101J5GACTU" H 8950 4850 50  0001 C CNN "Manufacturer PN"
+F 7 "50V" H 8950 4850 50  0001 C CNN "Voltage"
 	1    8950 4850
 	1    0    0    -1
@@
 F 2 "RespiraWorks_Std:C_0603_1608Metric" H 8538 5250 50  0001 C CNN
 F 3 "~" H 8500 5400 50  0001 C CNN
+F 4 "NP0" H 8500 5400 50  0001 C CNN "Dielectric"
+F 5 "Kemet" H 8500 5400 50  0001 C CNN "Manufacturer"
+F 6 "C0603C101J5GACTU" H 8500 5400 50  0001 C CNN "Manufacturer PN"
+F 7 "50V" H 8500 5400 50  0001 C CNN "Voltage"
 	1    8500 5400
 	1    0    0    -1
@@
 F 2 "RespiraWorks_Std:C_0603_1608Metric" H 3438 5300 50  0001 C CNN
 F 3 "~" H 3400 5450 50  0001 C CNN
+F 4 "NP0" H 3400 5450 50  0001 C CNN "Dielectric"
+F 5 "Murata" H 3400 5450 50  0001 C CNN "Manufacturer"
+F 6 "GRM1885C1H103JA01D" H 3400 5450 50  0001 C CNN "Manufacturer PN"
+F 7 "50V" H 3400 5450 50  0001 C CNN "Voltage"
 	1    3400 5450
 	1    0    0    -1
@@
 F 2 "RespiraWorks_Std:C_0603_1608Metric" H 3288 2350 50  0001 C CNN
 F 3 "~" H 3250 2500 50  0001 C CNN
+F 4 "X7R" H 3250 2500 50  0001 C CNN "Dielectric"
+F 5 "Kemet" H 3250 2500 50  0001 C CNN "Manufacturer"
+F 6 "C0603C104K5RACTU" H 3250 2500 50  0001 C CNN "Manufacturer PN"
+F 7 "50V" H 3250 2500 50  0001 C CNN "Voltage"
 	1    3250 2500
 	0    -1   -1   0
@@
 F 2 "RespiraWorks:VSONP-8-1EP_5x6_P1.27mm" H 2300 2025 50  0001 L CIN
 F 3 "https://www.ti.com/lit/ds/symlink/csd18563q5a.pdf" V 2100 2100 50  0001 L CNN
-F 4 "TI" V 2100 2100 50  0001 C CNN "Manufacturer"
+F 4 "Texas Instruments" V 2100 2100 50  0001 C CNN "Manufacturer"
 F 5 "CSD18563Q5A" V 2100 2100 50  0001 C CNN "Manufacturer PN"
 	1    2100 2100
@@
 F 2 "RespiraWorks_Std:C_0603_1608Metric" H 2388 2000 50  0001 C CNN
 F 3 "~" H 2350 2150 50  0001 C CNN
+F 4 "X7R" H 2350 2150 50  0001 C CNN "Dielectric"
+F 5 "Kemet" H 2350 2150 50  0001 C CNN "Manufacturer"
+F 6 "C0603C473K5RACTU" H 2350 2150 50  0001 C CNN "Manufacturer PN"
+F 7 "50V" H 2350 2150 50  0001 C CNN "Voltage"
 	1    2350 2150
 	1    0    0    -1
@@
 F 2 "RespiraWorks_Std:C_0603_1608Metric" H 8638 2000 50  0001 C CNN
 F 3 "~" H 8600 2150 50  0001 C CNN
-F 4 "25V" H 8650 1850 50  0000 L CNN "Voltage"
+F 4 "50V" H 8650 1850 50  0000 L CNN "Voltage"
+F 5 "NP0" H 8600 2150 50  0001 C CNN "Dielectric"
+F 6 "Murata" H 8600 2150 50  0001 C CNN "Manufacturer"
+F 7 "GRM1885C1H103JA01D" H 8600 2150 50  0001 C CNN "Manufacturer PN"
 	1    8600 2150
 	1    0    0    -1
@@
 F 2 "RespiraWorks_Std:R_1206_3216Metric" V 7730 2300 50  0001 C CNN
 F 3 "~" H 7800 2300 50  0001 C CNN
+F 4 "Vishay" H 7800 2300 50  0001 C CNN "Manufacturer"
+F 5 "WSL1206R0100FEA" H 7800 2300 50  0001 C CNN "Manufacturer PN"
 	1    7800 2300
 	-1   0    0    1
@@
 F 2 "RespiraWorks_Std:C_0603_1608Metric" H 7638 2150 50  0001 C CNN
 F 3 "~" H 7600 2300 50  0001 C CNN
+F 4 "X7R" H 7600 2300 50  0001 C CNN "Dielectric"
+F 5 "Kemet" H 7600 2300 50  0001 C CNN "Manufacturer"
+F 6 "C0603C104K5RACTU" H 7600 2300 50  0001 C CNN "Manufacturer PN"
+F 7 "50V" H 7600 2300 50  0001 C CNN "Voltage"
 	1    7600 2300
 	1    0    0    -1
@@
 F 2 "RespiraWorks_Std:C_0603_1608Metric" H 7238 2150 50  0001 C CNN
 F 3 "~" H 7200 2300 50  0001 C CNN
+F 4 "X7R" H 7200 2300 50  0001 C CNN "Dielectric"
+F 5 "Kemet" H 7200 2300 50  0001 C CNN "Manufacturer"
+F 6 "C0603C104K5RACTU" H 7200 2300 50  0001 C CNN "Manufacturer PN"
+F 7 "50V" H 7200 2300 50  0001 C CNN "Voltage"
 	1    7200 2300
 	1    0    0    -1
@@
 F 2 "RespiraWorks_Std:C_0603_1608Metric" H 7238 2500 50  0001 C CNN
 F 3 "~" H 7200 2650 50  0001 C CNN
+F 4 "X7R" H 7200 2650 50  0001 C CNN "Dielectric"
+F 5 "Kemet" H 7200 2650 50  0001 C CNN "Manufacturer"
+F 6 "C0603C104K5RACTU" H 7200 2650 50  0001 C CNN "Manufacturer PN"
+F 7 "50V" H 7200 2650 50  0001 C CNN "Voltage"
 	1    7200 2650
 	1    0    0    -1
@@
 F 2 "RespiraWorks_Std:C_0603_1608Metric" H 8038 5100 50  0001 C CNN
 F 3 "~" H 8000 5250 50  0001 C CNN
+F 4 "NP0" H 8000 5250 50  0001 C CNN "Dielectric"
+F 5 "Kemet" H 8000 5250 50  0001 C CNN "Manufacturer"
+F 6 "C0603C101J5GACTU" H 8000 5250 50  0001 C CNN "Manufacturer PN"
+F 7 "50V" H 8000 5250 50  0001 C CNN "Voltage"
 	1    8000 5250
 	1    0    0    -1
@@
 F 2 "RespiraWorks_Std:C_0603_1608Metric" H 3938 6350 50  0001 C CNN
 F 3 "~" H 3900 6500 50  0001 C CNN
+F 4 "NP0" H 3900 6500 50  0001 C CNN "Dielectric"
+F 5 "Murata" H 3900 6500 50  0001 C CNN "Manufacturer"
+F 6 "GRM1885C1H103JA01D" H 3900 6500 50  0001 C CNN "Manufacturer PN"
+F 7 "50V" H 3900 6500 50  0001 C CNN "Voltage"
 	1    3900 6500
 	1    0    0    -1
@@
 F 2 "RespiraWorks_Std:C_0603_1608Metric" H 3888 4500 50  0001 C CNN
 F 3 "~" H 3850 4650 50  0001 C CNN
+F 4 "X7R" H 3850 4650 50  0001 C CNN "Dielectric"
+F 5 "Kemet" H 3850 4650 50  0001 C CNN "Manufacturer"
+F 6 "C0805C105K5RACTU" H 3850 4650 50  0001 C CNN "Manufacturer PN"
+F 7 "50V" H 3850 4650 50  0001 C CNN "Voltage"
 	1    3850 4650
 	1    0    0    -1
@@
 F 2 "RespiraWorks:VSONP-8-1EP_5x6_P1.27mm" H 2900 2025 50  0001 L CIN
 F 3 "https://www.ti.com/lit/ds/symlink/csd18563q5a.pdf" V 2700 2100 50  0001 L CNN
-F 4 "TI" V 2700 2100 50  0001 C CNN "Manufacturer"
+F 4 "Texas Instruments" V 2700 2100 50  0001 C CNN "Manufacturer"
 F 5 "CSD18563Q5A" V 2700 2100 50  0001 C CNN "Manufacturer PN"
 	1    2700 2100
@@
 F 2 "RespiraWorks:VSONP-8-1EP_5x6_P1.27mm" H 4900 2125 50  0001 L CIN
 F 3 "https://www.ti.com/lit/ds/symlink/csd18563q5a.pdf" V 4700 2200 50  0001 L CNN
-F 4 "TI" V 4700 2200 50  0001 C CNN "Manufacturer"
+F 4 "Texas Instruments" V 4700 2200 50  0001 C CNN "Manufacturer"
 F 5 "CSD18563Q5A" V 4700 2200 50  0001 C CNN "Manufacturer PN"
 	1    4700 2200
@@
 F 2 "RespiraWorks:VSONP-8-1EP_5x6_P1.27mm" H 4550 2025 50  0001 L CIN
 F 3 "https://www.ti.com/lit/ds/symlink/csd18563q5a.pdf" V 4350 2100 50  0001 L CNN
-F 4 "TI" V 4350 2100 50  0001 C CNN "Manufacturer"
+F 4 "Texas Instruments" V 4350 2100 50  0001 C CNN "Manufacturer"
 F 5 "CSD18563Q5A" V 4350 2100 50  0001 C CNN "Manufacturer PN"
 	1    4350 2100
@@
 F 2 "RespiraWorks_Std:D_SOD-323F" H 2850 4625 50  0001 C CNN
 F 3 "https://assets.nexperia.com/documents/data-sheet/BAT54J.pdf" H 2850 4800 50  0001 C CNN
+F 4 "Nexperia" H 2850 4800 50  0001 C CNN "Manufacturer"
+F 5 "BAT54J,115" H 2850 4800 50  0001 C CNN "Manufacturer PN"
 	1    2850 4800
 	0    1    1    0
@@
 F 2 "RespiraWorks_Std:D_SOD-323F" H 2850 4325 50  0001 C CNN
 F 3 "https://assets.nexperia.com/documents/data-sheet/BAT54J.pdf" H 2850 4500 50  0001 C CNN
+F 4 "Nexperia" H 2850 4500 50  0001 C CNN "Manufacturer"
+F 5 "BAT54J,115" H 2850 4500 50  0001 C CNN "Manufacturer PN"
 	1    2850 4500
 	0    1    -1   0

Commit message: Stephanie fixes, net names
Removed duplicate global I2C pull-ups
Added missing BMP280 pin 7
Correcting pin names etc. on LM4120 voltage reference
Finished standardizing net names
Connections:
- net labels added: IAdp, IBat, PSys, Pack-P, RegN
- net labels removed: IADPT, IBAT, PACK_P, PSYS, REGN
Changed lines of the file:
@@
 $EndComp
 Text HLabel 7850 5000 2    50   Output ~ 0
-PSYS
+PSys
 Text HLabel 9100 5250 2    50   Output ~ 0
-IBAT
+IBat
 Text HLabel 9100 4700 2    50   Output ~ 0
-IADPT
+IAdp
 Wire Wire Line
 	7850 5000 7750 5000
@@
 	7150 5500 6850 5500
 Text Label 6950 5500 0    50   ~ 0
-REGN
+RegN
 Wire Wire Line
 	6850 4500 7150 4500
@@
 	7800 2000 8300 2000
 Text Label 3200 5000 0    50   ~ 0
-REGN
+RegN
 Wire Wire Line
 	5050 5100 5300 5100
@@
 	2850 4950 2400 4950
 Text Label 2400 4350 0    50   ~ 0
-PACK_P
+Pack-P
 Text Label 2400 4950 0    50   ~ 0
 Vin-Adp
@@
 Connection ~ 7800 3200
 Text HLabel 8850 3200 2    50   BiDi ~ 0
-PACK_P
+Pack-P
 Wire Wire Line
 	1800 2000 1250 2000
@@
 	-1   0    0    -1
 $EndComp
-Text Label 8350 3200 0    50   ~ 0
-PACK_P
 Text Label 3350 6050 0    50   ~ 0
-PACK_P
+Pack-P
 Wire Wire Line
 	3600 6050 3350 6050

Commit message: Diode symbol
Changed Schottky (BAT54J) from Diode library to Device library symbol
Parts:
- D? (x2): symbol Diode:BAT54J -> Device:D_Schottky
Changed lines of the file:
@@
 5.4V nominal
 $Comp
-L Diode:BAT54J D?
+L Device:D_Schottky D?
 U 1 1 60756F63
 P 2850 4800
@@
 $EndComp
 $Comp
-L Diode:BAT54J D?
+L Device:D_Schottky D?
 U 1 1 6075D700
 P 2850 4500

Commit message: Packages to RespiraWorks library
Parts:
- Q? (x4): symbol RespiraWorks_Std:CSD17304Q3 -> Device:Q_NMOS_SGD
- Q?: footprint Package_SON:Diodes_PowerDI3333-8 -> RespiraWorks_Std:Diodes_PowerDI3333-8
Changed lines of the file:
@@
 Connection ~ 3100 2650
 $Comp
-L RespiraWorks_Std:CSD17304Q3 Q?
+L Device:Q_NMOS_SGD Q?
 U 1 1 60580FC0
 P 2100 2100
@@
 $EndComp
 $Comp
-L RespiraWorks_Std:CSD17304Q3 Q?
+L Device:Q_NMOS_SGD Q?
 U 1 1 60321C9D
 P 2700 2100
@@
 Connection ~ 4800 2000
 $Comp
-L RespiraWorks_Std:CSD17304Q3 Q?
+L Device:Q_NMOS_SGD Q?
 U 1 1 60337344
 P 4700 2200
@@
 $EndComp
 $Comp
-L RespiraWorks_Std:CSD17304Q3 Q?
+L Device:Q_NMOS_SGD Q?
 U 1 1 6032FCBA
 P 4350 2100
@@
 F 0 "Q?" V 7850 2700 50  0000 L CNN
 F 1 "DMP3013SFV-7" V 7950 2550 50  0000 L CNN
-F 2 "Package_SON:Diodes_PowerDI3333-8" H 8300 2850 50  0001 C CNN
+F 2 "RespiraWorks_Std:Diodes_PowerDI3333-8" H 8300 2850 50  0001 C CNN
 F 3 "https://www.diodes.com/assets/Datasheets/DMP3013SFV.pdf" H 7700 3000 50  0001 C CNN
 F 4 "Diodes Inc." V 7800 3000 50  0001 C CNN "Manufacturer"
