File: pcb/battery_charger.sch (KiCad schematic (older format))
At the start: 59 parts

Commit message: updated alt parts on the battery charger page, updated link on system monitor ADC to the RW library
Parts:
- Q? (x4): value CSD18563Q5A -> BSC065N06LS5ATMA1; Manufacturer Texas Instruments -> Infineon; Manufacturer PN CSD18563Q5A -> BSC065N06LS5ATMA1
- Q?: value DMP3013SFV-7 -> SI7145DP-T1-GE3; footprint RespiraWorks_Std:Diodes_PowerDI3333-8 -> RespiraWorks:VSONP-8-1EP_5x6_P1.27mm; symbol RespiraWorks_Std:DMP3013SFV-7 -> Device:Q_PMOS_SGD; Manufacturer Diodes Inc. -> Vishay Siliconix; Manufacturer PN DMP3013SFV-7 -> SI7145DP-T1-GE3
Changed lines of the file:
@@
 AR Path="/5FCD4B8E/603C510C/60567144/60580FC0" Ref="Q?"  Part="1"
 AR Path="/6041384A/60567144/60580FC0" Ref="Q?"  Part="1"
-F 0 "Q?" V 2500 2100 50  0000 C CNN
-F 1 "CSD18563Q5A" V 2400 2150 50  0000 C CNN
+F 0 "Q?" V 2650 2100 50  0000 C CNN
+F 1 "BSC065N06LS5ATMA1" V 2550 2100 50  0000 C CNN
 F 2 "RespiraWorks:VSONP-8-1EP_5x6_P1.27mm" H 2300 2025 50  0001 L CIN
-F 3 "https://www.ti.com/lit/ds/symlink/csd18563q5a.pdf" V 2100 2100 50  0001 L CNN
-F 4 "Texas Instruments" V 2100 2100 50  0001 C CNN "Manufacturer"
-F 5 "CSD18563Q5A" V 2100 2100 50  0001 C CNN "Manufacturer PN"
+F 3 "https://www.infineon.com/dgdl/Infineon-BSC065N06LS5-DS-v02_00-EN.pdf?fileId=5546d4625c54d85b015cc5a9ad087b39" V 2100 2100 50  0001 L CNN
+F 4 "Infineon" V 2100 2100 50  0001 C CNN "Manufacturer"
+F 5 "BSC065N06LS5ATMA1" V 2100 2100 50  0001 C CNN "Manufacturer PN"
 	1    2100 2100
 	0    -1   -1   0
@@
 AR Path="/6041384A/60567144/60321C9D" Ref="Q?"  Part="1"
 F 0 "Q?" V 3100 2100 50  0000 C CNN
-F 1 "CSD18563Q5A" V 3000 2150 50  0000 C CNN
+F 1 "BSC065N06LS5ATMA1" V 3000 2150 50  0000 C CNN
 F 2 "RespiraWorks:VSONP-8-1EP_5x6_P1.27mm" H 2900 2025 50  0001 L CIN
-F 3 "https://www.ti.com/lit/ds/symlink/csd18563q5a.pdf" V 2700 2100 50  0001 L CNN
-F 4 "Texas Instruments" V 2700 2100 50  0001 C CNN "Manufacturer"
-F 5 "CSD18563Q5A" V 2700 2100 50  0001 C CNN "Manufacturer PN"
+F 3 "https://www.infineon.com/dgdl/Infineon-BSC065N06LS5-DS-v02_00-EN.pdf?fileId=5546d4625c54d85b015cc5a9ad087b39" V 2700 2100 50  0001 L CNN
+F 4 "Infineon" V 2700 2100 50  0001 C CNN "Manufacturer"
+F 5 "BSC065N06LS5ATMA1" V 2700 2100 50  0001 C CNN "Manufacturer PN"
 	1    2700 2100
 	0    1    -1   0
@@
 AR Path="/5FCD4B8E/603C510C/60567144/60337344" Ref="Q?"  Part="1"
 AR Path="/6041384A/60567144/60337344" Ref="Q?"  Part="1"
-F 0 "Q?" H 4750 2600 50  0000 C CNN
-F 1 "CSD18563Q5A" H 4900 2500 50  0000 C CNN
+F 0 "Q?" H 4800 2600 50  0000 C CNN
+F 1 "BSC065N06LS5ATMA1" H 4900 2500 50  0000 C CNN
 F 2 "RespiraWorks:VSONP-8-1EP_5x6_P1.27mm" H 4900 2125 50  0001 L CIN
-F 3 "https://www.ti.com/lit/ds/symlink/csd18563q5a.pdf" V 4700 2200 50  0001 L CNN
-F 4 "Texas Instruments" V 4700 2200 50  0001 C CNN "Manufacturer"
-F 5 "CSD18563Q5A" V 4700 2200 50  0001 C CNN "Manufacturer PN"
+F 3 "https://www.infineon.com/dgdl/Infineon-BSC065N06LS5-DS-v02_00-EN.pdf?fileId=5546d4625c54d85b015cc5a9ad087b39" V 4700 2200 50  0001 L CNN
+F 4 "Infineon" V 4700 2200 50  0001 C CNN "Manufacturer"
+F 5 "BSC065N06LS5ATMA1" V 4700 2200 50  0001 C CNN "Manufacturer PN"
 	1    4700 2200
 	1    0    0    -1
@@
 AR Path="/5FCD4B8E/603C510C/60567144/6032FCBA" Ref="Q?"  Part="1"
 AR Path="/6041384A/60567144/6032FCBA" Ref="Q?"  Part="1"
-F 0 "Q?" V 4750 2100 50  0000 C CNN
-F 1 "CSD18563Q5A" V 4650 2150 50  0000 C CNN
+F 0 "Q?" V 4800 2100 50  0000 C CNN
+F 1 "BSC065N06LS5ATMA1" V 4700 2150 50  0000 C CNN
 F 2 "RespiraWorks:VSONP-8-1EP_5x6_P1.27mm" H 4550 2025 50  0001 L CIN
-F 3 "https://www.ti.com/lit/ds/symlink/csd18563q5a.pdf" V 4350 2100 50  0001 L CNN
-F 4 "Texas Instruments" V 4350 2100 50  0001 C CNN "Manufacturer"
-F 5 "CSD18563Q5A" V 4350 2100 50  0001 C CNN "Manufacturer PN"
+F 3 "https://www.infineon.com/dgdl/Infineon-BSC065N06LS5-DS-v02_00-EN.pdf?fileId=5546d4625c54d85b015cc5a9ad087b39" V 4350 2100 50  0001 L CNN
+F 4 "Infineon" V 4350 2100 50  0001 C CNN "Manufacturer"
+F 5 "BSC065N06LS5ATMA1" V 4350 2100 50  0001 C CNN "Manufacturer PN"
 	1    4350 2100
 	0    -1   -1   0
 $EndComp
 $Comp
-L RespiraWorks_Std:DMP3013SFV-7 Q?
+L Device:Q_PMOS_SGD Q?
 U 1 1 605810DE
-P 7800 3000
+P 7700 3000
 AR Path="/601A64F8/605810DE" Ref="Q?"  Part="1"
 AR Path="/601A64F8/60567144/605810DE" Ref="Q?"  Part="1"
@@
 AR Path="/5FCD4B8E/603C510C/60567144/605810DE" Ref="Q?"  Part="1"
 AR Path="/6041384A/60567144/605810DE" Ref="Q?"  Part="1"
-F 0 "Q?" V 7850 2700 50  0000 L CNN
-F 1 "DMP3013SFV-7" V 7950 2550 50  0000 L CNN
-F 2 "RespiraWorks_Std:Diodes_PowerDI3333-8" H 8300 2850 50  0001 C CNN
-F 3 "https://www.diodes.com/assets/Datasheets/DMP3013SFV.pdf" H 7700 3000 50  0001 C CNN
-F 4 "Diodes Inc." V 7800 3000 50  0001 C CNN "Manufacturer"
-F 5 "DMP3013SFV-7" V 7800 3000 50  0001 C CNN "Manufacturer PN"
-	1    7800 3000
+F 0 "Q?" H 7950 2950 50  0000 L CNN
+F 1 "SI7145DP-T1-GE3" H 7950 3050 50  0000 L CNN
+F 2 "RespiraWorks:VSONP-8-1EP_5x6_P1.27mm" H 8200 2850 50  0001 C CNN
+F 3 "https://www.vishay.com/docs/64814/si7145dp.pdf" H 7600 3000 50  0001 C CNN
+F 4 "Vishay Siliconix" V 7700 3000 50  0001 C CNN "Manufacturer"
+F 5 "SI7145DP-T1-GE3" V 7700 3000 50  0001 C CNN "Manufacturer PN"
+	1    7700 3000
 	1    0    0    1
 $EndComp

Commit message: copied over NMOS and PMOS SGD symbols to RW library and swapped to RW library in schematic
Parts:
- Q? (x4): symbol Device:Q_NMOS_SGD -> RespiraWorks_Std:Q_NMOS_SGD
- Q?: symbol Device:Q_PMOS_SGD -> RespiraWorks_Std:Q_PMOS_SGD
Changed lines of the file:
@@
 	1800 2000 1900 2000
 Connection ~ 3100 2650
-$Comp
-L Device:Q_NMOS_SGD Q?
-U 1 1 60580FC0
-P 2100 2100
-AR Path="/601A64F8/60580FC0" Ref="Q?"  Part="1"
-AR Path="/601A64F8/60567144/60580FC0" Ref="Q?"  Part="1"
-AR Path="/6023BF6A/60567144/60580FC0" Ref="Q?"  Part="1"
-AR Path="/5FCD4B8E/603C510C/60567144/60580FC0" Ref="Q?"  Part="1"
-AR Path="/6041384A/60567144/60580FC0" Ref="Q?"  Part="1"
-F 0 "Q?" V 2650 2100 50  0000 C CNN
-F 1 "BSC065N06LS5ATMA1" V 2550 2100 50  0000 C CNN
-F 2 "RespiraWorks:VSONP-8-1EP_5x6_P1.27mm" H 2300 2025 50  0001 L CIN
-F 3 "https://www.infineon.com/dgdl/Infineon-BSC065N06LS5-DS-v02_00-EN.pdf?fileId=5546d4625c54d85b015cc5a9ad087b39" V 2100 2100 50  0001 L CNN
-F 4 "Infineon" V 2100 2100 50  0001 C CNN "Manufacturer"
-F 5 "BSC065N06LS5ATMA1" V 2100 2100 50  0001 C CNN "Manufacturer PN"
-	1    2100 2100
-	0    -1   -1   0
-$EndComp
 Wire Wire Line
 	2300 2000 2350 2000
@@
 $EndComp
 $Comp
-L Device:Q_NMOS_SGD Q?
+L RespiraWorks_Std:Q_NMOS_SGD Q?
 U 1 1 60321C9D
 P 2700 2100
@@
 Connection ~ 4800 2000
 $Comp
-L Device:Q_NMOS_SGD Q?
+L RespiraWorks_Std:Q_NMOS_SGD Q?
 U 1 1 60337344
 P 4700 2200
@@
 $EndComp
 $Comp
-L Device:Q_NMOS_SGD Q?
+L RespiraWorks_Std:Q_PMOS_SGD Q?
+U 1 1 605810DE
+P 7700 3000
+AR Path="/601A64F8/605810DE" Ref="Q?"  Part="1"
+AR Path="/601A64F8/60567144/605810DE" Ref="Q?"  Part="1"
+AR Path="/6023BF6A/60567144/605810DE" Ref="Q?"  Part="1"
+AR Path="/5FCD4B8E/603C510C/60567144/605810DE" Ref="Q?"  Part="1"
+AR Path="/6041384A/60567144/605810DE" Ref="Q?"  Part="1"
+F 0 "Q?" H 7950 2950 50  0000 L CNN
+F 1 "SI7145DP-T1-GE3" H 7950 3050 50  0000 L CNN
+F 2 "RespiraWorks:VSONP-8-1EP_5x6_P1.27mm" H 8200 2850 50  0001 C CNN
+F 3 "https://www.vishay.com/docs/64814/si7145dp.pdf" H 7600 3000 50  0001 C CNN
+F 4 "Vishay Siliconix" V 7700 3000 50  0001 C CNN "Manufacturer"
+F 5 "SI7145DP-T1-GE3" V 7700 3000 50  0001 C CNN "Manufacturer PN"
+	1    7700 3000
+	1    0    0    1
+$EndComp
+NoConn ~ 6850 5300
+Text Notes 700  4250 0    50   ~ 0
+Vin-Adp used when >13V\n(ACDET pin > 2.4V)
+Text Notes 9450 4800 0    50   ~ 0
+0.4 or 0.8V/A from Vin_Adp\n(with 10mΩ ACP/N resistor)
+Text Notes 9400 5300 0    50   ~ 0
+0.2V/A charging, 0.8 or 1.6V/A discharging\n(with 10mΩ ACP/N resistor)
+Connection ~ 8500 5250
+Text Notes 6950 5400 0    50   ~ 0
+5.4V nominal
+$Comp
+L Device:D_Schottky D?
+U 1 1 60756F63
+P 2850 4800
+AR Path="/6041384A/60567D6E/60756F63" Ref="D?"  Part="1"
+AR Path="/6041384A/60567144/60756F63" Ref="D?"  Part="1"
+F 0 "D?" H 2850 4900 50  0000 C CNN
+F 1 "BAT54J" V 2850 4600 50  0000 C CNN
+F 2 "RespiraWorks_Std:D_SOD-323F" H 2850 4625 50  0001 C CNN
+F 3 "https://assets.nexperia.com/documents/data-sheet/BAT54J.pdf" H 2850 4800 50  0001 C CNN
+F 4 "Nexperia" H 2850 4800 50  0001 C CNN "Manufacturer"
+F 5 "BAT54J,115" H 2850 4800 50  0001 C CNN "Manufacturer PN"
+	1    2850 4800
+	0    1    1    0
+$EndComp
+$Comp
+L Device:D_Schottky D?
+U 1 1 6075D700
+P 2850 4500
+AR Path="/6041384A/60567D6E/6075D700" Ref="D?"  Part="1"
+AR Path="/6041384A/60567144/6075D700" Ref="D?"  Part="1"
+F 0 "D?" H 2850 4600 50  0000 C CNN
+F 1 "BAT54J" V 2850 4300 50  0000 C CNN
+F 2 "RespiraWorks_Std:D_SOD-323F" H 2850 4325 50  0001 C CNN
+F 3 "https://assets.nexperia.com/documents/data-sheet/BAT54J.pdf" H 2850 4500 50  0001 C CNN
+F 4 "Nexperia" H 2850 4500 50  0001 C CNN "Manufacturer"
+F 5 "BAT54J,115" H 2850 4500 50  0001 C CNN "Manufacturer PN"
+	1    2850 4500
+	0    1    -1   0
+$EndComp
+Wire Wire Line
+	2850 4650 3050 4650
+Connection ~ 2850 4650
+$Comp
+L RespiraWorks_Std:Q_NMOS_SGD Q?
+U 1 1 60580FC0
+P 2100 2100
+AR Path="/601A64F8/60580FC0" Ref="Q?"  Part="1"
+AR Path="/601A64F8/60567144/60580FC0" Ref="Q?"  Part="1"
+AR Path="/6023BF6A/60567144/60580FC0" Ref="Q?"  Part="1"
+AR Path="/5FCD4B8E/603C510C/60567144/60580FC0" Ref="Q?"  Part="1"
+AR Path="/6041384A/60567144/60580FC0" Ref="Q?"  Part="1"
+F 0 "Q?" V 2650 2100 50  0000 C CNN
+F 1 "BSC065N06LS5ATMA1" V 2550 2100 50  0000 C CNN
+F 2 "RespiraWorks:VSONP-8-1EP_5x6_P1.27mm" H 2300 2025 50  0001 L CIN
+F 3 "https://www.infineon.com/dgdl/Infineon-BSC065N06LS5-DS-v02_00-EN.pdf?fileId=5546d4625c54d85b015cc5a9ad087b39" V 2100 2100 50  0001 L CNN
+F 4 "Infineon" V 2100 2100 50  0001 C CNN "Manufacturer"
+F 5 "BSC065N06LS5ATMA1" V 2100 2100 50  0001 C CNN "Manufacturer PN"
+	1    2100 2100
+	0    -1   -1   0
+$EndComp
+$Comp
+L RespiraWorks_Std:Q_NMOS_SGD Q?
 U 1 1 6032FCBA
 P 4350 2100
@@
 	0    -1   -1   0
 $EndComp
-$Comp
-L Device:Q_PMOS_SGD Q?
-U 1 1 605810DE
-P 7700 3000
-AR Path="/601A64F8/605810DE" Ref="Q?"  Part="1"
-AR Path="/601A64F8/60567144/605810DE" Ref="Q?"  Part="1"
-AR Path="/6023BF6A/60567144/605810DE" Ref="Q?"  Part="1"
-AR Path="/5FCD4B8E/603C510C/60567144/605810DE" Ref="Q?"  Part="1"
-AR Path="/6041384A/60567144/605810DE" Ref="Q?"  Part="1"
-F 0 "Q?" H 7950 2950 50  0000 L CNN
-F 1 "SI7145DP-T1-GE3" H 7950 3050 50  0000 L CNN
-F 2 "RespiraWorks:VSONP-8-1EP_5x6_P1.27mm" H 8200 2850 50  0001 C CNN
-F 3 "https://www.vishay.com/docs/64814/si7145dp.pdf" H 7600 3000 50  0001 C CNN
-F 4 "Vishay Siliconix" V 7700 3000 50  0001 C CNN "Manufacturer"
-F 5 "SI7145DP-T1-GE3" V 7700 3000 50  0001 C CNN "Manufacturer PN"
-	1    7700 3000
-	1    0    0    1
-$EndComp
-NoConn ~ 6850 5300
-Text Notes 700  4250 0    50   ~ 0
-Vin-Adp used when >13V\n(ACDET pin > 2.4V)
-Text Notes 9450 4800 0    50   ~ 0
-0.4 or 0.8V/A from Vin_Adp\n(with 10mΩ ACP/N resistor)
-Text Notes 9400 5300 0    50   ~ 0
-0.2V/A charging, 0.8 or 1.6V/A discharging\n(with 10mΩ ACP/N resistor)
-Connection ~ 8500 5250
-Text Notes 6950 5400 0    50   ~ 0
-5.4V nominal
-$Comp
-L Device:D_Schottky D?
-U 1 1 60756F63
-P 2850 4800
-AR Path="/6041384A/60567D6E/60756F63" Ref="D?"  Part="1"
-AR Path="/6041384A/60567144/60756F63" Ref="D?"  Part="1"
-F 0 "D?" H 2850 4900 50  0000 C CNN
-F 1 "BAT54J" V 2850 4600 50  0000 C CNN
-F 2 "RespiraWorks_Std:D_SOD-323F" H 2850 4625 50  0001 C CNN
-F 3 "https://assets.nexperia.com/documents/data-sheet/BAT54J.pdf" H 2850 4800 50  0001 C CNN
-F 4 "Nexperia" H 2850 4800 50  0001 C CNN "Manufacturer"
-F 5 "BAT54J,115" H 2850 4800 50  0001 C CNN "Manufacturer PN"
-	1    2850 4800
-	0    1    1    0
-$EndComp
-$Comp
-L Device:D_Schottky D?
-U 1 1 6075D700
-P 2850 4500
-AR Path="/6041384A/60567D6E/6075D700" Ref="D?"  Part="1"
-AR Path="/6041384A/60567144/6075D700" Ref="D?"  Part="1"
-F 0 "D?" H 2850 4600 50  0000 C CNN
-F 1 "BAT54J" V 2850 4300 50  0000 C CNN
-F 2 "RespiraWorks_Std:D_SOD-323F" H 2850 4325 50  0001 C CNN
-F 3 "https://assets.nexperia.com/documents/data-sheet/BAT54J.pdf" H 2850 4500 50  0001 C CNN
-F 4 "Nexperia" H 2850 4500 50  0001 C CNN "Manufacturer"
-F 5 "BAT54J,115" H 2850 4500 50  0001 C CNN "Manufacturer PN"
-	1    2850 4500
-	0    1    -1   0
-$EndComp
-Wire Wire Line
-	2850 4650 3050 4650
-Connection ~ 2850 4650
 $EndSCHEMATC
