File: pcb/battery_balancer.sch (KiCad schematic (older format))
At the start: 0 parts

Commit message: added battery balancer/fuel gauge
Parts:
- added C? (x5): 0.01uF, Capacitor_SMD:C_0603_1608Metric, symbol Device:C
- added C? (x2): 0.1uF, Capacitor_SMD:C_0603_1608Metric, symbol Device:C
- added C? (x4): 0.47uF, Capacitor_SMD:C_0603_1608Metric, symbol Device:C
- added J?: Conn_01x05_Male, symbol Connector:Conn_01x05_Male
- added Q? (x2): CSD17304Q3, Package_SON:VSON-8_3.3x3.3mm_P0.65mm_NexFET, symbol RespiraWorks_Std:CSD17304Q3
- added R?: 0.005, Capacitor_SMD:C_1206_3216Metric, symbol Device:R
- added R? (x4): 24k, Capacitor_SMD:C_1206_3216Metric, symbol Device:R
- added R?: 10, Capacitor_SMD:C_1206_3216Metric, symbol Device:R
- added R? (x2): 1k, Capacitor_SMD:C_1206_3216Metric, symbol Device:R
- added R?: 2k, Capacitor_SMD:C_1206_3216Metric, symbol Device:R
- added R? (x2): 100, Capacitor_SMD:C_1206_3216Metric, symbol Device:R
- added TH?: 10k, Resistor_SMD:R_0603_1608Metric, symbol Device:Thermistor_NTC
- added U?: MAX17320G20+, Package_DFN_QFN:WQFN-24-1EP_4x4mm_P0.5mm_EP2.6x2.6mm, symbol RespiraWorks:MAX17320G20+
Connections:
- net labels added: ALRT, BAT_N, BAT_P, GND, SCL, SDA, SYS_N, SYS_P
- wire segments 0 -> 72
- no-connect marks 0 -> 3
Other:
- note added: "Battery Balancing Connector"

Commit message: clean up, add part numbers to parts, added design comments
Parts:
- R?: footprint Capacitor_SMD:C_1206_3216Metric -> Resistor_SMD:R_1206_3216Metric
- R? (x4): value 24k -> 49.9; footprint Capacitor_SMD:C_1206_3216Metric -> Resistor_SMD:R_1206_3216Metric
- R? (x5): footprint Capacitor_SMD:C_1206_3216Metric -> RespiraWorks_Std:R_0603_1608Metric
- R?: footprint Capacitor_SMD:C_1206_3216Metric -> RespiraWorks_Std:R_1206_3216Metric
Other:
- note added: "Balancing current: 100mA MAX"
- moved on the sheet: C?
Changed lines of the file:
@@
 F 0 "R?" H 6900 5250 50  0000 C CNN
 F 1 "0.005" H 6950 5150 50  0000 C CNN
-F 2 "Capacitor_SMD:C_1206_3216Metric" V 6680 5200 50  0001 C CNN
+F 2 "Resistor_SMD:R_1206_3216Metric" V 6680 5200 50  0001 C CNN
 F 3 "~" H 6750 5200 50  0001 C CNN
 	1    6750 5200
@@
 AR Path="/601A64F8/60567757/603D7932" Ref="R?"  Part="1"
 F 0 "R?" V 7350 4750 50  0000 C CNN
-F 1 "24k" V 7250 4750 50  0000 C CNN
-F 2 "Capacitor_SMD:C_1206_3216Metric" V 7080 4750 50  0001 C CNN
+F 1 "49.9" V 7250 4750 50  0000 C CNN
+F 2 "Resistor_SMD:R_1206_3216Metric" V 7080 4750 50  0001 C CNN
 F 3 "~" H 7150 4750 50  0001 C CNN
 	1    7150 4750
@@
 AR Path="/601A64F8/60567757/603DA817" Ref="R?"  Part="1"
 F 0 "R?" V 7350 4450 50  0000 C CNN
-F 1 "24k" V 7250 4450 50  0000 C CNN
-F 2 "Capacitor_SMD:C_1206_3216Metric" V 7080 4450 50  0001 C CNN
+F 1 "49.9" V 7250 4450 50  0000 C CNN
+F 2 "Resistor_SMD:R_1206_3216Metric" V 7080 4450 50  0001 C CNN
 F 3 "~" H 7150 4450 50  0001 C CNN
 	1    7150 4450
@@
 AR Path="/601A64F8/60567757/603DAA1D" Ref="R?"  Part="1"
 F 0 "R?" V 7350 3850 50  0000 C CNN
-F 1 "24k" V 7250 3850 50  0000 C CNN
-F 2 "Capacitor_SMD:C_1206_3216Metric" V 7080 3850 50  0001 C CNN
+F 1 "49.9" V 7250 3850 50  0000 C CNN
+F 2 "Resistor_SMD:R_1206_3216Metric" V 7080 3850 50  0001 C CNN
 F 3 "~" H 7150 3850 50  0001 C CNN
 	1    7150 3850
@@
 AR Path="/601A64F8/60567757/603DA8CE" Ref="R?"  Part="1"
 F 0 "R?" V 7350 4150 50  0000 C CNN
-F 1 "24k" V 7250 4150 50  0000 C CNN
-F 2 "Capacitor_SMD:C_1206_3216Metric" V 7080 4150 50  0001 C CNN
+F 1 "49.9" V 7250 4150 50  0000 C CNN
+F 2 "Resistor_SMD:R_1206_3216Metric" V 7080 4150 50  0001 C CNN
 F 3 "~" H 7150 4150 50  0001 C CNN
 	1    7150 4150
@@
 F 0 "R?" H 9950 3450 50  0000 C CNN
 F 1 "10" H 9950 3350 50  0000 C CNN
-F 2 "Capacitor_SMD:C_1206_3216Metric" V 9730 3400 50  0001 C CNN
+F 2 "RespiraWorks_Std:R_0603_1608Metric" V 9730 3400 50  0001 C CNN
 F 3 "~" H 9800 3400 50  0001 C CNN
 	1    9800 3400
@@
 F 0 "R?" H 7200 3050 50  0000 C CNN
 F 1 "1k" H 7200 2950 50  0000 C CNN
-F 2 "Capacitor_SMD:C_1206_3216Metric" V 6980 3000 50  0001 C CNN
+F 2 "RespiraWorks_Std:R_0603_1608Metric" V 6980 3000 50  0001 C CNN
 F 3 "~" H 7050 3000 50  0001 C CNN
 	1    7050 3000
@@
 F 0 "R?" H 4450 2150 50  0000 C CNN
 F 1 "1k" H 4450 2050 50  0000 C CNN
-F 2 "Capacitor_SMD:C_1206_3216Metric" V 4280 2100 50  0001 C CNN
+F 2 "RespiraWorks_Std:R_0603_1608Metric" V 4280 2100 50  0001 C CNN
 F 3 "~" H 4350 2100 50  0001 C CNN
 	1    4350 2100
@@
 F 0 "R?" H 4550 2050 50  0000 C CNN
 F 1 "2k" H 4550 2150 50  0000 C CNN
-F 2 "Capacitor_SMD:C_1206_3216Metric" V 4580 2100 50  0001 C CNN
+F 2 "RespiraWorks_Std:R_1206_3216Metric" V 4580 2100 50  0001 C CNN
 F 3 "~" H 4650 2100 50  0001 C CNN
 	1    4650 2100
@@
 L Device:C C?
 U 1 1 604128F9
-P 2400 3900
+P 4000 3900
 AR Path="/601A64F8/604128F9" Ref="C?"  Part="1"
 AR Path="/601A64F8/60567144/604128F9" Ref="C?"  Part="1"
 AR Path="/601A64F8/60567757/604128F9" Ref="C?"  Part="1"
-F 0 "C?" H 2550 3950 50  0000 L CNN
-F 1 "0.47uF" H 2550 3850 50  0000 L CNN
-F 2 "Capacitor_SMD:C_0603_1608Metric" H 2438 3750 50  0001 C CNN
-F 3 "~" H 2400 3900 50  0001 C CNN
-	1    2400 3900
+F 0 "C?" H 4150 3950 50  0000 L CNN
+F 1 "0.47uF" H 4150 3850 50  0000 L CNN
+F 2 "Capacitor_SMD:C_0603_1608Metric" H 4038 3750 50  0001 C CNN
+F 3 "~" H 4000 3900 50  0001 C CNN
+	1    4000 3900
 	1    0    0    -1
 $EndComp
@@
 Wire Wire Line
 	9800 1550 9800 3250
-Wire Wire Line
-	6100 1850 5800 1850
 $Comp
 L Device:R R?
@@
 F 0 "R?" H 5950 2050 50  0000 C CNN
 F 1 "100" H 5950 1950 50  0000 C CNN
-F 2 "Capacitor_SMD:C_1206_3216Metric" V 5730 2000 50  0001 C CNN
+F 2 "RespiraWorks_Std:R_0603_1608Metric" V 5730 2000 50  0001 C CNN
 F 3 "~" H 5800 2000 50  0001 C CNN
 	1    5800 2000
@@
 F 0 "R?" H 5450 2050 50  0000 C CNN
 F 1 "100" H 5450 1950 50  0000 C CNN
-F 2 "Capacitor_SMD:C_1206_3216Metric" V 5230 2000 50  0001 C CNN
+F 2 "RespiraWorks_Std:R_0603_1608Metric" V 5230 2000 50  0001 C CNN
 F 3 "~" H 5300 2000 50  0001 C CNN
 	1    5300 2000
@@
 	3250 5250 3250 5550
 Wire Wire Line
-	4850 3750 2400 3750
+	4850 3750 4000 3750
 Text Label 7650 5050 0    50   ~ 0
 BAT_N
@@
 L power:GND #PWR?
 U 1 1 6046FA21
-P 2400 4050
+P 4000 4050
 AR Path="/601A64F8/6046FA21" Ref="#PWR?"  Part="1"
 AR Path="/601A64F8/60567757/6046FA21" Ref="#PWR?"  Part="1"
-F 0 "#PWR?" H 2400 3800 50  0001 C CNN
-F 1 "GND" H 2405 3877 50  0000 C CNN
-F 2 "" H 2400 4050 50  0001 C CNN
-F 3 "" H 2400 4050 50  0001 C CNN
-	1    2400 4050
+F 0 "#PWR?" H 4000 3800 50  0001 C CNN
+F 1 "GND" H 4005 3877 50  0000 C CNN
+F 2 "" H 4000 4050 50  0001 C CNN
+F 3 "" H 4000 4050 50  0001 C CNN
+	1    4000 4050
 	1    0    0    -1
 $EndComp
@@
 Text HLabel 10050 1550 2    50   Input ~ 0
 BAT_P
+Wire Wire Line
+	6100 1850 5800 1850
+Connection ~ 5800 1850
+Text Notes 7400 3750 0    50   ~ 0
+Balancing current: 100mA MAX
 $EndSCHEMATC

Commit message: WIP implement PR comments
Parts:
- added R?: 10k, RespiraWorks_Std:R_0603_1608Metric, symbol Device:R
- J?: value Conn_01x05_Male -> BAT-BALANCE JST XH 5-pin; symbol Connector:Conn_01x05_Male -> Connector_Generic:Conn_01x05
Connections:
- wire segments 72 -> 75
- no-connect marks 3 -> 4
Other:
- note added: "IC max balancing current: 100mA\nSet balancing current: 71mA"
- note removed: "Balancing current: 100mA MAX"
- moved on the sheet: C?, R?
Changed lines of the file:
@@
-$EndComp
-$Comp
-L Connector:Conn_01x05_Male J?
-U 1 1 603D30AF
-P 8700 4250
-F 0 "J?" H 8672 4137 50  0000 R CNN
-F 1 "Conn_01x05_Male" H 8672 4228 50  0000 R CNN
-F 2 "" H 8700 4250 50  0001 C CNN
-F 3 "https://www.jst-mfg.com/product/pdf/eng/eXH.pdf" H 8700 4250 50  0001 C CNN
-F 4 "JST" H 8700 4250 50  0001 C CNN "Manufacturer"
-F 5 "B5B-XH-A(LF)(SN)" H 8672 4319 50  0000 R CNN "Manufacturer PN"
-	1    8700 4250
-	-1   0    0    1
 $EndComp
 $Comp
@@
 L Device:R R?
 U 1 1 603DAD46
-P 9800 3400
+P 9950 3400
 AR Path="/601A64F8/603DAD46" Ref="R?"  Part="1"
 AR Path="/601A64F8/60567144/603DAD46" Ref="R?"  Part="1"
 AR Path="/601A64F8/60567757/603DAD46" Ref="R?"  Part="1"
 AR Path="/6023BF6A/60567757/603DAD46" Ref="R?"  Part="1"
-F 0 "R?" H 9950 3450 50  0000 C CNN
-F 1 "10" H 9950 3350 50  0000 C CNN
-F 2 "RespiraWorks_Std:R_0603_1608Metric" V 9730 3400 50  0001 C CNN
-F 3 "~" H 9800 3400 50  0001 C CNN
-	1    9800 3400
+F 0 "R?" H 10100 3450 50  0000 C CNN
+F 1 "10" H 10100 3350 50  0000 C CNN
+F 2 "RespiraWorks_Std:R_0603_1608Metric" V 9880 3400 50  0001 C CNN
+F 3 "~" H 9950 3400 50  0001 C CNN
+	1    9950 3400
 	1    0    0    -1
 $EndComp
@@
 Wire Wire Line
 	7300 3850 8300 3850
-Text Notes 8550 4550 0    50   ~ 0
-Battery Balancing Connector
-Wire Wire Line
-	6300 5050 6750 5050
-Wire Wire Line
-	6600 4750 6300 4750
+Wire Wire Line
+	6600 4750 6500 4750
 Wire Wire Line
 	6750 5350 6750 6100
@@
 Wire Wire Line
 	6600 4750 7000 4750
-Wire Wire Line
-	6750 5050 9800 5050
 Connection ~ 6750 5050
 $Comp
@@
 L Device:C C?
 U 1 1 603EA3B2
-P 9800 3700
+P 9950 3700
 AR Path="/601A64F8/603EA3B2" Ref="C?"  Part="1"
 AR Path="/601A64F8/60567144/603EA3B2" Ref="C?"  Part="1"
 AR Path="/601A64F8/60567757/603EA3B2" Ref="C?"  Part="1"
 AR Path="/6023BF6A/60567757/603EA3B2" Ref="C?"  Part="1"
-F 0 "C?" H 9950 3750 50  0000 L CNN
-F 1 "0.1uF" H 9950 3650 50  0000 L CNN
-F 2 "Capacitor_SMD:C_0603_1608Metric" H 9838 3550 50  0001 C CNN
-F 3 "~" H 9800 3700 50  0001 C CNN
-	1    9800 3700
+F 0 "C?" H 10100 3750 50  0000 L CNN
+F 1 "0.1uF" H 10100 3650 50  0000 L CNN
+F 2 "Capacitor_SMD:C_0603_1608Metric" H 9988 3550 50  0001 C CNN
+F 3 "~" H 9950 3700 50  0001 C CNN
+	1    9950 3700
 	1    0    0    -1
 $EndComp
@@
 Wire Wire Line
 	6300 3850 6600 3850
-Connection ~ 9800 3550
-Connection ~ 9800 1550
+Connection ~ 9950 3550
 Wire Wire Line
 	6300 3550 6500 3550
@@
 	1    0    0    -1
 $EndComp
-Connection ~ 6500 3550
-Wire Wire Line
-	6500 3550 9800 3550
 Wire Wire Line
 	6300 3250 6500 3250
@@
 $EndComp
 Wire Wire Line
-	9800 1550 9800 3250
+	9950 1550 9950 3250
 $Comp
 L Device:R R?
@@
 NoConn ~ 4850 4350
 Wire Wire Line
-	9800 3850 9800 5050
-Connection ~ 9800 5050
+	9950 3850 9950 5050
 Wire Wire Line
 	7050 3150 7050 3350
@@
 SYS_N
 Wire Wire Line
-	6400 1550 9800 1550
-Wire Wire Line
 	8300 3850 8300 4050
 Wire Wire Line
 	8300 4050 8500 4050
-Wire Wire Line
-	9800 5050 10050 5050
 Text HLabel 10050 5050 2    50   Input ~ 0
 BAT_N
-Wire Wire Line
-	9800 1550 10050 1550
 Text HLabel 10050 1550 2    50   Input ~ 0
 BAT_P
@@
 Connection ~ 5800 1850
 Text Notes 7400 3750 0    50   ~ 0
-Balancing current: 100mA MAX
+IC max balancing current: 100mA\nSet balancing current: 71mA
+Connection ~ 6500 4750
+Connection ~ 6500 5050
+Wire Wire Line
+	6500 5050 6750 5050
+Connection ~ 9950 1550
+Wire Wire Line
+	9950 1550 10050 1550
+Connection ~ 9950 5050
+Wire Wire Line
+	9950 5050 10050 5050
+Wire Wire Line
+	6300 5050 6500 5050
+Wire Wire Line
+	6750 5050 9950 5050
+Wire Wire Line
+	6400 1550 9950 1550
+Wire Wire Line
+	6300 4750 6500 4750
+Wire Wire Line
+	6500 3550 9950 3550
+Connection ~ 6500 3550
+$Comp
+L Connector_Generic:Conn_01x05 J?
+U 1 1 603D30AF
+P 8700 4250
+F 0 "J?" H 8900 4100 50  0000 R CNN
+F 1 "BAT-BALANCE JST XH 5-pin" H 9900 4200 50  0000 R CNN
+F 2 "" H 8700 4250 50  0001 C CNN
+F 3 "https://www.jst-mfg.com/product/pdf/eng/eXH.pdf" H 8700 4250 50  0001 C CNN
+F 4 "JST" H 8700 4250 50  0001 C CNN "Manufacturer"
+F 5 "B5B-XH-A(LF)(SN)" H 9550 4300 50  0000 R CNN "Manufacturer PN"
+	1    8700 4250
+	1    0    0    1
+$EndComp
+Text Notes 8800 4450 0    50   ~ 0
+Battery Balancing Connector
+NoConn ~ 8500 4450
+$Comp
+L Device:R R?
+U 1 1 6029693C
+P 3550 3900
+AR Path="/601A64F8/6029693C" Ref="R?"  Part="1"
+AR Path="/601A64F8/60567144/6029693C" Ref="R?"  Part="1"
+AR Path="/601A64F8/60567757/6029693C" Ref="R?"  Part="1"
+AR Path="/6023BF6A/60567757/6029693C" Ref="R?"  Part="1"
+F 0 "R?" H 3700 3950 50  0000 C CNN
+F 1 "10k" H 3700 3850 50  0000 C CNN
+F 2 "RespiraWorks_Std:R_0603_1608Metric" V 3480 3900 50  0001 C CNN
+F 3 "~" H 3550 3900 50  0001 C CNN
+	1    3550 3900
+	1    0    0    -1
+$EndComp
+Wire Wire Line
+	4000 3750 3550 3750
+Connection ~ 4000 3750
+$Comp
+L power:GND #PWR?
+U 1 1 6029AB22
+P 3550 4050
+AR Path="/601A64F8/6029AB22" Ref="#PWR?"  Part="1"
+AR Path="/601A64F8/60567757/6029AB22" Ref="#PWR?"  Part="1"
+AR Path="/6023BF6A/60567757/6029AB22" Ref="#PWR?"  Part="1"
+F 0 "#PWR?" H 3550 3800 50  0001 C CNN
+F 1 "GND" H 3555 3877 50  0000 C CNN
+F 2 "" H 3550 4050 50  0001 C CNN
+F 3 "" H 3550 4050 50  0001 C CNN
+	1    3550 4050
+	1    0    0    -1
+$EndComp
 $EndSCHEMATC

Commit message: updated footprints to reference to RW library
Parts:
- C? (x11): footprint Capacitor_SMD:C_0603_1608Metric -> RespiraWorks_Std:C_0603_1608Metric
- Q? (x2): footprint Package_SON:VSON-8_3.3x3.3mm_P0.65mm_NexFET -> RespiraWorks_Std:VSON-8_3.3x3.3mm_P0.65mm_NexFET
- R? (x5): footprint Resistor_SMD:R_1206_3216Metric -> RespiraWorks_Std:R_1206_3216Metric
- TH?: footprint Resistor_SMD:R_0603_1608Metric -> RespiraWorks_Std:R_0603_1608Metric
- U?: footprint Package_DFN_QFN:WQFN-24-1EP_4x4mm_P0.5mm_EP2.6x2.6mm -> RespiraWorks_Std:WQFN-24-1EP_4x4mm_P0.5mm_EP2.6x2.6mm
Changed lines of the file:
@@
 F 0 "U?" H 5575 2077 50  0000 C CNN
 F 1 "MAX17320G20+" H 5575 1986 50  0000 C CNN
-F 2 "Package_DFN_QFN:WQFN-24-1EP_4x4mm_P0.5mm_EP2.6x2.6mm" H 5500 1950 50  0001 C CNN
+F 2 "RespiraWorks_Std:WQFN-24-1EP_4x4mm_P0.5mm_EP2.6x2.6mm" H 5500 1950 50  0001 C CNN
 F 3 "https://datasheets.maximintegrated.com/en/ds/MAX17320.pdf" H 8300 4850 50  0001 C CNN
 F 4 "Maxim IC" H 5600 3800 50  0000 C CNN "Manufacturer"
@@
 F 0 "R?" H 6900 5250 50  0000 C CNN
 F 1 "0.005" H 6950 5150 50  0000 C CNN
-F 2 "Resistor_SMD:R_1206_3216Metric" V 6680 5200 50  0001 C CNN
+F 2 "RespiraWorks_Std:R_1206_3216Metric" V 6680 5200 50  0001 C CNN
 F 3 "~" H 6750 5200 50  0001 C CNN
 	1    6750 5200
@@
 F 0 "R?" V 7350 4750 50  0000 C CNN
 F 1 "49.9" V 7250 4750 50  0000 C CNN
-F 2 "Resistor_SMD:R_1206_3216Metric" V 7080 4750 50  0001 C CNN
+F 2 "RespiraWorks_Std:R_1206_3216Metric" V 7080 4750 50  0001 C CNN
 F 3 "~" H 7150 4750 50  0001 C CNN
 	1    7150 4750
@@
 F 0 "C?" H 6750 4650 50  0000 L CNN
 F 1 "0.01uF" H 6750 4550 50  0000 L CNN
-F 2 "Capacitor_SMD:C_0603_1608Metric" H 6638 4450 50  0001 C CNN
+F 2 "RespiraWorks_Std:C_0603_1608Metric" H 6638 4450 50  0001 C CNN
 F 3 "~" H 6600 4600 50  0001 C CNN
 	1    6600 4600
@@
 F 0 "C?" H 6650 4350 50  0000 L CNN
 F 1 "0.01uF" H 6650 4250 50  0000 L CNN
-F 2 "Capacitor_SMD:C_0603_1608Metric" H 6538 4150 50  0001 C CNN
+F 2 "RespiraWorks_Std:C_0603_1608Metric" H 6538 4150 50  0001 C CNN
 F 3 "~" H 6500 4300 50  0001 C CNN
 	1    6500 4300
@@
 F 0 "C?" H 6750 4050 50  0000 L CNN
 F 1 "0.01uF" H 6750 3950 50  0000 L CNN
-F 2 "Capacitor_SMD:C_0603_1608Metric" H 6638 3850 50  0001 C CNN
+F 2 "RespiraWorks_Std:C_0603_1608Metric" H 6638 3850 50  0001 C CNN
 F 3 "~" H 6600 4000 50  0001 C CNN
 	1    6600 4000
@@
 F 0 "R?" V 7350 4450 50  0000 C CNN
 F 1 "49.9" V 7250 4450 50  0000 C CNN
-F 2 "Resistor_SMD:R_1206_3216Metric" V 7080 4450 50  0001 C CNN
+F 2 "RespiraWorks_Std:R_1206_3216Metric" V 7080 4450 50  0001 C CNN
 F 3 "~" H 7150 4450 50  0001 C CNN
 	1    7150 4450
@@
 F 0 "R?" V 7350 3850 50  0000 C CNN
 F 1 "49.9" V 7250 3850 50  0000 C CNN
-F 2 "Resistor_SMD:R_1206_3216Metric" V 7080 3850 50  0001 C CNN
+F 2 "RespiraWorks_Std:R_1206_3216Metric" V 7080 3850 50  0001 C CNN
 F 3 "~" H 7150 3850 50  0001 C CNN
 	1    7150 3850
@@
 F 0 "R?" V 7350 4150 50  0000 C CNN
 F 1 "49.9" V 7250 4150 50  0000 C CNN
-F 2 "Resistor_SMD:R_1206_3216Metric" V 7080 4150 50  0001 C CNN
+F 2 "RespiraWorks_Std:R_1206_3216Metric" V 7080 4150 50  0001 C CNN
 F 3 "~" H 7150 4150 50  0001 C CNN
 	1    7150 4150
@@
 F 0 "Q?" V 6200 1650 50  0000 C CNN
 F 1 "CSD17304Q3" V 6100 1550 50  0000 C CNN
-F 2 "Package_SON:VSON-8_3.3x3.3mm_P0.65mm_NexFET" H 6000 1575 50  0001 L CIN
+F 2 "RespiraWorks_Std:VSON-8_3.3x3.3mm_P0.65mm_NexFET" H 6000 1575 50  0001 L CIN
 F 3 "https://www.ti.com/lit/ds/symlink/csd17304q3.pdf?ts=1608773956037" V 5800 1650 50  0001 L CNN
 	1    5800 1650
@@
 F 0 "C?" V 6200 2100 50  0000 L CNN
 F 1 "0.1uF" V 6300 2100 50  0000 L CNN
-F 2 "Capacitor_SMD:C_0603_1608Metric" H 6288 1700 50  0001 C CNN
+F 2 "RespiraWorks_Std:C_0603_1608Metric" H 6288 1700 50  0001 C CNN
 F 3 "~" H 6250 1850 50  0001 C CNN
 	1    6250 1850
@@
 F 0 "Q?" V 5700 1650 50  0000 C CNN
 F 1 "CSD17304Q3" V 5600 1550 50  0000 C CNN
-F 2 "Package_SON:VSON-8_3.3x3.3mm_P0.65mm_NexFET" H 5500 1575 50  0001 L CIN
+F 2 "RespiraWorks_Std:VSON-8_3.3x3.3mm_P0.65mm_NexFET" H 5500 1575 50  0001 L CIN
 F 3 "https://www.ti.com/lit/ds/symlink/csd17304q3.pdf?ts=1608773956037" V 5300 1650 50  0001 L CNN
 	1    5300 1650
@@
 F 0 "C?" H 10100 3750 50  0000 L CNN
 F 1 "0.1uF" H 10100 3650 50  0000 L CNN
-F 2 "Capacitor_SMD:C_0603_1608Metric" H 9988 3550 50  0001 C CNN
+F 2 "RespiraWorks_Std:C_0603_1608Metric" H 9988 3550 50  0001 C CNN
 F 3 "~" H 9950 3700 50  0001 C CNN
 	1    9950 3700
@@
 F 0 "C?" H 6650 4950 50  0000 L CNN
 F 1 "0.01uF" H 6650 4850 50  0000 L CNN
-F 2 "Capacitor_SMD:C_0603_1608Metric" H 6538 4750 50  0001 C CNN
+F 2 "RespiraWorks_Std:C_0603_1608Metric" H 6538 4750 50  0001 C CNN
 F 3 "~" H 6500 4900 50  0001 C CNN
 	1    6500 4900
@@
 F 0 "C?" H 6650 3450 50  0000 L CNN
 F 1 "0.47uF" H 6650 3350 50  0000 L CNN
-F 2 "Capacitor_SMD:C_0603_1608Metric" H 6538 3250 50  0001 C CNN
+F 2 "RespiraWorks_Std:C_0603_1608Metric" H 6538 3250 50  0001 C CNN
 F 3 "~" H 6500 3400 50  0001 C CNN
 	1    6500 3400
@@
 F 0 "C?" H 3400 5150 50  0000 L CNN
 F 1 "0.47uF" H 3400 5050 50  0000 L CNN
-F 2 "Capacitor_SMD:C_0603_1608Metric" H 3288 4950 50  0001 C CNN
+F 2 "RespiraWorks_Std:C_0603_1608Metric" H 3288 4950 50  0001 C CNN
 F 3 "~" H 3250 5100 50  0001 C CNN
 	1    3250 5100
@@
 F 0 "C?" H 4150 3950 50  0000 L CNN
 F 1 "0.47uF" H 4150 3850 50  0000 L CNN
-F 2 "Capacitor_SMD:C_0603_1608Metric" H 4038 3750 50  0001 C CNN
+F 2 "RespiraWorks_Std:C_0603_1608Metric" H 4038 3750 50  0001 C CNN
 F 3 "~" H 4000 3900 50  0001 C CNN
 	1    4000 3900
@@
 F 0 "C?" H 3950 5150 50  0000 L CNN
 F 1 "0.47uF" H 3950 5050 50  0000 L CNN
-F 2 "Capacitor_SMD:C_0603_1608Metric" H 3838 4950 50  0001 C CNN
+F 2 "RespiraWorks_Std:C_0603_1608Metric" H 3838 4950 50  0001 C CNN
 F 3 "~" H 3800 5100 50  0001 C CNN
 	1    3800 5100
@@
 F 0 "TH?" H 2947 4896 50  0000 L CNN
 F 1 "10k" H 2947 4805 50  0000 L CNN
-F 2 "Resistor_SMD:R_0603_1608Metric" H 2850 4900 50  0001 C CNN
+F 2 "RespiraWorks_Std:R_0603_1608Metric" H 2850 4900 50  0001 C CNN
 F 3 "~" H 2850 4900 50  0001 C CNN
 	1    2850 4850
@@
 F 0 "C?" H 4000 2500 50  0000 L CNN
 F 1 "0.01uF" H 4000 2400 50  0000 L CNN
-F 2 "Capacitor_SMD:C_0603_1608Metric" H 3888 2300 50  0001 C CNN
+F 2 "RespiraWorks_Std:C_0603_1608Metric" H 3888 2300 50  0001 C CNN
 F 3 "~" H 3850 2450 50  0001 C CNN
 	1    3850 2450

Commit message: swapping FETs for higher voltage and correcting return paths on batter balancer PR #951
Connections:
- net labels removed: GND
- wire segments 75 -> 81
Changed lines of the file:
@@
 Wire Wire Line
 	7050 3350 7400 3350
-Text Label 7400 3350 2    50   ~ 0
-BAT_N
-$Comp
-L power:GND #PWR?
-U 1 1 60422DE7
-P 3850 2600
-AR Path="/601A64F8/60422DE7" Ref="#PWR?"  Part="1"
-AR Path="/601A64F8/60567757/60422DE7" Ref="#PWR?"  Part="1"
-AR Path="/6023BF6A/60567757/60422DE7" Ref="#PWR?"  Part="1"
-F 0 "#PWR?" H 3850 2350 50  0001 C CNN
-F 1 "GND" H 3855 2427 50  0000 C CNN
-F 2 "" H 3850 2600 50  0001 C CNN
-F 3 "" H 3850 2600 50  0001 C CNN
-	1    3850 2600
-	1    0    0    -1
-$EndComp
 $Comp
 L Device:C C?
@@
 Text HLabel 4300 3550 0    50   Output ~ 0
 ALRT
-$Comp
-L power:GND #PWR?
-U 1 1 6046FA21
-P 4000 4050
-AR Path="/601A64F8/6046FA21" Ref="#PWR?"  Part="1"
-AR Path="/601A64F8/60567757/6046FA21" Ref="#PWR?"  Part="1"
-AR Path="/6023BF6A/60567757/6046FA21" Ref="#PWR?"  Part="1"
-F 0 "#PWR?" H 4000 3800 50  0001 C CNN
-F 1 "GND" H 4005 3877 50  0000 C CNN
-F 2 "" H 4000 4050 50  0001 C CNN
-F 3 "" H 4000 4050 50  0001 C CNN
-	1    4000 4050
-	1    0    0    -1
-$EndComp
 Text HLabel 1600 1550 0    50   Output ~ 0
 SYS_P
@@
 	4000 3750 3550 3750
 Connection ~ 4000 3750
-$Comp
-L power:GND #PWR?
-U 1 1 6029AB22
-P 3550 4050
-AR Path="/601A64F8/6029AB22" Ref="#PWR?"  Part="1"
-AR Path="/601A64F8/60567757/6029AB22" Ref="#PWR?"  Part="1"
-AR Path="/6023BF6A/60567757/6029AB22" Ref="#PWR?"  Part="1"
-F 0 "#PWR?" H 3550 3800 50  0001 C CNN
-F 1 "GND" H 3555 3877 50  0000 C CNN
-F 2 "" H 3550 4050 50  0001 C CNN
-F 3 "" H 3550 4050 50  0001 C CNN
-	1    3550 4050
-	1    0    0    -1
-$EndComp
+Text Label 7400 3350 2    50   ~ 0
+BAT_N
+Wire Wire Line
+	4000 4050 4000 4150
+Wire Wire Line
+	4000 4150 3550 4150
+Wire Wire Line
+	3550 4050 3550 4150
+Connection ~ 3550 4150
+Wire Wire Line
+	3550 4150 2850 4150
+Text Label 2850 4150 0    50   ~ 0
+BAT_N
+Wire Wire Line
+	3850 2600 3850 2700
+Wire Wire Line
+	3850 2700 2850 2700
+Text Label 2850 2700 0    50   ~ 0
+BAT_N
 $EndSCHEMATC

Commit message: Top-level beginnings, minor fixes
Started on top-level schematic blocks and connections
Started changing some net names to mixed-case-with-dash format
Fixed version number, added titles and version to all schematic sheets
Fixed incorrect SWO pin assignment in cycle controller
Added a few add'l annotations to battery sheets
Other:
- note added: "5mΩ:\n5-155 mV short-circuit threshold = 1-31 A\n2.5-77.5 mV medium over-discharge threshold = 0.5-15.5 A\n0-51.2 mV slow over-discharge threshold = 0-10.24 A\n0-38.75 mV charge threshold = 0-7.75 A"
- note added: "I2C address: 0b01100110 and 0b0001110"
- note added: "IC max balancing current: 100mA\nSet balancing current: 71mA\n= 4.2V cell voltage / (49.9Ω + 9Ω internal)"
- note added: "Max. recovery charge current =\nVin/(2K+10) = 8.5 mA @ 17 Vin"
- note removed: "IC max balancing current: 100mA\nSet balancing current: 71mA"
- moved on the sheet: C?, R?
