File: pcb/battery_balancer.sch (KiCad schematic (older format))
At the start: 28 parts

Commit message: CC-I2C, BOM
Added missing pull-ups on CC-SDA, CC-SCL
First pass at BOM consolidation
Parts:
- added R?: 0.01, RespiraWorks_Std:R_1206_3216Metric, symbol Device:R
- C? (x5): value 0.01uF -> 10nF
- C? (x2): value 0.1uF -> 100nF
- C? (x4): value 0.47uF -> 470nF
- R?: value 0.005 -> 0.01
Connections:
- wire segments 81 -> 85
Changed lines of the file:
@@
 AR Path="/6041384A/60567757/603D71EF" Ref="R?"  Part="1"
 F 0 "R?" H 6900 5250 50  0000 C CNN
-F 1 "0.005" H 6950 5150 50  0000 C CNN
+F 1 "0.01" H 6950 5150 50  0000 C CNN
 F 2 "RespiraWorks_Std:R_1206_3216Metric" V 6680 5200 50  0001 C CNN
 F 3 "~" H 6750 5200 50  0001 C CNN
@@
 AR Path="/6041384A/60567757/603D9107" Ref="C?"  Part="1"
 F 0 "C?" H 6750 4650 50  0000 L CNN
-F 1 "0.01uF" H 6750 4550 50  0000 L CNN
+F 1 "10nF" H 6750 4550 50  0000 L CNN
 F 2 "RespiraWorks_Std:C_0603_1608Metric" H 6638 4450 50  0001 C CNN
 F 3 "~" H 6600 4600 50  0001 C CNN
@@
 AR Path="/6041384A/60567757/603D9CD3" Ref="C?"  Part="1"
 F 0 "C?" H 6650 4350 50  0000 L CNN
-F 1 "0.01uF" H 6650 4250 50  0000 L CNN
+F 1 "10nF" H 6650 4250 50  0000 L CNN
 F 2 "RespiraWorks_Std:C_0603_1608Metric" H 6538 4150 50  0001 C CNN
 F 3 "~" H 6500 4300 50  0001 C CNN
@@
 AR Path="/6041384A/60567757/603D9EC2" Ref="C?"  Part="1"
 F 0 "C?" H 6750 4050 50  0000 L CNN
-F 1 "0.01uF" H 6750 3950 50  0000 L CNN
+F 1 "10nF" H 6750 3950 50  0000 L CNN
 F 2 "RespiraWorks_Std:C_0603_1608Metric" H 6638 3850 50  0001 C CNN
 F 3 "~" H 6600 4000 50  0001 C CNN
@@
 	6600 4750 6500 4750
 Wire Wire Line
-	6750 5350 6750 6100
+	6750 5350 6750 5450
 Wire Wire Line
 	6750 6100 1600 6100
@@
 AR Path="/6041384A/60567757/603E4953" Ref="C?"  Part="1"
 F 0 "C?" V 6200 2100 50  0000 L CNN
-F 1 "0.1uF" V 6300 2100 50  0000 L CNN
+F 1 "100nF" V 6300 2100 50  0000 L CNN
 F 2 "RespiraWorks_Std:C_0603_1608Metric" H 6288 1700 50  0001 C CNN
 F 3 "~" H 6250 1850 50  0001 C CNN
@@
 AR Path="/6041384A/60567757/603EA3B2" Ref="C?"  Part="1"
 F 0 "C?" H 10100 3750 50  0000 L CNN
-F 1 "0.1uF" H 10100 3650 50  0000 L CNN
+F 1 "100nF" H 10100 3650 50  0000 L CNN
 F 2 "RespiraWorks_Std:C_0603_1608Metric" H 9988 3550 50  0001 C CNN
 F 3 "~" H 9950 3700 50  0001 C CNN
@@
 AR Path="/6041384A/60567757/603EACF1" Ref="C?"  Part="1"
 F 0 "C?" H 6650 4950 50  0000 L CNN
-F 1 "0.01uF" H 6650 4850 50  0000 L CNN
+F 1 "10nF" H 6650 4850 50  0000 L CNN
 F 2 "RespiraWorks_Std:C_0603_1608Metric" H 6538 4750 50  0001 C CNN
 F 3 "~" H 6500 4900 50  0001 C CNN
@@
 AR Path="/6041384A/60567757/603F4DD5" Ref="C?"  Part="1"
 F 0 "C?" H 6650 3450 50  0000 L CNN
-F 1 "0.47uF" H 6650 3350 50  0000 L CNN
+F 1 "470nF" H 6650 3350 50  0000 L CNN
 F 2 "RespiraWorks_Std:C_0603_1608Metric" H 6538 3250 50  0001 C CNN
 F 3 "~" H 6500 3400 50  0001 C CNN
@@
 AR Path="/6041384A/60567757/60411B41" Ref="C?"  Part="1"
 F 0 "C?" H 3400 5150 50  0000 L CNN
-F 1 "0.47uF" H 3400 5050 50  0000 L CNN
+F 1 "470nF" H 3400 5050 50  0000 L CNN
 F 2 "RespiraWorks_Std:C_0603_1608Metric" H 3288 4950 50  0001 C CNN
 F 3 "~" H 3250 5100 50  0001 C CNN
@@
 AR Path="/6041384A/60567757/604128F9" Ref="C?"  Part="1"
 F 0 "C?" H 4150 3950 50  0000 L CNN
-F 1 "0.47uF" H 4150 3850 50  0000 L CNN
+F 1 "470nF" H 4150 3850 50  0000 L CNN
 F 2 "RespiraWorks_Std:C_0603_1608Metric" H 4038 3750 50  0001 C CNN
 F 3 "~" H 4000 3900 50  0001 C CNN
@@
 AR Path="/6041384A/60567757/60413618" Ref="C?"  Part="1"
 F 0 "C?" H 3950 5150 50  0000 L CNN
-F 1 "0.47uF" H 3950 5050 50  0000 L CNN
+F 1 "470nF" H 3950 5050 50  0000 L CNN
 F 2 "RespiraWorks_Std:C_0603_1608Metric" H 3838 4950 50  0001 C CNN
 F 3 "~" H 3800 5100 50  0001 C CNN
@@
 AR Path="/6041384A/60567757/60421F86" Ref="C?"  Part="1"
 F 0 "C?" H 2650 2500 50  0000 L CNN
-F 1 "0.01uF" H 2650 2400 50  0000 L CNN
+F 1 "10nF" H 2650 2400 50  0000 L CNN
 F 2 "RespiraWorks_Std:C_0603_1608Metric" H 2538 2300 50  0001 C CNN
 F 3 "~" H 2500 2450 50  0001 C CNN
@@
 	6300 5050 6500 5050
 Wire Wire Line
-	6750 5050 9950 5050
+	6750 5050 7200 5050
 Wire Wire Line
 	6400 1550 9950 1550
@@
 Wire Wire Line
 	3000 2700 4850 2700
-Text Notes 6850 5800 0    50   ~ 0
+Text Notes 6850 5900 0    50   ~ 0
 5mΩ:\n5-155 mV short-circuit threshold = 1-31 A\n2.5-77.5 mV medium over-discharge threshold = 0.5-15.5 A\n0-51.2 mV slow over-discharge threshold = 0-10.24 A\n0-38.75 mV charge threshold = 0-7.75 A
 Text Notes 4650 5850 0    50   ~ 0
 I2C address: 0b01100110 and 0b0001110
+$Comp
+L Device:R R?
+U 1 1 60552A00
+P 7200 5200
+AR Path="/601A64F8/60552A00" Ref="R?"  Part="1"
+AR Path="/601A64F8/60567144/60552A00" Ref="R?"  Part="1"
+AR Path="/601A64F8/60567757/60552A00" Ref="R?"  Part="1"
+AR Path="/6023BF6A/60567757/60552A00" Ref="R?"  Part="1"
+AR Path="/6041384A/60567757/60552A00" Ref="R?"  Part="1"
+F 0 "R?" H 7350 5250 50  0000 C CNN
+F 1 "0.01" H 7400 5150 50  0000 C CNN
+F 2 "RespiraWorks_Std:R_1206_3216Metric" V 7130 5200 50  0001 C CNN
+F 3 "~" H 7200 5200 50  0001 C CNN
+	1    7200 5200
+	1    0    0    -1
+$EndComp
+Connection ~ 7200 5050
+Wire Wire Line
+	7200 5050 9950 5050
+Wire Wire Line
+	6750 5450 7200 5450
+Wire Wire Line
+	7200 5450 7200 5350
+Connection ~ 6750 5450
+Wire Wire Line
+	6750 5450 6750 6100
 $EndSCHEMATC

Commit message: Edwin fixes
Assigned remaining footprints
Re-assigned UI computer pins to put RTS/CTS on hardware RTS/CTS, GUI-Buzzer on PWM pin
Incremented UI_ID on UI computer
Changed Oxygen-Level to Oxygen-FiO2
Removed STLink-controlled power switch on 5V-USB
Parts:
- J?: footprint (none) -> RespiraWorks_Std:JST_XH_B5B-XH-A_1x05_P2.50mm_Vertical
Changed lines of the file:
@@
 F 0 "J?" H 8900 4100 50  0000 R CNN
 F 1 "BAT-BALANCE JST XH 5-pin" H 9900 4200 50  0000 R CNN
-F 2 "" H 8700 4250 50  0001 C CNN
+F 2 "RespiraWorks_Std:JST_XH_B5B-XH-A_1x05_P2.50mm_Vertical" H 8700 4250 50  0001 C CNN
 F 3 "https://www.jst-mfg.com/product/pdf/eng/eXH.pdf" H 8700 4250 50  0001 C CNN
 F 4 "JST" H 8700 4250 50  0001 C CNN "Manufacturer"

Commit message: BOM, fixes
Finished assigning parts, footprints except generic resistors
Added series resistors for logic signals received by UI computer to protect against UI computer power-down
Added tolerance notes on main schem
Replaced PSol fuse with PTC
Enlarged PSol driver bypass resistors to 0 ohm
Changed PSol unpopulated current-limiting resistor to divider
Parts:
- C? (x5): Dielectric (none) -> NP0; Manufacturer (none) -> Murata; Manufacturer PN (none) -> GRM1885C1H103JA01D; Voltage (none) -> 50V
- C? (x2): Dielectric (none) -> X7R; Manufacturer (none) -> Kemet; Manufacturer PN (none) -> C0603C104K5RACTU; Voltage (none) -> 50V
- C? (x4): footprint RespiraWorks_Std:C_0603_1608Metric -> RespiraWorks_Std:C_0805_2012Metric; Dielectric (none) -> X7R; Manufacturer (none) -> Kemet; Manufacturer PN (none) -> C0805C474K5RACTU; Voltage (none) -> 50V
- Q? (x2): Manufacturer (none) -> Texas Instruments; Manufacturer PN (none) -> CSD17304Q3
- R? (x2): Manufacturer (none) -> Vishay; Manufacturer PN (none) -> WSL1206R0100FEA
- U?: Manufacturer PN MAX17320G20+ -> MAX17320G22+; Sourcing Notes (none) -> Alt. MAX17320G20+
Changed lines of the file:
@@
 F 3 "https://datasheets.maximintegrated.com/en/ds/MAX17320.pdf" H 8300 4850 50  0001 C CNN
 F 4 "Maxim IC" H 5600 3800 50  0000 C CNN "Manufacturer"
-F 5 "MAX17320G20+" H 5600 3700 50  0000 C CNN "Manufacturer PN"
+F 5 "MAX17320G22+" H 5600 3700 50  0000 C CNN "Manufacturer PN"
+F 6 "Alt. MAX17320G20+" H 5600 3800 50  0001 C CNN "Sourcing Notes"
 	1    5600 3800
 	1    0    0    -1
@@
 F 2 "RespiraWorks_Std:R_1206_3216Metric" V 6680 5200 50  0001 C CNN
 F 3 "~" H 6750 5200 50  0001 C CNN
+F 4 "Vishay" H 6750 5200 50  0001 C CNN "Manufacturer"
+F 5 "WSL1206R0100FEA" H 6750 5200 50  0001 C CNN "Manufacturer PN"
 	1    6750 5200
 	1    0    0    -1
@@
 F 2 "RespiraWorks_Std:C_0603_1608Metric" H 6638 4450 50  0001 C CNN
 F 3 "~" H 6600 4600 50  0001 C CNN
+F 4 "NP0" H 6600 4600 50  0001 C CNN "Dielectric"
+F 5 "Murata" H 6600 4600 50  0001 C CNN "Manufacturer"
+F 6 "GRM1885C1H103JA01D" H 6600 4600 50  0001 C CNN "Manufacturer PN"
+F 7 "50V" H 6600 4600 50  0001 C CNN "Voltage"
 	1    6600 4600
 	1    0    0    -1
@@
 F 2 "RespiraWorks_Std:C_0603_1608Metric" H 6538 4150 50  0001 C CNN
 F 3 "~" H 6500 4300 50  0001 C CNN
+F 4 "NP0" H 6500 4300 50  0001 C CNN "Dielectric"
+F 5 "Murata" H 6500 4300 50  0001 C CNN "Manufacturer"
+F 6 "GRM1885C1H103JA01D" H 6500 4300 50  0001 C CNN "Manufacturer PN"
+F 7 "50V" H 6500 4300 50  0001 C CNN "Voltage"
 	1    6500 4300
 	1    0    0    -1
@@
 F 2 "RespiraWorks_Std:C_0603_1608Metric" H 6638 3850 50  0001 C CNN
 F 3 "~" H 6600 4000 50  0001 C CNN
+F 4 "NP0" H 6600 4000 50  0001 C CNN "Dielectric"
+F 5 "Murata" H 6600 4000 50  0001 C CNN "Manufacturer"
+F 6 "GRM1885C1H103JA01D" H 6600 4000 50  0001 C CNN "Manufacturer PN"
+F 7 "50V" H 6600 4000 50  0001 C CNN "Voltage"
 	1    6600 4000
 	1    0    0    -1
@@
 F 2 "RespiraWorks_Std:VSON-8_3.3x3.3mm_P0.65mm_NexFET" H 6000 1575 50  0001 L CIN
 F 3 "https://www.ti.com/lit/ds/symlink/csd17304q3.pdf?ts=1608773956037" V 5800 1650 50  0001 L CNN
+F 4 "Texas Instruments" H 5800 1650 50  0001 C CNN "Manufacturer"
+F 5 "CSD17304Q3" H 5800 1650 50  0001 C CNN "Manufacturer PN"
 	1    5800 1650
 	0    -1   -1   0
@@
 F 2 "RespiraWorks_Std:C_0603_1608Metric" H 6288 1700 50  0001 C CNN
 F 3 "~" H 6250 1850 50  0001 C CNN
+F 4 "X7R" H 6250 1850 50  0001 C CNN "Dielectric"
+F 5 "Kemet" H 6250 1850 50  0001 C CNN "Manufacturer"
+F 6 "C0603C104K5RACTU" H 6250 1850 50  0001 C CNN "Manufacturer PN"
+F 7 "50V" H 6250 1850 50  0001 C CNN "Voltage"
 	1    6250 1850
 	0    1    1    0
@@
 F 2 "RespiraWorks_Std:VSON-8_3.3x3.3mm_P0.65mm_NexFET" H 5500 1575 50  0001 L CIN
 F 3 "https://www.ti.com/lit/ds/symlink/csd17304q3.pdf?ts=1608773956037" V 5300 1650 50  0001 L CNN
+F 4 "Texas Instruments" H 5300 1650 50  0001 C CNN "Manufacturer"
+F 5 "CSD17304Q3" H 5300 1650 50  0001 C CNN "Manufacturer PN"
 	1    5300 1650
 	0    1    -1   0
@@
 F 2 "RespiraWorks_Std:C_0603_1608Metric" H 9988 3550 50  0001 C CNN
 F 3 "~" H 9950 3700 50  0001 C CNN
+F 4 "X7R" H 9950 3700 50  0001 C CNN "Dielectric"
+F 5 "Kemet" H 9950 3700 50  0001 C CNN "Manufacturer"
+F 6 "C0603C104K5RACTU" H 9950 3700 50  0001 C CNN "Manufacturer PN"
+F 7 "50V" H 9950 3700 50  0001 C CNN "Voltage"
 	1    9950 3700
 	1    0    0    -1
@@
 F 2 "RespiraWorks_Std:C_0603_1608Metric" H 6538 4750 50  0001 C CNN
 F 3 "~" H 6500 4900 50  0001 C CNN
+F 4 "NP0" H 6500 4900 50  0001 C CNN "Dielectric"
+F 5 "Murata" H 6500 4900 50  0001 C CNN "Manufacturer"
+F 6 "GRM1885C1H103JA01D" H 6500 4900 50  0001 C CNN "Manufacturer PN"
+F 7 "50V" H 6500 4900 50  0001 C CNN "Voltage"
 	1    6500 4900
 	1    0    0    -1
@@
 F 0 "C?" H 6650 3450 50  0000 L CNN
 F 1 "470nF" H 6650 3350 50  0000 L CNN
-F 2 "RespiraWorks_Std:C_0603_1608Metric" H 6538 3250 50  0001 C CNN
+F 2 "RespiraWorks_Std:C_0805_2012Metric" H 6538 3250 50  0001 C CNN
 F 3 "~" H 6500 3400 50  0001 C CNN
+F 4 "X7R" H 6500 3400 50  0001 C CNN "Dielectric"
+F 5 "50V" H 6500 3400 50  0001 C CNN "Voltage"
+F 6 "Kemet" H 6500 3400 50  0001 C CNN "Manufacturer"
+F 7 "C0805C474K5RACTU" H 6500 3400 50  0001 C CNN "Manufacturer PN"
 	1    6500 3400
 	1    0    0    -1
@@
 F 0 "C?" H 3400 5150 50  0000 L CNN
 F 1 "470nF" H 3400 5050 50  0000 L CNN
-F 2 "RespiraWorks_Std:C_0603_1608Metric" H 3288 4950 50  0001 C CNN
+F 2 "RespiraWorks_Std:C_0805_2012Metric" H 3288 4950 50  0001 C CNN
 F 3 "~" H 3250 5100 50  0001 C CNN
+F 4 "X7R" H 3250 5100 50  0001 C CNN "Dielectric"
+F 5 "50V" H 3250 5100 50  0001 C CNN "Voltage"
+F 6 "Kemet" H 3250 5100 50  0001 C CNN "Manufacturer"
+F 7 "C0805C474K5RACTU" H 3250 5100 50  0001 C CNN "Manufacturer PN"
 	1    3250 5100
 	1    0    0    -1
@@
 F 0 "C?" H 4150 3950 50  0000 L CNN
 F 1 "470nF" H 4150 3850 50  0000 L CNN
-F 2 "RespiraWorks_Std:C_0603_1608Metric" H 4038 3750 50  0001 C CNN
+F 2 "RespiraWorks_Std:C_0805_2012Metric" H 4038 3750 50  0001 C CNN
 F 3 "~" H 4000 3900 50  0001 C CNN
+F 4 "X7R" H 4000 3900 50  0001 C CNN "Dielectric"
+F 5 "50V" H 4000 3900 50  0001 C CNN "Voltage"
+F 6 "Kemet" H 4000 3900 50  0001 C CNN "Manufacturer"
+F 7 "C0805C474K5RACTU" H 4000 3900 50  0001 C CNN "Manufacturer PN"
 	1    4000 3900
 	1    0    0    -1
@@
 F 0 "C?" H 3950 5150 50  0000 L CNN
 F 1 "470nF" H 3950 5050 50  0000 L CNN
-F 2 "RespiraWorks_Std:C_0603_1608Metric" H 3838 4950 50  0001 C CNN
+F 2 "RespiraWorks_Std:C_0805_2012Metric" H 3838 4950 50  0001 C CNN
 F 3 "~" H 3800 5100 50  0001 C CNN
+F 4 "X7R" H 3800 5100 50  0001 C CNN "Dielectric"
+F 5 "50V" H 3800 5100 50  0001 C CNN "Voltage"
+F 6 "Kemet" H 3800 5100 50  0001 C CNN "Manufacturer"
+F 7 "C0805C474K5RACTU" H 3800 5100 50  0001 C CNN "Manufacturer PN"
 	1    3800 5100
 	1    0    0    -1
@@
 F 2 "RespiraWorks_Std:C_0603_1608Metric" H 2538 2300 50  0001 C CNN
 F 3 "~" H 2500 2450 50  0001 C CNN
+F 4 "NP0" H 2500 2450 50  0001 C CNN "Dielectric"
+F 5 "Murata" H 2500 2450 50  0001 C CNN "Manufacturer"
+F 6 "GRM1885C1H103JA01D" H 2500 2450 50  0001 C CNN "Manufacturer PN"
+F 7 "50V" H 2500 2450 50  0001 C CNN "Voltage"
 	1    2500 2450
 	1    0    0    -1
@@
 F 2 "RespiraWorks_Std:R_1206_3216Metric" V 7130 5200 50  0001 C CNN
 F 3 "~" H 7200 5200 50  0001 C CNN
+F 4 "Vishay" H 7200 5200 50  0001 C CNN "Manufacturer"
+F 5 "WSL1206R0100FEA" H 7200 5200 50  0001 C CNN "Manufacturer PN"
 	1    7200 5200
 	1    0    0    -1

Commit message: Stephanie fixes, net names
Removed duplicate global I2C pull-ups
Added missing BMP280 pin 7
Correcting pin names etc. on LM4120 voltage reference
Finished standardizing net names
Connections:
- net labels added: Alrt, Bat-N, Bat-P, Sys-N, Sys-P
- net labels removed: ALRT, BAT_N, BAT_P, SYS_N, SYS_P
Changed lines of the file:
@@
 Wire Wire Line
 	4850 3750 4000 3750
-Text Label 7650 5050 0    50   ~ 0
-BAT_N
 Text Label 4050 5550 0    50   ~ 0
-BAT_N
+Bat-N
 Connection ~ 3250 5550
 Wire Wire Line
@@
 SDA
 Text HLabel 4300 3550 0    50   Output ~ 0
-ALRT
+Alrt
 Text HLabel 1600 1550 0    50   Output ~ 0
-SYS_P
+Sys-P
 Text HLabel 1600 6100 0    50   Output ~ 0
-SYS_N
+Sys-N
 Wire Wire Line
 	8300 3850 8300 4050
@@
 	8300 4050 8500 4050
 Text HLabel 10050 5050 2    50   Input ~ 0
-BAT_N
+Bat-N
 Text HLabel 10050 1550 2    50   Input ~ 0
-BAT_P
+Bat-P
 Wire Wire Line
 	6100 1850 5800 1850
@@
 Connection ~ 4000 3750
 Text Label 7400 3350 2    50   ~ 0
-BAT_N
+Bat-N
 Wire Wire Line
 	4000 4050 4000 4150
@@
 	3550 4150 2850 4150
 Text Label 2850 4150 0    50   ~ 0
-BAT_N
+Bat-N
 Wire Wire Line
 	2500 2600 2500 2700
@@
 	2500 2700 2100 2700
 Text Label 2100 2700 0    50   ~ 0
-BAT_N
+Bat-N
 Text Notes 3700 2150 0    50   ~ 0
 Max. recovery charge current =\nVin/(2K+10) = 8.5 mA @ 17 Vin

Commit message: updated FETs to alternates on battery balancer
Parts:
- Q? (x2): value CSD17304Q3 -> BSZ019N03LSATMA1; footprint RespiraWorks_Std:VSON-8_3.3x3.3mm_P0.65mm_NexFET -> RespiraWorks:VSON-8-SGD_3.3x3.3mm_P0.65mm_NexFET; symbol RespiraWorks_Std:CSD17304Q3 -> RespiraWorks_Std:Q_NMOS_SGD; Manufacturer Texas Instruments -> Infineon; Manufacturer PN CSD17304Q3 -> BSZ019N03LSATMA1
Changed lines of the file:
@@
 Connection ~ 6750 5050
-$Comp
-L RespiraWorks_Std:CSD17304Q3 Q?
-U 1 1 603E4945
-P 5800 1650
-AR Path="/601A64F8/603E4945" Ref="Q?"  Part="1"
-AR Path="/601A64F8/60567144/603E4945" Ref="Q?"  Part="1"
-AR Path="/601A64F8/60567757/603E4945" Ref="Q?"  Part="1"
-AR Path="/6023BF6A/60567757/603E4945" Ref="Q?"  Part="1"
-AR Path="/6041384A/60567757/603E4945" Ref="Q?"  Part="1"
-F 0 "Q?" V 6200 1650 50  0000 C CNN
-F 1 "CSD17304Q3" V 6100 1550 50  0000 C CNN
-F 2 "RespiraWorks_Std:VSON-8_3.3x3.3mm_P0.65mm_NexFET" H 6000 1575 50  0001 L CIN
-F 3 "https://www.ti.com/lit/ds/symlink/csd17304q3.pdf?ts=1608773956037" V 5800 1650 50  0001 L CNN
-F 4 "Texas Instruments" H 5800 1650 50  0001 C CNN "Manufacturer"
-F 5 "CSD17304Q3" H 5800 1650 50  0001 C CNN "Manufacturer PN"
-	1    5800 1650
-	0    -1   -1   0
-$EndComp
 $Comp
 L Device:C C?
@@
 $EndComp
 $Comp
-L RespiraWorks_Std:CSD17304Q3 Q?
+L RespiraWorks_Std:Q_NMOS_SGD Q?
 U 1 1 603E494C
 P 5300 1650
@@
 AR Path="/6023BF6A/60567757/603E494C" Ref="Q?"  Part="1"
 AR Path="/6041384A/60567757/603E494C" Ref="Q?"  Part="1"
-F 0 "Q?" V 5700 1650 50  0000 C CNN
-F 1 "CSD17304Q3" V 5600 1550 50  0000 C CNN
-F 2 "RespiraWorks_Std:VSON-8_3.3x3.3mm_P0.65mm_NexFET" H 5500 1575 50  0001 L CIN
-F 3 "https://www.ti.com/lit/ds/symlink/csd17304q3.pdf?ts=1608773956037" V 5300 1650 50  0001 L CNN
-F 4 "Texas Instruments" H 5300 1650 50  0001 C CNN "Manufacturer"
-F 5 "CSD17304Q3" H 5300 1650 50  0001 C CNN "Manufacturer PN"
+F 0 "Q?" V 5850 1650 50  0000 C CNN
+F 1 "BSZ019N03LSATMA1" V 5750 1650 50  0000 C CNN
+F 2 "RespiraWorks:VSON-8-SGD_3.3x3.3mm_P0.65mm_NexFET" H 5500 1575 50  0001 L CIN
+F 3 "https://www.infineon.com/dgdl/BSZ019N03LS_Rev+2.1.pdf?folderId=db3a304326dfb1300126fb3bec803f1a&fileId=db3a304326dfb1300126fb7ddf173f4e" V 5300 1650 50  0001 L CNN
+F 4 "Infineon" H 5300 1650 50  0001 C CNN "Manufacturer"
+F 5 "BSZ019N03LSATMA1" H 5300 1650 50  0001 C CNN "Manufacturer PN"
 	1    5300 1650
 	0    1    -1   0
@@
 Wire Wire Line
 	6750 5450 6750 6100
+$Comp
+L RespiraWorks_Std:Q_NMOS_SGD Q?
+U 1 1 603E4945
+P 5800 1650
+AR Path="/601A64F8/603E4945" Ref="Q?"  Part="1"
+AR Path="/601A64F8/60567144/603E4945" Ref="Q?"  Part="1"
+AR Path="/601A64F8/60567757/603E4945" Ref="Q?"  Part="1"
+AR Path="/6023BF6A/60567757/603E4945" Ref="Q?"  Part="1"
+AR Path="/6041384A/60567757/603E4945" Ref="Q?"  Part="1"
+F 0 "Q?" V 6200 1650 50  0000 C CNN
+F 1 "BSZ019N03LSATMA1" V 6100 1550 50  0000 C CNN
+F 2 "RespiraWorks:VSON-8-SGD_3.3x3.3mm_P0.65mm_NexFET" H 6000 1575 50  0001 L CIN
+F 3 "https://www.infineon.com/dgdl/BSZ019N03LS_Rev+2.1.pdf?folderId=db3a304326dfb1300126fb3bec803f1a&fileId=db3a304326dfb1300126fb7ddf173f4e" V 5800 1650 50  0001 L CNN
+F 4 "Infineon" H 5800 1650 50  0001 C CNN "Manufacturer"
+F 5 "BSZ019N03LSATMA1" H 5800 1650 50  0001 C CNN "Manufacturer PN"
+	1    5800 1650
+	0    -1   -1   0
+$EndComp
 $EndSCHEMATC

Commit message: PCB Rev A Floorplanning (#1079)
* annotate schematics

* generate netlist

* define board edges at 150x300mm

* add parts to board (some pending errors)

* fix schem-pcb footprint mismatches and push to PCB

* preliminary packing at 155x300mm board size - marginal

* PCB floor planning

* added fan power and swapped solenoid/touchscreen power to vertical connectors
Parts:
- gave numbers to parts that had none: 29
