File: pcb/battery_controller.sch (KiCad schematic (older format))
At the start: 6 parts

Commit message: added battery balancer/fuel gauge
Parts:
- D?: value D_Zener -> 24V
Connections:
- net labels added: BAT_ALRT
- wire segments 24 -> 32
Other:
- moved on the sheet: C?, F?

Commit message: clean up, add part numbers to parts, added design comments
Parts:
- removed F?: Fuse 10A, symbol Device:Fuse
- added F?: Fuse 10A, symbol Device:Fuse
- D?: value 24V -> 20V; footprint (none) -> Diode_SMD:D_SMC; Manufacturer (none) -> Diodes Inc.; Manufacturer PN (none) -> SMBJ20AQ-13-F
- F?: Manufacturer (none) -> Littelfuse; Manufacturer PN (none) -> 0154010.DR
Changed lines of the file:
@@
 AR Path="/601A64F8/605C3588" Ref="D?"  Part="1"
 AR Path="/601A64F8/60567144/605C3588" Ref="D?"  Part="1"
-F 0 "D?" V 2400 3600 50  0000 L CNN
-F 1 "24V" V 2500 3600 50  0000 L CNN
-F 2 "" H 2400 3450 50  0001 C CNN
-F 3 "~" H 2400 3450 50  0001 C CNN
+F 0 "D?" V 2350 3550 50  0000 L CNN
+F 1 "20V" V 2450 3550 50  0000 L CNN
+F 2 "Diode_SMD:D_SMC" H 2400 3450 50  0001 C CNN
+F 3 "https://www.diodes.com/assets/Datasheets/ds40740.pdf" H 2400 3450 50  0001 C CNN
+F 4 "Diodes Inc." V 2400 3450 50  0001 C CNN "Manufacturer"
+F 5 "SMBJ20AQ-13-F" V 2550 3800 50  0000 C CNN "Manufacturer PN"
 	1    2400 3450
 	0    1    1    0
@@
 F 1 "Fuse 10A" V 3094 3300 50  0000 C CNN
 F 2 "" V 3130 3300 50  0001 C CNN
-F 3 "~" H 3200 3300 50  0001 C CNN
+F 3 "https://www.littelfuse.com/~/media/electronics/datasheets/fuses/littelfuse_fuse_154_154t_154l_154tl_datasheet.pdf.pdf" H 3200 3300 50  0001 C CNN
+F 4 "Littelfuse" V 3200 3300 50  0001 C CNN "Manufacturer"
+F 5 "0154010.DR" V 3300 3300 50  0000 C CNN "Manufacturer PN"
 	1    3200 3300
 	0    1    1    0
@@
 $Comp
 L Device:Fuse F?
-U 1 1 603A4540
+U 1 1 602914E1
 P 8200 4850
-F 0 "F?" V 8003 4850 50  0000 C CNN
-F 1 "Fuse 10A" V 8094 4850 50  0000 C CNN
+F 0 "F?" V 7900 4850 50  0000 C CNN
+F 1 "Fuse 10A" V 8000 4850 50  0000 C CNN
 F 2 "" V 8130 4850 50  0001 C CNN
-F 3 "~" H 8200 4850 50  0001 C CNN
+F 3 "https://www.littelfuse.com/~/media/electronics/datasheets/fuses/littelfuse_fuse_154_154t_154l_154tl_datasheet.pdf.pdf" H 8200 4850 50  0001 C CNN
+F 4 "Littelfuse" V 8200 4850 50  0001 C CNN "Manufacturer"
+F 5 "0154010.DR" V 8100 4850 50  0000 C CNN "Manufacturer PN"
 	1    8200 4850
 	0    1    1    0

Commit message: WIP implement comments from review
Parts:
- added C?: 33uF, symbol Device:CP
- F? (x2): footprint (none) -> RespiraWorks:Fuseholder_Littelfuse_OMNI-BLOK-154
Connections:
- net labels added: SWITCHED_VLINK
- wire segments 32 -> 36
Other:
- note added: "12.0-16.8V"
Changed lines of the file:
@@
 F3 "SDA" B L 3950 3800 50
 F4 "VLOGIC" I L 3950 3600 50
-F5 "PSYS" I R 5150 3500 50
-F6 "IBAT" I R 5150 3600 50
-F7 "IADPT" I R 5150 3700 50
-F8 "ACOK" I R 5150 3800 50
-F9 "VIN_ADP" I L 3950 3300 50
-F10 "VLINK" I R 5150 3300 50
-F11 "PACK_P" B R 5150 3400 50
+F5 "VIN_ADP" I L 3950 3300 50
+F6 "PACK_P" B R 5150 3400 50
+F7 "VLINK" O R 5150 3300 50
+F8 "PSYS" O R 5150 3500 50
+F9 "IBAT" O R 5150 3600 50
+F10 "IADPT" O R 5150 3700 50
+F11 "ACOK" O R 5150 3800 50
 $EndSheet
 $Sheet
@@
 L Connector:Conn_01x04_Male J?
 U 1 1 605A607B
-P 2000 3300
-F 0 "J?" H 2250 2750 50  0000 R CNN
-F 1 "MegaFit 2x2" H 2250 2850 50  0000 R CNN
-F 2 "RespiraWorks_Std:Molex_Mega-Fit_76829-0104_2x02_P5.70mm_Vertical" H 2000 3300 50  0001 C CNN
-F 3 "~" H 2000 3300 50  0001 C CNN
-F 4 "Molex" H 2000 3300 50  0001 C CNN "Manufacturer"
-F 5 "768290104" H 2250 2950 50  0000 R CNN "Manufacturer P/N"
-	1    2000 3300
+P 1250 3300
+F 0 "J?" H 1500 2750 50  0000 R CNN
+F 1 "MegaFit 2x2" H 1500 2850 50  0000 R CNN
+F 2 "RespiraWorks_Std:Molex_Mega-Fit_76829-0104_2x02_P5.70mm_Vertical" H 1250 3300 50  0001 C CNN
+F 3 "~" H 1250 3300 50  0001 C CNN
+F 4 "Molex" H 1250 3300 50  0001 C CNN "Manufacturer"
+F 5 "768290104" H 1500 2950 50  0000 R CNN "Manufacturer P/N"
+	1    1250 3300
 	1    0    0    1
 $EndComp
@@
 AR Path="/601A64F8/605C357B" Ref="J?"  Part="1"
 AR Path="/601A64F8/60567144/605C357B" Ref="J?"  Part="1"
+AR Path="/6023BF6A/605C357B" Ref="J?"  Part="1"
 F 0 "J?" H 8800 5050 50  0000 R CNN
 F 1 "MegaFit 2x1" H 8800 5150 50  0000 R CNN
@@
 L power:GND #PWR?
 U 1 1 605C3581
-P 2200 3400
+P 1450 3400
 AR Path="/601A64F8/605C3581" Ref="#PWR?"  Part="1"
 AR Path="/601A64F8/60567144/605C3581" Ref="#PWR?"  Part="1"
-F 0 "#PWR?" H 2200 3150 50  0001 C CNN
-F 1 "GND" H 2205 3227 50  0000 C CNN
-F 2 "" H 2200 3400 50  0001 C CNN
-F 3 "" H 2200 3400 50  0001 C CNN
-	1    2200 3400
+AR Path="/6023BF6A/605C3581" Ref="#PWR?"  Part="1"
+F 0 "#PWR?" H 1450 3150 50  0001 C CNN
+F 1 "GND" H 1455 3227 50  0000 C CNN
+F 2 "" H 1450 3400 50  0001 C CNN
+F 3 "" H 1450 3400 50  0001 C CNN
+	1    1450 3400
 	1    0    0    -1
 $EndComp
@@
 L Device:D_Zener D?
 U 1 1 605C3588
-P 2400 3450
+P 1650 3450
 AR Path="/601A64F8/605C3588" Ref="D?"  Part="1"
 AR Path="/601A64F8/60567144/605C3588" Ref="D?"  Part="1"
-F 0 "D?" V 2350 3550 50  0000 L CNN
-F 1 "20V" V 2450 3550 50  0000 L CNN
-F 2 "Diode_SMD:D_SMC" H 2400 3450 50  0001 C CNN
-F 3 "https://www.diodes.com/assets/Datasheets/ds40740.pdf" H 2400 3450 50  0001 C CNN
-F 4 "Diodes Inc." V 2400 3450 50  0001 C CNN "Manufacturer"
-F 5 "SMBJ20AQ-13-F" V 2550 3800 50  0000 C CNN "Manufacturer PN"
-	1    2400 3450
+AR Path="/6023BF6A/605C3588" Ref="D?"  Part="1"
+F 0 "D?" V 1600 3550 50  0000 L CNN
+F 1 "20V" V 1700 3550 50  0000 L CNN
+F 2 "Diode_SMD:D_SMC" H 1650 3450 50  0001 C CNN
+F 3 "https://www.diodes.com/assets/Datasheets/ds40740.pdf" H 1650 3450 50  0001 C CNN
+F 4 "Diodes Inc." V 1650 3450 50  0001 C CNN "Manufacturer"
+F 5 "SMBJ20AQ-13-F" V 1800 3800 50  0000 C CNN "Manufacturer PN"
+	1    1650 3450
 	0    1    1    0
 $EndComp
@@
 L power:GND #PWR?
 U 1 1 605C358F
-P 2400 3600
+P 1650 3600
 AR Path="/601A64F8/605C358F" Ref="#PWR?"  Part="1"
 AR Path="/601A64F8/60567144/605C358F" Ref="#PWR?"  Part="1"
-F 0 "#PWR?" H 2400 3350 50  0001 C CNN
-F 1 "GND" H 2405 3427 50  0000 C CNN
-F 2 "" H 2400 3600 50  0001 C CNN
-F 3 "" H 2400 3600 50  0001 C CNN
-	1    2400 3600
-	1    0    0    -1
-$EndComp
-Connection ~ 2400 3300
+AR Path="/6023BF6A/605C358F" Ref="#PWR?"  Part="1"
+F 0 "#PWR?" H 1650 3350 50  0001 C CNN
+F 1 "GND" H 1655 3427 50  0000 C CNN
+F 2 "" H 1650 3600 50  0001 C CNN
+F 3 "" H 1650 3600 50  0001 C CNN
+	1    1650 3600
+	1    0    0    -1
+$EndComp
+Connection ~ 1650 3300
 Text Label 3600 3300 0    50   ~ 0
 VIN_ADP
 Wire Wire Line
-	2200 3200 2800 3200
-Wire Wire Line
-	2800 3100 2200 3100
-Text Label 2800 3100 2    50   ~ 0
+	1450 3200 2050 3200
+Wire Wire Line
+	2050 3100 1450 3100
+Text Label 2050 3100 2    50   ~ 0
 POWER_SW_P
-Text Label 2800 3200 2    50   ~ 0
+Text Label 2050 3200 2    50   ~ 0
 POWER_SW_N
 Wire Wire Line
-	2200 3300 2400 3300
-Wire Wire Line
-	6600 3300 7200 3300
+	1450 3300 1650 3300
+Wire Wire Line
+	6600 3300 7150 3300
 Text Label 6600 3300 0    50   ~ 0
 POWER_SW_N
@@
 F 0 "F?" V 3003 3300 50  0000 C CNN
 F 1 "Fuse 10A" V 3094 3300 50  0000 C CNN
-F 2 "" V 3130 3300 50  0001 C CNN
+F 2 "RespiraWorks:Fuseholder_Littelfuse_OMNI-BLOK-154" V 3130 3300 50  0001 C CNN
 F 3 "https://www.littelfuse.com/~/media/electronics/datasheets/fuses/littelfuse_fuse_154_154t_154l_154tl_datasheet.pdf.pdf" H 3200 3300 50  0001 C CNN
 F 4 "Littelfuse" V 3200 3300 50  0001 C CNN "Manufacturer"
@@
 $EndComp
 Wire Wire Line
-	2400 3300 3050 3300
-Wire Wire Line
 	3350 3300 3950 3300
 Wire Wire Line
@@
 AR Path="/601A64F8/6047EA81" Ref="#PWR?"  Part="1"
 AR Path="/601A64F8/60567144/6047EA81" Ref="#PWR?"  Part="1"
+AR Path="/6023BF6A/6047EA81" Ref="#PWR?"  Part="1"
 F 0 "#PWR?" H 6150 4950 50  0001 C CNN
 F 1 "GND" H 6155 5027 50  0000 C CNN
@@
 F 0 "F?" V 7900 4850 50  0000 C CNN
 F 1 "Fuse 10A" V 8000 4850 50  0000 C CNN
-F 2 "" V 8130 4850 50  0001 C CNN
+F 2 "RespiraWorks:Fuseholder_Littelfuse_OMNI-BLOK-154" V 8130 4850 50  0001 C CNN
 F 3 "https://www.littelfuse.com/~/media/electronics/datasheets/fuses/littelfuse_fuse_154_154t_154l_154tl_datasheet.pdf.pdf" H 8200 4850 50  0001 C CNN
 F 4 "Littelfuse" V 8200 4850 50  0001 C CNN "Manufacturer"
@@
 	0    1    1    0
 $EndComp
+Wire Wire Line
+	7150 3300 7150 3000
+Wire Wire Line
+	7150 3000 8150 3000
+Connection ~ 7150 3300
+Wire Wire Line
+	7150 3300 7200 3300
+Text HLabel 8150 3000 2    50   Output ~ 0
+SWITCHED_VLINK
+Text Notes 7600 3000 0    50   ~ 0
+12.0-16.8V
+Wire Wire Line
+	1650 3300 2550 3300
+$Comp
+L Device:CP C?
+U 1 1 6026FB4D
+P 2550 3450
+AR Path="/601A64F8/6026FB4D" Ref="C?"  Part="1"
+AR Path="/601A64F8/60567144/6026FB4D" Ref="C?"  Part="1"
+AR Path="/6023BF6A/60567144/6026FB4D" Ref="C?"  Part="1"
+AR Path="/6023BF6A/6026FB4D" Ref="C?"  Part="1"
+F 0 "C?" H 2700 3450 50  0000 L CNN
+F 1 "33uF" H 2700 3350 50  0000 L CNN
+F 2 "" H 2588 3300 50  0001 C CNN
+F 3 "~" H 2550 3450 50  0001 C CNN
+F 4 "50V" H 2700 3250 50  0000 L CNN "Voltage"
+	1    2550 3450
+	1    0    0    -1
+$EndComp
+$Comp
+L power:GND #PWR?
+U 1 1 602707F0
+P 2550 3600
+AR Path="/601A64F8/602707F0" Ref="#PWR?"  Part="1"
+AR Path="/601A64F8/60567144/602707F0" Ref="#PWR?"  Part="1"
+AR Path="/6023BF6A/602707F0" Ref="#PWR?"  Part="1"
+F 0 "#PWR?" H 2550 3350 50  0001 C CNN
+F 1 "GND" H 2555 3427 50  0000 C CNN
+F 2 "" H 2550 3600 50  0001 C CNN
+F 3 "" H 2550 3600 50  0001 C CNN
+	1    2550 3600
+	1    0    0    -1
+$EndComp
+Connection ~ 2550 3300
+Wire Wire Line
+	2550 3300 3050 3300
 $EndSCHEMATC

Commit message: WIP implement PR comments
Parts:
- J?: value MegaFit 2x2 -> POWER-ENTRY MegaFit 2x2; symbol Connector:Conn_01x04_Male -> Connector_Generic:Conn_01x04
- J?: value MegaFit 2x1 -> BAT-PWR MegaFit 2x1; symbol Connector:Conn_01x02_Male -> Connector_Generic:Conn_01x02
Other:
- moved on the sheet: C?, F?

Commit message: updated footprints to reference to RW library
Parts:
- C?: footprint (none) -> RespiraWorks_Std:CP_Elec_6.3x7.7; Manufacturer (none) -> Panasonic; Manufacturer PN (none) -> EEE-FK1H330XP
- C?: footprint Capacitor_SMD:C_0603_1608Metric -> RespiraWorks_Std:C_0603_1608Metric
- D?: footprint Diode_SMD:D_SMC -> RespiraWorks_Std:D_SMC
- F? (x2): symbol Device:Fuse -> RespiraWorks:0154010.DR
- J?: symbol Connector_Generic:Conn_01x04 -> RespiraWorks_Std:Conn_01x04
Changed lines of the file:
@@
 F 0 "C?" H 8550 4850 50  0000 L CNN
 F 1 "10uF" H 8550 4700 50  0000 L CNN
-F 2 "Capacitor_SMD:C_0603_1608Metric" H 8788 4650 50  0001 C CNN
+F 2 "RespiraWorks_Std:C_0603_1608Metric" H 8788 4650 50  0001 C CNN
 F 3 "~" H 8750 4800 50  0001 C CNN
 	1    8750 4800
@@
 F 0 "D?" V 3050 3550 50  0000 L CNN
 F 1 "20V" V 3150 3550 50  0000 L CNN
-F 2 "Diode_SMD:D_SMC" H 3100 3450 50  0001 C CNN
+F 2 "RespiraWorks_Std:D_SMC" H 3100 3450 50  0001 C CNN
 F 3 "https://www.diodes.com/assets/Datasheets/ds40740.pdf" H 3100 3450 50  0001 C CNN
 F 4 "Diodes Inc." V 3100 3450 50  0001 C CNN "Manufacturer"
@@
 POWER_SW_P
 $Comp
-L Device:Fuse F?
+L RespiraWorks:0154010.DR F?
 U 1 1 603A1854
 P 2700 3300
@@
 	9150 4850 9250 4850
 $Comp
-L Device:Fuse F?
+L RespiraWorks:0154010.DR F?
 U 1 1 602914E1
 P 9400 4850
@@
 F 0 "C?" H 4050 3450 50  0000 L CNN
 F 1 "33uF" H 4050 3350 50  0000 L CNN
-F 2 "" H 3938 3300 50  0001 C CNN
-F 3 "~" H 3900 3450 50  0001 C CNN
+F 2 "RespiraWorks_Std:CP_Elec_6.3x7.7" H 3938 3300 50  0001 C CNN
+F 3 "https://industrial.panasonic.com/cdbs/www-data/pdf/RDE0000/ABA0000C1181.pdf" H 3900 3450 50  0001 C CNN
 F 4 "50V" H 4050 3250 50  0000 L CNN "Voltage"
+F 5 "Panasonic" H 3900 3450 50  0001 C CNN "Manufacturer"
+F 6 "EEE-FK1H330XP" H 3900 3450 50  0001 C CNN "Manufacturer PN"
 	1    3900 3450
 	1    0    0    -1
@@
 Connection ~ 3100 3300
 $Comp
-L Connector_Generic:Conn_01x04 J?
+L RespiraWorks_Std:Conn_01x04 J?
 U 1 1 605A607B
 P 1550 3300

Commit message: inductor footprint assignments
Parts:
- removed C?: 10uF, RespiraWorks_Std:C_0603_1608Metric, symbol Device:C
- added C?: 10uF, RespiraWorks_Std:C_0805_2012Metric, symbol Device:C
Changed lines of the file:
@@
 BAT_P
-$Comp
-L Device:C C?
-U 1 1 605A6090
-P 8750 4800
-F 0 "C?" H 8550 4850 50  0000 L CNN
-F 1 "10uF" H 8550 4700 50  0000 L CNN
-F 2 "RespiraWorks_Std:C_0603_1608Metric" H 8788 4650 50  0001 C CNN
-F 3 "~" H 8750 4800 50  0001 C CNN
-	1    8750 4800
-	1    0    0    -1
-$EndComp
 $Comp
 L Connector_Generic:Conn_01x02 J?
@@
 Text HLabel 4650 3800 0    50   BiDi ~ 0
 SDA
-Wire Wire Line
-	8750 4950 9700 4950
-Wire Wire Line
-	8750 4650 8450 4650
-Connection ~ 8750 4650
-Wire Wire Line
-	8750 4950 8450 4950
-Connection ~ 8750 4950
 $Comp
 L power:GND #PWR?
@@
 Text HLabel 7050 4950 0    50   Output ~ 0
 BAT_ALRT
-Wire Wire Line
-	8750 4650 9150 4650
 Wire Wire Line
 	9150 4650 9150 4850
@@
 	-1   0    0    1
 $EndComp
+Wire Wire Line
+	8450 4650 8650 4650
+Wire Wire Line
+	8450 4950 8650 4950
+$Comp
+L Device:C C?
+U 1 1 603046C0
+P 8650 4800
+AR Path="/601A64F8/603046C0" Ref="C?"  Part="1"
+AR Path="/601A64F8/60567144/603046C0" Ref="C?"  Part="1"
+AR Path="/6023BF6A/60567144/603046C0" Ref="C?"  Part="1"
+AR Path="/6023BF6A/603046C0" Ref="C?"  Part="1"
+F 0 "C?" H 8750 4900 50  0000 L CNN
+F 1 "10uF" H 8750 4800 50  0000 L CNN
+F 2 "RespiraWorks_Std:C_0805_2012Metric" H 8688 4650 50  0001 C CNN
+F 3 "~" H 8650 4800 50  0001 C CNN
+F 4 "25V" H 8750 4700 50  0000 L CNN "Voltage"
+	1    8650 4800
+	1    0    0    -1
+$EndComp
+Connection ~ 8650 4650
+Wire Wire Line
+	8650 4650 9150 4650
+Connection ~ 8650 4950
+Wire Wire Line
+	8650 4950 9700 4950
 $EndSCHEMATC

Commit message: Top-level beginnings, minor fixes
Started on top-level schematic blocks and connections
Started changing some net names to mixed-case-with-dash format
Fixed version number, added titles and version to all schematic sheets
Fixed incorrect SWO pin assignment in cycle controller
Added a few add'l annotations to battery sheets
Connections:
- net labels added: 12Vout, Bat-Alert, PG-12V, PMon-ACOK, PMon-IAdp, PMon-IBat, PMon-PSys, Power-Sw-N, Power-Sw-P, Switched-VLink, VLogic, Vin-Adp
- net labels removed: 12VOUT, BAT_ALRT, PG_12V, PMON_ACOK, PMON_IADP, PMON_IBAT, PMON_PSYS, POWER_SW_N, POWER_SW_P, SWITCHED_VLINK, VIN_ADP, VLOGIC
Other:
- note added: "SMBJ20AQ: 32.4V max clamping @ 18.5A"
Changed lines of the file:
@@
 $Descr A4 11693 8268
 encoding utf-8
-Sheet 31 34
-Title ""
+Sheet 32 37
+Title "Power Entry / Battery Controller"
 Date ""
-Rev ""
-Comp ""
+Rev "A"
+Comp "RespiraWorks"
 Comment1 ""
 Comment2 ""
@@
 S 5150 3200 1200 700
 U 60567144
-F0 "Sheet60567143" 50
+F0 "Battery Charger / Source Switching" 50
 F1 "battery_charger.sch" 50
 F2 "SCL" I L 5150 3700 50
 F3 "SDA" B L 5150 3800 50
-F4 "VLOGIC" I L 5150 3600 50
-F5 "VIN_ADP" I L 5150 3300 50
-F6 "PACK_P" B R 6350 3400 50
-F7 "VLINK" O R 6350 3300 50
-F8 "PSYS" O R 6350 3500 50
-F9 "IBAT" O R 6350 3600 50
-F10 "IADPT" O R 6350 3700 50
-F11 "ACOK" O R 6350 3800 50
+F4 "VLogic" I L 5150 3600 50
+F5 "PACK_P" B R 6350 3400 50
+F6 "VLINK" O R 6350 3300 50
+F7 "PSYS" O R 6350 3500 50
+F8 "IBAT" O R 6350 3600 50
+F9 "IADPT" O R 6350 3700 50
+F10 "ACOK" O R 6350 3800 50
+F11 "VIn-Adp" I L 5150 3300 50
 $EndSheet
 $Sheet
 S 7550 4550 900  550
 U 60567757
-F0 "Sheet60567756" 50
+F0 "Battery Balancer" 50
 F1 "battery_balancer.sch" 50
 F2 "BAT_N" I R 8450 4950 50
@@
 AR Path="/601A64F8/60567144/605C357B" Ref="J?"  Part="1"
 AR Path="/6023BF6A/605C357B" Ref="J?"  Part="1"
+AR Path="/5FCD4B8E/603C510C/605C357B" Ref="J?"  Part="1"
+AR Path="/6041384A/605C357B" Ref="J?"  Part="1"
 F 0 "J?" H 10000 5050 50  0000 R CNN
 F 1 "BAT-PWR MegaFit 2x1" H 10000 5150 50  0000 R CNN
@@
 AR Path="/601A64F8/60567144/605C3581" Ref="#PWR?"  Part="1"
 AR Path="/6023BF6A/605C3581" Ref="#PWR?"  Part="1"
+AR Path="/5FCD4B8E/603C510C/605C3581" Ref="#PWR?"  Part="1"
+AR Path="/6041384A/605C3581" Ref="#PWR?"  Part="1"
 F 0 "#PWR?" H 1750 3150 50  0001 C CNN
 F 1 "GND" H 1755 3227 50  0000 C CNN
@@
 AR Path="/601A64F8/60567144/605C3588" Ref="D?"  Part="1"
 AR Path="/6023BF6A/605C3588" Ref="D?"  Part="1"
+AR Path="/5FCD4B8E/603C510C/605C3588" Ref="D?"  Part="1"
+AR Path="/6041384A/605C3588" Ref="D?"  Part="1"
 F 0 "D?" V 3050 3550 50  0000 L CNN
 F 1 "20V" V 3150 3550 50  0000 L CNN
@@
 AR Path="/601A64F8/60567144/605C358F" Ref="#PWR?"  Part="1"
 AR Path="/6023BF6A/605C358F" Ref="#PWR?"  Part="1"
+AR Path="/5FCD4B8E/603C510C/605C358F" Ref="#PWR?"  Part="1"
+AR Path="/6041384A/605C358F" Ref="#PWR?"  Part="1"
 F 0 "#PWR?" H 3100 3350 50  0001 C CNN
 F 1 "GND" H 3105 3427 50  0000 C CNN
@@
 $EndComp
 Text Label 4800 3300 0    50   ~ 0
-VIN_ADP
+Vin-Adp
 Wire Wire Line
 	1750 3200 2350 3200
@@
 	2350 3100 1750 3100
 Text Label 2350 3100 2    50   ~ 0
-POWER_SW_P
+Power-Sw-P
 Text Label 2350 3200 2    50   ~ 0
-POWER_SW_N
+Power-Sw-N
 Wire Wire Line
 	7800 3300 8350 3300
 Text Label 7800 3300 0    50   ~ 0
-POWER_SW_N
+Power-Sw-N
 Wire Wire Line
 	6950 3300 6350 3300
 Text Label 6950 3300 2    50   ~ 0
-POWER_SW_P
+Power-Sw-P
 $Comp
 L RespiraWorks:0154010.DR F?
 U 1 1 603A1854
 P 2700 3300
+AR Path="/5FCD4B8E/603C510C/603A1854" Ref="F?"  Part="1"
+AR Path="/6041384A/603A1854" Ref="F?"  Part="1"
 F 0 "F?" V 2503 3300 50  0000 C CNN
 F 1 "Fuse 10A" V 2594 3300 50  0000 C CNN
@@
 	5150 3600 4650 3600
 Text HLabel 4650 3600 0    50   Input ~ 0
-VLOGIC
+VLogic
 Text Label 4700 3600 0    50   ~ 0
-VLOGIC
+VLogic
 Wire Wire Line
 	8400 3450 7900 3450
 Text Label 7900 3450 0    50   ~ 0
-VLOGIC
+VLogic
 Wire Wire Line
 	9100 3450 9350 3450
@@
 	9100 3300 9350 3300
 Text HLabel 9350 3300 2    50   Output ~ 0
-12VOUT
+12Vout
 Text HLabel 9350 3450 2    50   Output ~ 0
-PG_12V
+PG-12V
 Wire Wire Line
 	6350 3500 6600 3500
 Text HLabel 6600 3500 2    50   Output ~ 0
-PMON_PSYS
+PMon-PSys
 Wire Wire Line
 	6350 3600 6600 3600
 Text HLabel 6600 3600 2    50   Output ~ 0
-PMON_IBAT
+PMon-IBat
 Wire Wire Line
 	6350 3700 6600 3700
 Text HLabel 6600 3700 2    50   Output ~ 0
-PMON_IADP
+PMon-IAdp
 Wire Wire Line
 	6350 3800 6600 3800
 Text HLabel 6600 3800 2    50   Output ~ 0
-PMON_ACOK
+PMon-ACOK
 Wire Wire Line
 	5150 3700 4650 3700
@@
 AR Path="/601A64F8/60567144/6047EA81" Ref="#PWR?"  Part="1"
 AR Path="/6023BF6A/6047EA81" Ref="#PWR?"  Part="1"
+AR Path="/5FCD4B8E/603C510C/6047EA81" Ref="#PWR?"  Part="1"
+AR Path="/6041384A/6047EA81" Ref="#PWR?"  Part="1"
 F 0 "#PWR?" H 7350 4950 50  0001 C CNN
 F 1 "GND" H 7355 5027 50  0000 C CNN
@@
 	7050 4950 7550 4950
 Text HLabel 7050 4950 0    50   Output ~ 0
-BAT_ALRT
+Bat-Alert
 Wire Wire Line
 	9150 4650 9150 4850
@@
 U 1 1 602914E1
 P 9400 4850
+AR Path="/5FCD4B8E/603C510C/602914E1" Ref="F?"  Part="1"
+AR Path="/6041384A/602914E1" Ref="F?"  Part="1"
 F 0 "F?" V 9100 4850 50  0000 C CNN
 F 1 "Fuse 10A" V 9200 4850 50  0000 C CNN
@@
 	8350 3300 8400 3300
 Text HLabel 9350 3000 2    50   Output ~ 0
-SWITCHED_VLINK
+Switched-VLink
 Text Notes 8800 3000 0    50   ~ 0
 12.0-16.8V
@@
 AR Path="/6023BF6A/60567144/6026FB4D" Ref="C?"  Part="1"
 AR Path="/6023BF6A/6026FB4D" Ref="C?"  Part="1"
+AR Path="/5FCD4B8E/603C510C/6026FB4D" Ref="C?"  Part="1"
+AR Path="/6041384A/6026FB4D" Ref="C?"  Part="1"
 F 0 "C?" H 4050 3450 50  0000 L CNN
 F 1 "33uF" H 4050 3350 50  0000 L CNN
@@
 AR Path="/601A64F8/60567144/602707F0" Ref="#PWR?"  Part="1"
 AR Path="/6023BF6A/602707F0" Ref="#PWR?"  Part="1"
+AR Path="/5FCD4B8E/603C510C/602707F0" Ref="#PWR?"  Part="1"
+AR Path="/6041384A/602707F0" Ref="#PWR?"  Part="1"
 F 0 "#PWR?" H 3900 3350 50  0001 C CNN
 F 1 "GND" H 3905 3427 50  0000 C CNN
@@
 U 1 1 605A607B
 P 1550 3300
+AR Path="/5FCD4B8E/603C510C/605A607B" Ref="J?"  Part="1"
+AR Path="/6041384A/605A607B" Ref="J?"  Part="1"
 F 0 "J?" H 1500 2750 50  0000 R CNN
 F 1 "POWER-ENTRY MegaFit 2x2" H 2150 2850 50  0000 R CNN
@@
 AR Path="/6023BF6A/60567144/603046C0" Ref="C?"  Part="1"
 AR Path="/6023BF6A/603046C0" Ref="C?"  Part="1"
+AR Path="/5FCD4B8E/603C510C/603046C0" Ref="C?"  Part="1"
+AR Path="/6041384A/603046C0" Ref="C?"  Part="1"
 F 0 "C?" H 8750 4900 50  0000 L CNN
 F 1 "10uF" H 8750 4800 50  0000 L CNN
@@
 Wire Wire Line
 	8650 4950 9700 4950
+Text Notes 2100 3900 0    50   ~ 0
+SMBJ20AQ: 32.4V max clamping @ 18.5A
 $EndSCHEMATC

Commit message: Stepper drivers, alarms, power
Broke out SPI pins from cycle controller, routed to stepper drivers
Alarm/alarm battery changes:
(Fixed incorrect use of +BATT instead of +5V_Batt)
(Removed "run FPGA from alarm battery" circuitry and moved alarm battery circuitry to alarms sheet)
Converted fixed power symbols on logic/control power sheet, solenoid driver sheet to hierarchical labels to make power flow more clear from top level
Minor parts consolidation
Changed lines of the file:
@@
 $Descr A4 11693 8268
 encoding utf-8
-Sheet 32 37
+Sheet 31 37
 Title "Power Entry / Battery Controller"
 Date ""
@@
 S 8400 3200 700  450
 U 60567D6E
-F0 "Sheet60567D6D" 50
+F0 "12V System Buck Converter" 50
 F1 "power_vsys.sch" 50
 F2 "VIN" I L 8400 3300 50
