File: pcb/battery_controller.sch (KiCad schematic (older format))
At the start: 7 parts

Commit message: Monitoring
Finished top-level connections
Added separate SysMonADC for FPGA
Added voltage dividers for sensing input voltage levels
Broke out oxygen/temp sensor power to a hierarchical pin
Changed stepper STBY names to Reset to match ICD
Added OR'ed pull-downs to Stepper-nReset
Added FPGA alarm, external clamping for Low-Alarm-Bat signal
Added ability for FPGA to turn off 5V-UI
Changed CC's GND/GNDA connection from hardwired jumper to net tie
Added testpoints for probing
Parts:
- added C? (x2): 10nF, RespiraWorks_Std:C_0603_1608Metric, symbol Device:C
- added R? (x2): 442k, RespiraWorks_Std:R_0603_1608Metric, symbol Device:R
- added R? (x4): 39k, RespiraWorks_Std:R_0603_1608Metric, symbol Device:R
Connections:
- net labels added: VBat-Sense, Vin-Sense
- wire segments 36 -> 49
Other:
- note added: "Scaling of 0.15x:\n22Vin = 3.3Vout\n18Vin = 2.7Vout\n13Vin = 1.95Vout\n11Vin = 1.65Vout\n\n240 Hz LPF"

Commit message: CC-I2C, BOM
Added missing pull-ups on CC-SDA, CC-SCL
First pass at BOM consolidation
Parts:
- J?: Manufacturer P/N 768290104 -> (none); Manufacturer PN (none) -> 768290104
- J?: Manufacturer P/N 768290102 -> (none); Manufacturer PN (none) -> 768290102
Changed lines of the file:
@@
 F 3 "~" H 9900 4950 50  0001 C CNN
 F 4 "Molex" H 9900 4950 50  0001 C CNN "Manufacturer"
-F 5 "768290102" H 9800 5250 50  0000 C CNN "Manufacturer P/N"
+F 5 "768290102" H 9900 4950 50  0001 C CNN "Manufacturer PN"
 	1    9900 4950
 	1    0    0    1
@@
 F 3 "~" H 1550 3300 50  0001 C CNN
 F 4 "Molex" H 1550 3300 50  0001 C CNN "Manufacturer"
-F 5 "768290104" H 1800 2950 50  0000 R CNN "Manufacturer P/N"
+F 5 "768290104" H 1550 2950 50  0001 C CNN "Manufacturer PN"
 	1    1550 3300
 	-1   0    0    1

Commit message: BOM
More BOM consolidation with bulk capacitors + changed tantalum stepper caps to aluminum, added bulk cap to PSol driver
Made stepper's 3.3V power naming consistent with others (3.3V->3V3)
Slightly increased current limit on PSOL/heater driver
Changed 3906 transistors to 2907 to better support +5V_Batt current
Parts:
- C?: Dielectric (none) -> Aluminum
- C?: footprint RespiraWorks_Std:C_0805_2012Metric -> RespiraWorks_Std:C_1210_3225Metric; Dielectric (none) -> X7S; Manufacturer (none) -> Murata; Manufacturer PN (none) -> GRM32EC72A106KE05L; Voltage 25V -> 100V
Changed lines of the file:
@@
 F 5 "Panasonic" H 3900 3450 50  0001 C CNN "Manufacturer"
 F 6 "EEE-FK1H330XP" H 3900 3450 50  0001 C CNN "Manufacturer PN"
+F 7 "Aluminum" H 3900 3450 50  0001 C CNN "Dielectric"
 	1    3900 3450
 	1    0    0    -1
@@
 F 0 "C?" H 8750 4900 50  0000 L CNN
 F 1 "10uF" H 8750 4800 50  0000 L CNN
-F 2 "RespiraWorks_Std:C_0805_2012Metric" H 8688 4650 50  0001 C CNN
+F 2 "RespiraWorks_Std:C_1210_3225Metric" H 8688 4650 50  0001 C CNN
 F 3 "~" H 8650 4800 50  0001 C CNN
-F 4 "25V" H 8750 4700 50  0000 L CNN "Voltage"
+F 4 "100V" H 8750 4700 50  0000 L CNN "Voltage"
+F 5 "X7S" H 8650 4800 50  0001 C CNN "Dielectric"
+F 6 "Murata" H 8650 4800 50  0001 C CNN "Manufacturer"
+F 7 "GRM32EC72A106KE05L" H 8650 4800 50  0001 C CNN "Manufacturer PN"
 	1    8650 4800
 	1    0    0    -1

Commit message: BOM, fixes
Finished assigning parts, footprints except generic resistors
Added series resistors for logic signals received by UI computer to protect against UI computer power-down
Added tolerance notes on main schem
Replaced PSol fuse with PTC
Enlarged PSol driver bypass resistors to 0 ohm
Changed PSol unpopulated current-limiting resistor to divider
Parts:
- C? (x2): Dielectric (none) -> NP0; Manufacturer (none) -> Murata; Manufacturer PN (none) -> GRM1885C1H103JA01D; Voltage (none) -> 50V
- F? (x2): value Fuse 10A -> 10A
Changed lines of the file:
@@
 AR Path="/6041384A/603A1854" Ref="F?"  Part="1"
 F 0 "F?" V 2503 3300 50  0000 C CNN
-F 1 "Fuse 10A" V 2594 3300 50  0000 C CNN
+F 1 "10A" V 2594 3300 50  0000 C CNN
 F 2 "RespiraWorks:Fuseholder_Littelfuse_OMNI-BLOK-154" V 2630 3300 50  0001 C CNN
 F 3 "https://www.littelfuse.com/~/media/electronics/datasheets/fuses/littelfuse_fuse_154_154t_154l_154tl_datasheet.pdf.pdf" H 2700 3300 50  0001 C CNN
@@
 AR Path="/6041384A/602914E1" Ref="F?"  Part="1"
 F 0 "F?" V 9100 4850 50  0000 C CNN
-F 1 "Fuse 10A" V 9200 4850 50  0000 C CNN
+F 1 "10A" V 9200 4850 50  0000 C CNN
 F 2 "RespiraWorks:Fuseholder_Littelfuse_OMNI-BLOK-154" V 9330 4850 50  0001 C CNN
 F 3 "https://www.littelfuse.com/~/media/electronics/datasheets/fuses/littelfuse_fuse_154_154t_154l_154tl_datasheet.pdf.pdf" H 9400 4850 50  0001 C CNN
@@
 F 2 "RespiraWorks_Std:C_0603_1608Metric" H 3938 5800 50  0001 C CNN
 F 3 "~" H 3900 5950 50  0001 C CNN
+F 4 "NP0" H 3900 5950 50  0001 C CNN "Dielectric"
+F 5 "Murata" H 3900 5950 50  0001 C CNN "Manufacturer"
+F 6 "GRM1885C1H103JA01D" H 3900 5950 50  0001 C CNN "Manufacturer PN"
+F 7 "50V" H 3900 5950 50  0001 C CNN "Voltage"
 	1    3900 5950
 	-1   0    0    -1
@@
 F 2 "RespiraWorks_Std:C_0603_1608Metric" H 6688 5800 50  0001 C CNN
 F 3 "~" H 6650 5950 50  0001 C CNN
+F 4 "NP0" H 6650 5950 50  0001 C CNN "Dielectric"
+F 5 "Murata" H 6650 5950 50  0001 C CNN "Manufacturer"
+F 6 "GRM1885C1H103JA01D" H 6650 5950 50  0001 C CNN "Manufacturer PN"
+F 7 "50V" H 6650 5950 50  0001 C CNN "Voltage"
 	1    6650 5950
 	-1   0    0    -1

Commit message: Stephanie fixes, net names
Removed duplicate global I2C pull-ups
Added missing BMP280 pin 7
Correcting pin names etc. on LM4120 voltage reference
Finished standardizing net names
Connections:
- net labels added: Bat-N, Bat-P
- net labels removed: BAT_N, BAT_P
Changed lines of the file:
@@
 F3 "SDA" B L 5150 3800 50
 F4 "VLogic" I L 5150 3600 50
-F5 "PACK_P" B R 6350 3400 50
-F6 "VLINK" O R 6350 3300 50
-F7 "PSYS" O R 6350 3500 50
-F8 "IBAT" O R 6350 3600 50
-F9 "IADPT" O R 6350 3700 50
+F5 "Pack-P" B R 6350 3400 50
+F6 "VLink" O R 6350 3300 50
+F7 "PSys" O R 6350 3500 50
+F8 "IBat" O R 6350 3600 50
+F9 "IAdp" O R 6350 3700 50
 F10 "ACOK" O R 6350 3800 50
-F11 "VIn-Adp" I L 5150 3300 50
+F11 "Vin-Adp" I L 5150 3300 50
 $EndSheet
 $Sheet
@@
 F0 "Battery Balancer" 50
 F1 "battery_balancer.sch" 50
-F2 "BAT_N" I R 8450 4950 50
-F3 "SYS_N" O L 7550 5050 50
-F4 "BAT_P" I R 8450 4650 50
-F5 "SYS_P" O L 7550 4650 50
+F2 "Bat-N" I R 8450 4950 50
+F3 "Sys-N" O L 7550 5050 50
+F4 "Bat-P" I R 8450 4650 50
+F5 "Sys-P" O L 7550 4650 50
 F6 "SCL" I L 7550 4750 50
 F7 "SDA" B L 7550 4850 50
-F8 "ALRT" O L 7550 4950 50
+F8 "Alrt" O L 7550 4950 50
 $EndSheet
 $Sheet
@@
 F0 "12V System Buck Converter" 50
 F1 "power_vsys.sch" 50
-F2 "VIN" I L 8400 3300 50
-F3 "12VOUT" O R 9100 3300 50
-F4 "VLOGIC" I L 8400 3450 50
+F2 "Vin" I L 8400 3300 50
+F3 "12Vout" O R 9100 3300 50
+F4 "VLogic" I L 8400 3450 50
 F5 "PG" O R 9100 3450 50
 $EndSheet
 Text Label 8950 4950 0    50   ~ 0
-BAT_N
+Bat-N
 Text Label 8950 4650 0    50   ~ 0
-BAT_P
+Bat-P
 $Comp
 L Connector_Generic:Conn_01x02 J?

Commit message: Added VSys-Power-Off connection to FPGA
Connections:
- net labels added: VSys-Power-Off
- wire segments 49 -> 50
Other:
- note added: "12V @ 7A"
Changed lines of the file:
@@
 $EndSheet
 $Sheet
-S 8400 3200 700  450
+S 8400 3200 700  500
 U 60567D6E
 F0 "12V System Buck Converter" 50
@@
 F4 "VLogic" I L 8400 3450 50
 F5 "PG" O R 9100 3450 50
+F6 "VSys-Power-Off" I L 8400 3600 50
 $EndSheet
 Text Label 8950 4950 0    50   ~ 0
@@
 Text Notes 7100 6400 0    50   ~ 0
 Scaling of 0.15x:\n22Vin = 3.3Vout\n18Vin = 2.7Vout\n13Vin = 1.95Vout\n11Vin = 1.65Vout\n\n240 Hz LPF
+Text Notes 9800 3350 0    50   ~ 0
+12V @ 7A
+Text HLabel 8300 3600 0    50   Input ~ 0
+VSys-Power-Off
+Wire Wire Line
+	8300 3600 8400 3600
 $EndSCHEMATC

Commit message: PCB Rev A Floorplanning (#1079)
* annotate schematics

* generate netlist

* define board edges at 150x300mm

* add parts to board (some pending errors)

* fix schem-pcb footprint mismatches and push to PCB

* preliminary packing at 155x300mm board size - marginal

* PCB floor planning

* added fan power and swapped solenoid/touchscreen power to vertical connectors
Parts:
- gave numbers to parts that had none: 15
Changed lines of the file:
@@
 AR Path="/6023BF6A/605C357B" Ref="J?"  Part="1"
 AR Path="/5FCD4B8E/603C510C/605C357B" Ref="J?"  Part="1"
-AR Path="/6041384A/605C357B" Ref="J?"  Part="1"
-F 0 "J?" H 10000 5050 50  0000 R CNN
+AR Path="/6041384A/605C357B" Ref="J45"  Part="1"
+F 0 "J45" H 10000 5050 50  0000 R CNN
 F 1 "BAT-PWR MegaFit 2x1" H 10000 5150 50  0000 R CNN
 F 2 "RespiraWorks_Std:Molex_Mega-Fit_76829-0102_2x01_P5.70mm_Vertical" H 9900 4950 50  0001 C CNN
@@
 AR Path="/6023BF6A/605C3581" Ref="#PWR?"  Part="1"
 AR Path="/5FCD4B8E/603C510C/605C3581" Ref="#PWR?"  Part="1"
-AR Path="/6041384A/605C3581" Ref="#PWR?"  Part="1"
-F 0 "#PWR?" H 1750 3150 50  0001 C CNN
+AR Path="/6041384A/605C3581" Ref="#PWR0321"  Part="1"
+F 0 "#PWR0321" H 1750 3150 50  0001 C CNN
 F 1 "GND" H 1755 3227 50  0000 C CNN
 F 2 "" H 1750 3400 50  0001 C CNN
@@
 AR Path="/6023BF6A/605C3588" Ref="D?"  Part="1"
 AR Path="/5FCD4B8E/603C510C/605C3588" Ref="D?"  Part="1"
-AR Path="/6041384A/605C3588" Ref="D?"  Part="1"
-F 0 "D?" V 3050 3550 50  0000 L CNN
+AR Path="/6041384A/605C3588" Ref="D26"  Part="1"
+F 0 "D26" V 3050 3550 50  0000 L CNN
 F 1 "20V" V 3150 3550 50  0000 L CNN
 F 2 "RespiraWorks_Std:D_SMC" H 3100 3450 50  0001 C CNN
@@
 AR Path="/6023BF6A/605C358F" Ref="#PWR?"  Part="1"
 AR Path="/5FCD4B8E/603C510C/605C358F" Ref="#PWR?"  Part="1"
-AR Path="/6041384A/605C358F" Ref="#PWR?"  Part="1"
-F 0 "#PWR?" H 3100 3350 50  0001 C CNN
+AR Path="/6041384A/605C358F" Ref="#PWR0322"  Part="1"
+F 0 "#PWR0322" H 3100 3350 50  0001 C CNN
 F 1 "GND" H 3105 3427 50  0000 C CNN
 F 2 "" H 3100 3600 50  0001 C CNN
@@
 P 2700 3300
 AR Path="/5FCD4B8E/603C510C/603A1854" Ref="F?"  Part="1"
-AR Path="/6041384A/603A1854" Ref="F?"  Part="1"
-F 0 "F?" V 2503 3300 50  0000 C CNN
+AR Path="/6041384A/603A1854" Ref="F2"  Part="1"
+F 0 "F2" V 2503 3300 50  0000 C CNN
 F 1 "10A" V 2594 3300 50  0000 C CNN
 F 2 "RespiraWorks:Fuseholder_Littelfuse_OMNI-BLOK-154" V 2630 3300 50  0001 C CNN
@@
 AR Path="/6023BF6A/6047EA81" Ref="#PWR?"  Part="1"
 AR Path="/5FCD4B8E/603C510C/6047EA81" Ref="#PWR?"  Part="1"
-AR Path="/6041384A/6047EA81" Ref="#PWR?"  Part="1"
-F 0 "#PWR?" H 7350 4950 50  0001 C CNN
+AR Path="/6041384A/6047EA81" Ref="#PWR0328"  Part="1"
+F 0 "#PWR0328" H 7350 4950 50  0001 C CNN
 F 1 "GND" H 7355 5027 50  0000 C CNN
 F 2 "" H 7350 5200 50  0001 C CNN
@@
 P 9400 4850
 AR Path="/5FCD4B8E/603C510C/602914E1" Ref="F?"  Part="1"
-AR Path="/6041384A/602914E1" Ref="F?"  Part="1"
-F 0 "F?" V 9100 4850 50  0000 C CNN
+AR Path="/6041384A/602914E1" Ref="F3"  Part="1"
+F 0 "F3" V 9100 4850 50  0000 C CNN
 F 1 "10A" V 9200 4850 50  0000 C CNN
 F 2 "RespiraWorks:Fuseholder_Littelfuse_OMNI-BLOK-154" V 9330 4850 50  0001 C CNN
@@
 AR Path="/6023BF6A/6026FB4D" Ref="C?"  Part="1"
 AR Path="/5FCD4B8E/603C510C/6026FB4D" Ref="C?"  Part="1"
-AR Path="/6041384A/6026FB4D" Ref="C?"  Part="1"
-F 0 "C?" H 4050 3450 50  0000 L CNN
+AR Path="/6041384A/6026FB4D" Ref="C94"  Part="1"
+F 0 "C94" H 4050 3450 50  0000 L CNN
 F 1 "33uF" H 4050 3350 50  0000 L CNN
 F 2 "RespiraWorks_Std:CP_Elec_6.3x7.7" H 3938 3300 50  0001 C CNN
@@
 AR Path="/6023BF6A/602707F0" Ref="#PWR?"  Part="1"
 AR Path="/5FCD4B8E/603C510C/602707F0" Ref="#PWR?"  Part="1"
-AR Path="/6041384A/602707F0" Ref="#PWR?"  Part="1"
-F 0 "#PWR?" H 3900 3350 50  0001 C CNN
+AR Path="/6041384A/602707F0" Ref="#PWR0324"  Part="1"
+F 0 "#PWR0324" H 3900 3350 50  0001 C CNN
 F 1 "GND" H 3905 3427 50  0000 C CNN
 F 2 "" H 3900 3600 50  0001 C CNN
@@
 P 1550 3300
 AR Path="/5FCD4B8E/603C510C/605A607B" Ref="J?"  Part="1"
-AR Path="/6041384A/605A607B" Ref="J?"  Part="1"
-F 0 "J?" H 1500 2750 50  0000 R CNN
+AR Path="/6041384A/605A607B" Ref="J44"  Part="1"
+F 0 "J44" H 1500 2750 50  0000 R CNN
 F 1 "POWER-ENTRY MegaFit 2x2" H 2150 2850 50  0000 R CNN
 F 2 "RespiraWorks_Std:Molex_Mega-Fit_76829-0104_2x02_P5.70mm_Vertical" H 1550 3300 50  0001 C CNN
@@
 AR Path="/6023BF6A/603046C0" Ref="C?"  Part="1"
 AR Path="/5FCD4B8E/603C510C/603046C0" Ref="C?"  Part="1"
-AR Path="/6041384A/603046C0" Ref="C?"  Part="1"
-F 0 "C?" H 8750 4900 50  0000 L CNN
+AR Path="/6041384A/603046C0" Ref="C97"  Part="1"
+F 0 "C97" H 8750 4900 50  0000 L CNN
 F 1 "10uF" H 8750 4800 50  0000 L CNN
 F 2 "RespiraWorks_Std:C_1210_3225Metric" H 8688 4650 50  0001 C CNN
@@
 AR Path="/5FCD4B8E/603C510C/60567144/60E0E216" Ref="R?"  Part="1"
 AR Path="/6041384A/60567144/60E0E216" Ref="R?"  Part="1"
-AR Path="/6041384A/60E0E216" Ref="R?"  Part="1"
-F 0 "R?" H 6270 5696 50  0000 L CNN
+AR Path="/6041384A/60E0E216" Ref="R166"  Part="1"
+F 0 "R166" H 6270 5696 50  0000 L CNN
 F 1 "442k" H 6270 5605 50  0000 L CNN
 F 2 "RespiraWorks_Std:R_0603_1608Metric" V 6130 5650 50  0001 C CNN
@@
 AR Path="/5FCD4B8E/603C510C/60567144/60E0E21C" Ref="R?"  Part="1"
 AR Path="/6041384A/60567144/60E0E21C" Ref="R?"  Part="1"
-AR Path="/6041384A/60E0E21C" Ref="R?"  Part="1"
-F 0 "R?" H 6270 6046 50  0000 L CNN
+AR Path="/6041384A/60E0E21C" Ref="R167"  Part="1"
+F 0 "R167" H 6270 6046 50  0000 L CNN
 F 1 "39k" H 6270 5955 50  0000 L CNN
 F 2 "RespiraWorks_Std:R_0603_1608Metric" V 6130 6000 50  0001 C CNN
@@
 AR Path="/5FCD4B8E/603C510C/60567144/60E0E223" Ref="#PWR?"  Part="1"
 AR Path="/6041384A/60567144/60E0E223" Ref="#PWR?"  Part="1"
-AR Path="/6041384A/60E0E223" Ref="#PWR?"  Part="1"
-F 0 "#PWR?" H 6200 6200 50  0001 C CNN
+AR Path="/6041384A/60E0E223" Ref="#PWR0326"  Part="1"
+F 0 "#PWR0326" H 6200 6200 50  0001 C CNN
 F 1 "GND" H 6205 6277 50  0000 C CNN
 F 2 "" H 6200 6450 50  0001 C CNN
@@
 AR Path="/5FCD4B8E/603C510C/60567144/60E1EDE3" Ref="R?"  Part="1"
 AR Path="/6041384A/60567144/60E1EDE3" Ref="R?"  Part="1"
-AR Path="/6041384A/60E1EDE3" Ref="R?"  Part="1"
-F 0 "R?" H 6270 6346 50  0000 L CNN
+AR Path="/6041384A/60E1EDE3" Ref="R168"  Part="1"
+F 0 "R168" H 6270 6346 50  0000 L CNN
 F 1 "39k" H 6270 6255 50  0000 L CNN
 F 2 "RespiraWorks_Std:R_0603_1608Metric" V 6130 6300 50  0001 C CNN
@@
 AR Path="/5FCD4B8E/603C510C/60567144/60E28A37" Ref="#PWR?"  Part="1"
 AR Path="/6041384A/60567144/60E28A37" Ref="#PWR?"  Part="1"
-AR Path="/6041384A/60E28A37" Ref="#PWR?"  Part="1"
-F 0 "#PWR?" H 6650 5850 50  0001 C CNN
+AR Path="/6041384A/60E28A37" Ref="#PWR0327"  Part="1"
+F 0 "#PWR0327" H 6650 5850 50  0001 C CNN
 F 1 "GND" H 6655 5927 50  0000 C CNN
 F 2 "" H 6650 6100 50  0001 C CNN
@@
 AR Path="/5FCD4B8E/603C510C/60567144/60E304BA" Ref="R?"  Part="1"
 AR Path="/6041384A/60567144/60E304BA" Ref="R?"  Part="1"
-AR Path="/6041384A/60E304BA" Ref="R?"  Part="1"
-F 0 "R?" H 3520 5696 50  0000 L CNN
+AR Path="/6041384A/60E304BA" Ref="R163"  Part="1"
+F 0 "R163" H 3520 5696 50  0000 L CNN
 F 1 "442k" H 3520 5605 50  0000 L CNN
 F 2 "RespiraWorks_Std:R_0603_1608Metric" V 3380 5650 50  0001 C CNN
@@
 AR Path="/5FCD4B8E/603C510C/60567144/60E304C0" Ref="R?"  Part="1"
 AR Path="/6041384A/60567144/60E304C0" Ref="R?"  Part="1"
-AR Path="/6041384A/60E304C0" Ref="R?"  Part="1"
-F 0 "R?" H 3520 6046 50  0000 L CNN
+AR Path="/6041384A/60E304C0" Ref="R164"  Part="1"
+F 0 "R164" H 3520 6046 50  0000 L CNN
 F 1 "39k" H 3520 5955 50  0000 L CNN
 F 2 "RespiraWorks_Std:R_0603_1608Metric" V 3380 6000 50  0001 C CNN
@@
 AR Path="/5FCD4B8E/603C510C/60567144/60E304C7" Ref="#PWR?"  Part="1"
 AR Path="/6041384A/60567144/60E304C7" Ref="#PWR?"  Part="1"
-AR Path="/6041384A/60E304C7" Ref="#PWR?"  Part="1"
-F 0 "#PWR?" H 3450 6200 50  0001 C CNN
+AR Path="/6041384A/60E304C7" Ref="#PWR0323"  Part="1"
+F 0 "#PWR0323" H 3450 6200 50  0001 C CNN
 F 1 "GND" H 3455 6277 50  0000 C CNN
 F 2 "" H 3450 6450 50  0001 C CNN
@@
 AR Path="/5FCD4B8E/603C510C/60567144/60E304D0" Ref="R?"  Part="1"
 AR Path="/6041384A/60567144/60E304D0" Ref="R?"  Part="1"
-AR Path="/6041384A/60E304D0" Ref="R?"  Part="1"
-F 0 "R?" H 3520 6346 50  0000 L CNN
+AR Path="/6041384A/60E304D0" Ref="R165"  Part="1"
+F 0 "R165" H 3520 6346 50  0000 L CNN
 F 1 "39k" H 3520 6255 50  0000 L CNN
 F 2 "RespiraWorks_Std:R_0603_1608Metric" V 3380 6300 50  0001 C CNN
@@
 AR Path="/5FCD4B8E/603C510C/60567144/60E304DE" Ref="#PWR?"  Part="1"
 AR Path="/6041384A/60567144/60E304DE" Ref="#PWR?"  Part="1"
-AR Path="/6041384A/60E304DE" Ref="#PWR?"  Part="1"
-F 0 "#PWR?" H 3900 5850 50  0001 C CNN
+AR Path="/6041384A/60E304DE" Ref="#PWR0325"  Part="1"
+F 0 "#PWR0325" H 3900 5850 50  0001 C CNN
 F 1 "GND" H 3905 5927 50  0000 C CNN
 F 2 "" H 3900 6100 50  0001 C CNN
@@
 AR Path="/5FCD4B8E/603C510C/60567144/60E3B234" Ref="C?"  Part="1"
 AR Path="/6041384A/60567144/60E3B234" Ref="C?"  Part="1"
-AR Path="/6041384A/60E3B234" Ref="C?"  Part="1"
-F 0 "C?" H 3650 5950 50  0000 L CNN
+AR Path="/6041384A/60E3B234" Ref="C95"  Part="1"
+F 0 "C95" H 3650 5950 50  0000 L CNN
 F 1 "10nF" H 3650 5850 50  0000 L CNN
 F 2 "RespiraWorks_Std:C_0603_1608Metric" H 3938 5800 50  0001 C CNN
@@
 AR Path="/5FCD4B8E/603C510C/60567144/60E3DD19" Ref="C?"  Part="1"
 AR Path="/6041384A/60567144/60E3DD19" Ref="C?"  Part="1"
-AR Path="/6041384A/60E3DD19" Ref="C?"  Part="1"
-F 0 "C?" H 6400 5950 50  0000 L CNN
+AR Path="/6041384A/60E3DD19" Ref="C96"  Part="1"
+F 0 "C96" H 6400 5950 50  0000 L CNN
 F 1 "10nF" H 6400 5850 50  0000 L CNN
 F 2 "RespiraWorks_Std:C_0603_1608Metric" H 6688 5800 50  0001 C CNN
