File: pcb/power_vsys.sch (KiCad schematic (older format))
At the start: 30 parts

Commit message: clean up, add part numbers to parts, added design comments
Parts:
- removed D?: D_Schottky, symbol Device:D_Schottky
- added D?: BAT54J, Diode_SMD:D_SOD-323F, symbol Diode:BAT54J
Changed lines of the file:
@@
 	6450 2950 7250 2950
 Connection ~ 7250 2950
-Wire Wire Line
-	4950 1800 4950 2150
-Connection ~ 4950 1800
-$Comp
-L Device:D_Schottky D?
-U 1 1 60205CBE
-P 5100 1800
-AR Path="/601A64F8/60205CBE" Ref="D?"  Part="1"
-AR Path="/601A64F8/60567144/60205CBE" Ref="D?"  Part="1"
-AR Path="/601A64F8/60567D6E/60205CBE" Ref="D?"  Part="1"
-F 0 "D?" H 5050 1700 50  0000 C CNN
-F 1 "D_Schottky" H 5400 1700 50  0000 C CNN
-F 2 "" H 5100 1800 50  0001 C CNN
-F 3 "~" H 5100 1800 50  0001 C CNN
-	1    5100 1800
-	1    0    0    -1
-$EndComp
 Text Notes 2550 1250 0    50   ~ 0
 13-20V IN
@@
 	1    0    0    -1
 $EndComp
-Wire Wire Line
-	4950 1650 4950 1800
 Connection ~ 4700 1350
 $Comp
@@
 Wire Wire Line
 	6450 4400 7450 4400
+$Comp
+L Diode:BAT54J D?
+U 1 1 6028E91B
+P 5100 1800
+F 0 "D?" H 5100 1900 50  0000 C CNN
+F 1 "BAT54J" H 5150 1650 50  0000 C CNN
+F 2 "Diode_SMD:D_SOD-323F" H 5100 1625 50  0001 C CNN
+F 3 "https://assets.nexperia.com/documents/data-sheet/BAT54J.pdf" H 5100 1800 50  0001 C CNN
+	1    5100 1800
+	1    0    0    -1
+$EndComp
+Wire Wire Line
+	4950 1650 4950 1800
+Connection ~ 4950 1800
+Wire Wire Line
+	4950 1800 4950 2150
 $EndSCHEMATC

Commit message: WIP implement comments from review
Parts:
- added R?: 10, Resistor_SMD:R_0603_1608Metric, symbol Device:R
- C?: value 120nF -> 0.1uF
- C?: value 200nF -> 220nF

Commit message: WIP implement PR comments
Parts:
- removed R?: 3k, Resistor_SMD:R_0603_1608Metric, symbol Device:R
- added Q?: MMBT3904, Package_TO_SOT_SMD:SOT-23, symbol Transistor_BJT:MMBT3904
- added R?: 0.006, RespiraWorks_Std:R_1206_3216Metric, symbol Device:R
- added R? (x2): 10k, Resistor_SMD:R_0603_1608Metric, symbol Device:R
- C?: value 0.22uF -> 33pF
Connections:
- net labels added: VSYS_EN
- wire segments 94 -> 96
Other:
- note added: "12.5-16.8V IN"
- note added: "Cycle-by-cycle current limit: 75mA -> 12.5A"
- note removed: "13-20V IN"
Changed lines of the file:
@@
 	4050 3150 4550 3150
-Wire Wire Line
-	5000 3500 4600 3500
 Wire Wire Line
 	4550 2550 4550 2750
@@
 Connection ~ 7250 2950
 Text Notes 2550 1250 0    50   ~ 0
-13-20V IN
+12.5-16.8V IN
 Text HLabel 2750 1350 0    50   Input ~ 0
 VIN
@@
 Wire Wire Line
 	6450 2150 6600 2150
-Connection ~ 6600 1650
-Wire Wire Line
-	6000 1650 6600 1650
 Wire Wire Line
 	7250 1350 7500 1350
@@
 	7250 1350 7250 2650
 Wire Wire Line
-	7050 1350 7250 1350
-Wire Wire Line
 	4200 1550 4200 2750
 Wire Wire Line
 	4500 1750 4500 1850
-Connection ~ 7050 1350
-Connection ~ 6900 1650
-Wire Wire Line
-	7050 1650 7050 1350
-Wire Wire Line
-	6900 1650 7050 1650
 Wire Wire Line
 	6900 2350 6900 1650
-Wire Wire Line
-	5450 1350 5600 1350
-Connection ~ 5450 1350
-Wire Wire Line
-	5450 1650 5450 1350
-Wire Wire Line
-	5700 1650 5450 1650
-$Comp
-L Device:R R?
-U 1 1 601EDEE1
-P 5850 1650
-AR Path="/601A64F8/601EDEE1" Ref="R?"  Part="1"
-AR Path="/601A64F8/60567144/601EDEE1" Ref="R?"  Part="1"
-AR Path="/601A64F8/60567D6E/601EDEE1" Ref="R?"  Part="1"
-AR Path="/6023BF6A/60567D6E/601EDEE1" Ref="R?"  Part="1"
-F 0 "R?" V 5800 1400 50  0000 L CNN
-F 1 "3k" V 5800 1800 50  0000 L CNN
-F 2 "Resistor_SMD:R_0603_1608Metric" V 5780 1650 50  0001 C CNN
-F 3 "~" H 5850 1650 50  0001 C CNN
-	1    5850 1650
-	0    1    1    0
-$EndComp
 $Comp
 L Device:C C?
@@
 AR Path="/601A64F8/60567D6E/601ED324" Ref="C?"  Part="1"
 AR Path="/6023BF6A/60567D6E/601ED324" Ref="C?"  Part="1"
-F 0 "C?" V 6900 1850 50  0000 L CNN
-F 1 "0.22uF" V 6800 1700 50  0000 L CNN
+F 0 "C?" V 6600 1700 50  0000 L CNN
+F 1 "33pF" V 6500 1600 50  0000 L CNN
 F 2 "Capacitor_SMD:C_0603_1608Metric" H 6788 1500 50  0001 C CNN
 F 3 "~" H 6750 1650 50  0001 C CNN
@@
 	4050 1650 4050 3150
 Wire Wire Line
-	5900 1350 7050 1350
-Wire Wire Line
-	4950 1350 5450 1350
+	5900 1350 6600 1350
 Connection ~ 4950 1350
 $Comp
@@
 $EndComp
 Wire Wire Line
-	5000 3700 4600 3700
-Wire Wire Line
-	4600 3700 4600 3500
-Wire Wire Line
 	6450 3900 7750 3900
 Wire Wire Line
@@
 Wire Wire Line
 	6450 5100 7150 5100
-Connection ~ 4600 3500
 Connection ~ 3750 1350
 Wire Wire Line
@@
 	1    0    0    -1
 $EndComp
-Wire Wire Line
-	4600 3500 3750 3500
-Wire Wire Line
-	3750 3500 3750 1350
 $Comp
 L Device:C C?
@@
 Wire Wire Line
 	4850 2550 5000 2550
+$Comp
+L Device:R R?
+U 1 1 60286B7B
+P 6750 1350
+AR Path="/601A64F8/60286B7B" Ref="R?"  Part="1"
+AR Path="/601A64F8/60567144/60286B7B" Ref="R?"  Part="1"
+AR Path="/601A64F8/60567D6E/60286B7B" Ref="R?"  Part="1"
+AR Path="/6023BF6A/60567D6E/60286B7B" Ref="R?"  Part="1"
+F 0 "R?" V 6550 1300 50  0000 L CNN
+F 1 "0.006" V 6650 1250 50  0000 L CNN
+F 2 "RespiraWorks_Std:R_1206_3216Metric" V 6680 1350 50  0001 C CNN
+F 3 "https://www.te.com/commerce/DocumentDelivery/DDEController?Action=srchrtrv&DocNm=1773449-3&DocType=DS&DocLang=English" H 6750 1350 50  0001 C CNN
+F 4 "TE Connectivity" V 6750 1350 50  0001 C CNN "Manufacturer"
+F 5 "TLR2B10DR006FTDG" V 6750 1350 50  0001 C CNN "Manufacturer PN"
+	1    6750 1350
+	0    1    1    0
+$EndComp
+Wire Wire Line
+	4950 1350 5600 1350
+Wire Wire Line
+	6900 1350 7250 1350
+Wire Wire Line
+	6600 1650 6600 1350
+Connection ~ 6600 1650
+Connection ~ 6600 1350
+Wire Wire Line
+	6900 1650 6900 1350
+Connection ~ 6900 1650
+Connection ~ 6900 1350
+Text Notes 6100 1050 0    50   ~ 0
+Cycle-by-cycle current limit: 75mA -> 12.5A
+Wire Wire Line
+	3750 3500 3750 2500
+$Comp
+L Transistor_BJT:MMBT3904 Q?
+U 1 1 602A3DA2
+P 2900 3100
+F 0 "Q?" H 3091 3146 50  0000 L CNN
+F 1 "MMBT3904" H 3091 3055 50  0000 L CNN
+F 2 "Package_TO_SOT_SMD:SOT-23" H 3100 3025 50  0001 L CIN
+F 3 "https://www.onsemi.com/pub/Collateral/2N3903-D.PDF" H 2900 3100 50  0001 L CNN
+	1    2900 3100
+	1    0    0    -1
+$EndComp
+$Comp
+L power:GND #PWR?
+U 1 1 602A5044
+P 3000 3300
+AR Path="/601A64F8/602A5044" Ref="#PWR?"  Part="1"
+AR Path="/601A64F8/60567144/602A5044" Ref="#PWR?"  Part="1"
+AR Path="/601A64F8/60567D6E/602A5044" Ref="#PWR?"  Part="1"
+AR Path="/6023BF6A/60567D6E/602A5044" Ref="#PWR?"  Part="1"
+F 0 "#PWR?" H 3000 3050 50  0001 C CNN
+F 1 "GND" H 3005 3127 50  0000 C CNN
+F 2 "" H 3000 3300 50  0001 C CNN
+F 3 "" H 3000 3300 50  0001 C CNN
+	1    3000 3300
+	1    0    0    -1
+$EndComp
+$Comp
+L Device:R R?
+U 1 1 602A8288
+P 3000 2650
+AR Path="/601A64F8/602A8288" Ref="R?"  Part="1"
+AR Path="/601A64F8/60567144/602A8288" Ref="R?"  Part="1"
+AR Path="/601A64F8/60567D6E/602A8288" Ref="R?"  Part="1"
+AR Path="/6023BF6A/60567D6E/602A8288" Ref="R?"  Part="1"
+F 0 "R?" H 2700 2700 50  0000 L CNN
+F 1 "10k" H 2700 2600 50  0000 L CNN
+F 2 "Resistor_SMD:R_0603_1608Metric" V 2930 2650 50  0001 C CNN
+F 3 "~" H 3000 2650 50  0001 C CNN
+	1    3000 2650
+	1    0    0    -1
+$EndComp
+Wire Wire Line
+	3000 2500 3750 2500
+Connection ~ 3750 2500
+Wire Wire Line
+	3750 2500 3750 1350
+Wire Wire Line
+	3000 2800 3000 2850
+Wire Wire Line
+	3000 2850 3600 2850
+Wire Wire Line
+	3600 2850 3600 3700
+Connection ~ 3000 2850
+Wire Wire Line
+	3000 2850 3000 2900
+Wire Wire Line
+	3600 3700 5000 3700
+Wire Wire Line
+	3750 3500 5000 3500
+Wire Wire Line
+	2700 3100 2300 3100
+Text HLabel 1350 3100 0    50   Input ~ 0
+VSYS_EN
+$Comp
+L Device:R R?
+U 1 1 602BAB86
+P 2150 3100
+AR Path="/601A64F8/602BAB86" Ref="R?"  Part="1"
+AR Path="/601A64F8/60567144/602BAB86" Ref="R?"  Part="1"
+AR Path="/601A64F8/60567D6E/602BAB86" Ref="R?"  Part="1"
+AR Path="/6023BF6A/60567D6E/602BAB86" Ref="R?"  Part="1"
+F 0 "R?" V 1950 3050 50  0000 L CNN
+F 1 "10k" V 2050 3050 50  0000 L CNN
+F 2 "Resistor_SMD:R_0603_1608Metric" V 2080 3100 50  0001 C CNN
+F 3 "~" H 2150 3100 50  0001 C CNN
+	1    2150 3100
+	0    1    1    0
+$EndComp
+Wire Wire Line
+	2000 3100 1350 3100
 $EndSCHEMATC

Commit message: updated footprints to reference to RW library
Parts:
- C? (x9): footprint Capacitor_SMD:C_0603_1608Metric -> RespiraWorks_Std:C_0603_1608Metric
- C? (x6): footprint Capacitor_SMD:C_0805_2012Metric -> RespiraWorks_Std:C_0805_2012Metric
- D?: footprint Diode_SMD:D_SOD-323F -> RespiraWorks_Std:D_SOD-323F
- Q? (x2): footprint Package_SON:VSON-8_3.3x3.3mm_P0.65mm_NexFET -> RespiraWorks_Std:VSON-8_3.3x3.3mm_P0.65mm_NexFET
- Q?: footprint Package_TO_SOT_SMD:SOT-23 -> RespiraWorks_Std:SOT-23
- R? (x10): footprint Resistor_SMD:R_0603_1608Metric -> RespiraWorks_Std:C_0603_1608Metric
- R?: footprint Resistor_SMD:R_0603_1608Metric -> RespiraWorks_Std:R_0603_1608Metric
- U?: footprint Package_DFN_QFN:VQFN-24-1EP_4x4mm_P0.5mm_EP2.45x2.45mm_ThermalVias -> RespiraWorks_Std:VQFN-24-1EP_4x4mm_P0.5mm_EP2.45x2.45mm_ThermalVias
Changed lines of the file:
@@
 F 0 "R?" V 4650 2700 50  0000 L CNN
 F 1 "10" V 4650 3100 50  0000 L CNN
-F 2 "Resistor_SMD:R_0603_1608Metric" V 4630 2950 50  0001 C CNN
+F 2 "RespiraWorks_Std:C_0603_1608Metric" V 4630 2950 50  0001 C CNN
 F 3 "~" H 4700 2950 50  0001 C CNN
 	1    4700 2950
@@
 F 0 "R?" H 6950 2850 50  0000 L CNN
 F 1 "90.9k" H 6950 2750 50  0000 L CNN
-F 2 "Resistor_SMD:R_0603_1608Metric" V 7180 2800 50  0001 C CNN
+F 2 "RespiraWorks_Std:C_0603_1608Metric" V 7180 2800 50  0001 C CNN
 F 3 "~" H 7250 2800 50  0001 C CNN
 	1    7250 2800
@@
 F 0 "R?" H 6950 3150 50  0000 L CNN
 F 1 "10.1k" H 6950 3050 50  0000 L CNN
-F 2 "Resistor_SMD:R_0603_1608Metric" V 7180 3100 50  0001 C CNN
+F 2 "RespiraWorks_Std:C_0603_1608Metric" V 7180 3100 50  0001 C CNN
 F 3 "~" H 7250 3100 50  0001 C CNN
 	1    7250 3100
@@
 F 0 "C?" H 8450 1400 50  0000 L CNN
 F 1 "10uF" H 8450 1300 50  0000 L CNN
-F 2 "Capacitor_SMD:C_0805_2012Metric" H 8438 1350 50  0001 C CNN
+F 2 "RespiraWorks_Std:C_0805_2012Metric" H 8438 1350 50  0001 C CNN
 F 3 "~" H 8400 1500 50  0001 C CNN
 F 4 "35V" H 8450 1200 50  0000 L CNN "Voltage"
@@
 F 0 "C?" H 8150 1400 50  0000 L CNN
 F 1 "10uF" H 8150 1300 50  0000 L CNN
-F 2 "Capacitor_SMD:C_0805_2012Metric" H 8138 1350 50  0001 C CNN
+F 2 "RespiraWorks_Std:C_0805_2012Metric" H 8138 1350 50  0001 C CNN
 F 3 "~" H 8100 1500 50  0001 C CNN
 F 4 "35V" H 8150 1200 50  0000 L CNN "Voltage"
@@
 F 0 "C?" H 7850 1400 50  0000 L CNN
 F 1 "10uF" H 7850 1300 50  0000 L CNN
-F 2 "Capacitor_SMD:C_0805_2012Metric" H 7838 1350 50  0001 C CNN
+F 2 "RespiraWorks_Std:C_0805_2012Metric" H 7838 1350 50  0001 C CNN
 F 3 "~" H 7800 1500 50  0001 C CNN
 F 4 "35V" H 7850 1200 50  0000 L CNN "Voltage"
@@
 F 0 "C?" H 7550 1400 50  0000 L CNN
 F 1 "10uF" H 7550 1300 50  0000 L CNN
-F 2 "Capacitor_SMD:C_0805_2012Metric" H 7538 1350 50  0001 C CNN
+F 2 "RespiraWorks_Std:C_0805_2012Metric" H 7538 1350 50  0001 C CNN
 F 3 "~" H 7500 1500 50  0001 C CNN
 F 4 "35V" H 7550 1200 50  0000 L CNN "Voltage"
@@
 F 0 "C?" V 6600 1700 50  0000 L CNN
 F 1 "33pF" V 6500 1600 50  0000 L CNN
-F 2 "Capacitor_SMD:C_0603_1608Metric" H 6788 1500 50  0001 C CNN
+F 2 "RespiraWorks_Std:C_0603_1608Metric" H 6788 1500 50  0001 C CNN
 F 3 "~" H 6750 1650 50  0001 C CNN
 	1    6750 1650
@@
 F 0 "C?" H 3500 1400 50  0000 L CNN
 F 1 "10uF" H 3500 1300 50  0000 L CNN
-F 2 "Capacitor_SMD:C_0805_2012Metric" H 3488 1350 50  0001 C CNN
+F 2 "RespiraWorks_Std:C_0805_2012Metric" H 3488 1350 50  0001 C CNN
 F 3 "~" H 3450 1500 50  0001 C CNN
 F 4 "35V" H 3500 1200 50  0000 L CNN "Voltage"
@@
 F 0 "C?" H 3200 1400 50  0000 L CNN
 F 1 "10uF" H 3200 1300 50  0000 L CNN
-F 2 "Capacitor_SMD:C_0805_2012Metric" H 3188 1350 50  0001 C CNN
+F 2 "RespiraWorks_Std:C_0805_2012Metric" H 3188 1350 50  0001 C CNN
 F 3 "~" H 3150 1500 50  0001 C CNN
 F 4 "35V" H 3200 1200 50  0000 L CNN "Voltage"
@@
 F 0 "Q?" H 4450 1950 50  0000 L CNN
 F 1 "CSD17304Q3" H 4300 1850 50  0000 L CNN
-F 2 "Package_SON:VSON-8_3.3x3.3mm_P0.65mm_NexFET" H 4600 1475 50  0001 L CIN
+F 2 "RespiraWorks_Std:VSON-8_3.3x3.3mm_P0.65mm_NexFET" H 4600 1475 50  0001 L CIN
 F 3 "https://www.ti.com/lit/ds/symlink/csd17304q3.pdf?ts=1608773956037" V 4400 1550 50  0001 L CNN
 	1    4400 1550
@@
 F 0 "C?" H 5065 1546 50  0000 L CNN
 F 1 "0.1uF" H 5065 1455 50  0000 L CNN
-F 2 "Capacitor_SMD:C_0603_1608Metric" H 4988 1350 50  0001 C CNN
+F 2 "RespiraWorks_Std:C_0603_1608Metric" H 4988 1350 50  0001 C CNN
 F 3 "~" H 4950 1500 50  0001 C CNN
 	1    4950 1500
@@
 F 0 "Q?" V 4450 1450 50  0000 C CNN
 F 1 "CSD17304Q3" V 4350 1500 50  0000 C CNN
-F 2 "Package_SON:VSON-8_3.3x3.3mm_P0.65mm_NexFET" H 4250 1375 50  0001 L CIN
+F 2 "RespiraWorks_Std:VSON-8_3.3x3.3mm_P0.65mm_NexFET" H 4250 1375 50  0001 L CIN
 F 3 "https://www.ti.com/lit/ds/symlink/csd17304q3.pdf?ts=1608773956037" V 4050 1450 50  0001 L CNN
 	1    4050 1450
@@
 F 0 "U?" H 5400 1850 50  0000 C CNN
 F 1 "LM5141" H 5500 1750 50  0000 C CNN
-F 2 "Package_DFN_QFN:VQFN-24-1EP_4x4mm_P0.5mm_EP2.45x2.45mm_ThermalVias" H 5650 1700 50  0001 C CNN
+F 2 "RespiraWorks_Std:VQFN-24-1EP_4x4mm_P0.5mm_EP2.45x2.45mm_ThermalVias" H 5650 1700 50  0001 C CNN
 F 3 "https://www.ti.com/lit/ds/symlink/lm5141-q1.pdf" H 8450 4600 50  0001 C CNN
 F 4 "Texas Instruments" H 5750 3750 50  0000 C CNN "Manufacturer"
@@
 F 0 "C?" H 7850 4350 50  0000 L CNN
 F 1 "2.2uF" H 7700 4450 50  0000 L CNN
-F 2 "Capacitor_SMD:C_0603_1608Metric" H 8088 4200 50  0001 C CNN
+F 2 "RespiraWorks_Std:C_0603_1608Metric" H 8088 4200 50  0001 C CNN
 F 3 "~" H 8050 4350 50  0001 C CNN
 	1    8050 4350
@@
 F 0 "R?" H 7450 3800 50  0000 L CNN
 F 1 "10k" H 7450 3700 50  0000 L CNN
-F 2 "Resistor_SMD:R_0603_1608Metric" V 7680 3750 50  0001 C CNN
+F 2 "RespiraWorks_Std:C_0603_1608Metric" V 7680 3750 50  0001 C CNN
 F 3 "~" H 7750 3750 50  0001 C CNN
 	1    7750 3750
@@
 F 0 "C?" H 7565 4596 50  0000 L CNN
 F 1 "0.1uF" H 7565 4505 50  0000 L CNN
-F 2 "Capacitor_SMD:C_0603_1608Metric" H 7488 4400 50  0001 C CNN
+F 2 "RespiraWorks_Std:C_0603_1608Metric" H 7488 4400 50  0001 C CNN
 F 3 "~" H 7450 4550 50  0001 C CNN
 	1    7450 4550
@@
 F 0 "R?" H 4700 5350 50  0000 L CNN
 F 1 "56.2k" H 4700 5250 50  0000 L CNN
-F 2 "Resistor_SMD:R_0603_1608Metric" V 4530 5250 50  0001 C CNN
+F 2 "RespiraWorks_Std:C_0603_1608Metric" V 4530 5250 50  0001 C CNN
 F 3 "~" H 4600 5250 50  0001 C CNN
 	1    4600 5250
@@
 F 0 "C?" H 2950 4400 50  0000 L CNN
 F 1 "0.1uF" H 2850 4550 50  0000 L CNN
-F 2 "Capacitor_SMD:C_0603_1608Metric" H 3188 4300 50  0001 C CNN
+F 2 "RespiraWorks_Std:C_0603_1608Metric" H 3188 4300 50  0001 C CNN
 F 3 "~" H 3150 4450 50  0001 C CNN
 	1    3150 4450
@@
 F 0 "R?" H 2300 4850 50  0000 L CNN
 F 1 "6.49k" H 2300 4750 50  0000 L CNN
-F 2 "Resistor_SMD:R_0603_1608Metric" V 2480 4950 50  0001 C CNN
+F 2 "RespiraWorks_Std:C_0603_1608Metric" V 2480 4950 50  0001 C CNN
 F 3 "~" H 2550 4950 50  0001 C CNN
 	1    2550 4950
@@
 F 0 "C?" H 2850 5000 50  0000 L CNN
 F 1 "100pF" H 2850 4700 50  0000 L CNN
-F 2 "Capacitor_SMD:C_0603_1608Metric" H 2838 4700 50  0001 C CNN
+F 2 "RespiraWorks_Std:C_0603_1608Metric" H 2838 4700 50  0001 C CNN
 F 3 "~" H 2800 4850 50  0001 C CNN
 	1    2800 4850
@@
 F 0 "R?" H 1850 4100 50  0000 L CNN
 F 1 "10k" H 1850 4000 50  0000 L CNN
-F 2 "Resistor_SMD:R_0603_1608Metric" V 2080 4050 50  0001 C CNN
+F 2 "RespiraWorks_Std:C_0603_1608Metric" V 2080 4050 50  0001 C CNN
 F 3 "~" H 2150 4050 50  0001 C CNN
 	1    2150 4050
@@
 F 0 "R?" H 1850 3850 50  0000 L CNN
 F 1 "10k" H 1850 3750 50  0000 L CNN
-F 2 "Resistor_SMD:R_0603_1608Metric" V 2080 3750 50  0001 C CNN
+F 2 "RespiraWorks_Std:C_0603_1608Metric" V 2080 3750 50  0001 C CNN
 F 3 "~" H 2150 3750 50  0001 C CNN
 F 4 "DNP" H 1950 3650 50  0000 C CNN "DNP"
@@
 F 0 "C?" H 2300 4850 50  0000 L CNN
 F 1 "2.7nF" H 2300 4750 50  0000 L CNN
-F 2 "Capacitor_SMD:C_0603_1608Metric" H 2588 4500 50  0001 C CNN
+F 2 "RespiraWorks_Std:C_0603_1608Metric" H 2588 4500 50  0001 C CNN
 F 3 "~" H 2550 4650 50  0001 C CNN
 	1    2550 4650
@@
 F 0 "C?" H 3400 4600 50  0000 L CNN
 F 1 "220nF" H 3300 4750 50  0000 L CNN
-F 2 "Capacitor_SMD:C_0603_1608Metric" H 3638 4500 50  0001 C CNN
+F 2 "RespiraWorks_Std:C_0603_1608Metric" H 3638 4500 50  0001 C CNN
 F 3 "~" H 3600 4650 50  0001 C CNN
 	1    3600 4650
@@
 F 0 "C?" H 4000 5000 50  0000 L CNN
 F 1 "220nF" H 3900 5150 50  0000 L CNN
-F 2 "Capacitor_SMD:C_0603_1608Metric" H 4238 4900 50  0001 C CNN
+F 2 "RespiraWorks_Std:C_0603_1608Metric" H 4238 4900 50  0001 C CNN
 F 3 "~" H 4200 5050 50  0001 C CNN
 	1    4200 5050
@@
 F 0 "D?" H 5100 1900 50  0000 C CNN
 F 1 "BAT54J" H 5150 1650 50  0000 C CNN
-F 2 "Diode_SMD:D_SOD-323F" H 5100 1625 50  0001 C CNN
+F 2 "RespiraWorks_Std:D_SOD-323F" H 5100 1625 50  0001 C CNN
 F 3 "https://assets.nexperia.com/documents/data-sheet/BAT54J.pdf" H 5100 1800 50  0001 C CNN
 	1    5100 1800
@@
 F 0 "R?" V 4650 2300 50  0000 L CNN
 F 1 "10" V 4650 2700 50  0000 L CNN
-F 2 "Resistor_SMD:R_0603_1608Metric" V 4630 2550 50  0001 C CNN
+F 2 "RespiraWorks_Std:C_0603_1608Metric" V 4630 2550 50  0001 C CNN
 F 3 "~" H 4700 2550 50  0001 C CNN
 	1    4700 2550
@@
 F 0 "Q?" H 3091 3146 50  0000 L CNN
 F 1 "MMBT3904" H 3091 3055 50  0000 L CNN
-F 2 "Package_TO_SOT_SMD:SOT-23" H 3100 3025 50  0001 L CIN
+F 2 "RespiraWorks_Std:SOT-23" H 3100 3025 50  0001 L CIN
 F 3 "https://www.onsemi.com/pub/Collateral/2N3903-D.PDF" H 2900 3100 50  0001 L CNN
 	1    2900 3100
@@
 F 0 "R?" H 2700 2700 50  0000 L CNN
 F 1 "10k" H 2700 2600 50  0000 L CNN
-F 2 "Resistor_SMD:R_0603_1608Metric" V 2930 2650 50  0001 C CNN
+F 2 "RespiraWorks_Std:R_0603_1608Metric" V 2930 2650 50  0001 C CNN
 F 3 "~" H 3000 2650 50  0001 C CNN
 	1    3000 2650
@@
 F 0 "R?" V 1950 3050 50  0000 L CNN
 F 1 "10k" V 2050 3050 50  0000 L CNN
-F 2 "Resistor_SMD:R_0603_1608Metric" V 2080 3100 50  0001 C CNN
+F 2 "RespiraWorks_Std:C_0603_1608Metric" V 2080 3100 50  0001 C CNN
 F 3 "~" H 2150 3100 50  0001 C CNN
 	1    2150 3100

Commit message: inductor footprint assignments
Parts:
- L?: footprint Inductor_SMD:L_TDK_SLF12565 -> RespiraWorks:L_TDK_SPM12565VT
Changed lines of the file:
@@
 F 0 "L?" H 5750 1650 50  0000 C CNN
 F 1 "6.8uH" H 5750 1550 50  0000 C CNN
-F 2 "Inductor_SMD:L_TDK_SLF12565" V 5750 1350 50  0001 C CNN
+F 2 "RespiraWorks:L_TDK_SPM12565VT" V 5750 1350 50  0001 C CNN
 F 3 "https://product.tdk.com/info/en/catalog/datasheets/inductor_automotive_power_spm12565vt-d_en.pdf" V 5750 1350 50  0001 C CNN
 F 4 "TDK" H 5750 1350 50  0001 C CNN "Manufacturer"

Commit message: Top-level beginnings, minor fixes
Started on top-level schematic blocks and connections
Started changing some net names to mixed-case-with-dash format
Fixed version number, added titles and version to all schematic sheets
Fixed incorrect SWO pin assignment in cycle controller
Added a few add'l annotations to battery sheets
Other:
- note added: "220nF modulates fsw +/- 5% @ ~~380 Hz"
- note added: "440 kHz fsw nominal"
- note added: "56.2K fine-tunes fsw = 436 kHz nominal"
- note added: "Diode emulation mode\n@ light load"
- note added: "Forced-PWM CCM mode\n@ light load"
- note added: "Soft-start time = 1.2V*100nF/20uA = 6 ms"
