File: pcb/power_vsys.sch (KiCad schematic (older format))
At the start: 34 parts

Commit message: CC-I2C, BOM
Added missing pull-ups on CC-SDA, CC-SCL
First pass at BOM consolidation
Parts:
- C? (x3): value 0.1uF -> 100nF
- C?: footprint RespiraWorks_Std:C_0603_1608Metric -> RespiraWorks_Std:C_1206_3216Metric
- R? (x8): footprint RespiraWorks_Std:C_0603_1608Metric -> RespiraWorks_Std:R_0603_1608Metric
- R?: value 10.1k -> 10k; footprint RespiraWorks_Std:C_0603_1608Metric -> RespiraWorks_Std:R_0603_1608Metric
- R?: value 56.2k -> 52.3k; footprint RespiraWorks_Std:C_0603_1608Metric -> RespiraWorks_Std:R_0603_1608Metric
Other:
- note added: "53.2k fine-tunes fsw = 422 kHz nominal"
- note removed: "56.2K fine-tunes fsw = 436 kHz nominal"
Changed lines of the file:
@@
 F 0 "R?" V 4650 2700 50  0000 L CNN
 F 1 "10" V 4650 3100 50  0000 L CNN
-F 2 "RespiraWorks_Std:C_0603_1608Metric" V 4630 2950 50  0001 C CNN
+F 2 "RespiraWorks_Std:R_0603_1608Metric" V 4630 2950 50  0001 C CNN
 F 3 "~" H 4700 2950 50  0001 C CNN
 	1    4700 2950
@@
 F 0 "R?" H 6950 2850 50  0000 L CNN
 F 1 "90.9k" H 6950 2750 50  0000 L CNN
-F 2 "RespiraWorks_Std:C_0603_1608Metric" V 7180 2800 50  0001 C CNN
+F 2 "RespiraWorks_Std:R_0603_1608Metric" V 7180 2800 50  0001 C CNN
 F 3 "~" H 7250 2800 50  0001 C CNN
 	1    7250 2800
@@
 AR Path="/6041384A/60567D6E/601F52A9" Ref="R?"  Part="1"
 F 0 "R?" H 6950 3150 50  0000 L CNN
-F 1 "10.1k" H 6950 3050 50  0000 L CNN
-F 2 "RespiraWorks_Std:C_0603_1608Metric" V 7180 3100 50  0001 C CNN
+F 1 "10k" H 6950 3050 50  0000 L CNN
+F 2 "RespiraWorks_Std:R_0603_1608Metric" V 7180 3100 50  0001 C CNN
 F 3 "~" H 7250 3100 50  0001 C CNN
 	1    7250 3100
@@
 AR Path="/6041384A/60567D6E/601DFDEE" Ref="C?"  Part="1"
 F 0 "C?" H 5065 1546 50  0000 L CNN
-F 1 "0.1uF" H 5065 1455 50  0000 L CNN
+F 1 "100nF" H 5065 1455 50  0000 L CNN
 F 2 "RespiraWorks_Std:C_0603_1608Metric" H 4988 1350 50  0001 C CNN
 F 3 "~" H 4950 1500 50  0001 C CNN
@@
 F 0 "C?" H 7850 4350 50  0000 L CNN
 F 1 "2.2uF" H 7700 4450 50  0000 L CNN
-F 2 "RespiraWorks_Std:C_0603_1608Metric" H 8088 4200 50  0001 C CNN
+F 2 "RespiraWorks_Std:C_1206_3216Metric" H 8088 4200 50  0001 C CNN
 F 3 "~" H 8050 4350 50  0001 C CNN
 	1    8050 4350
@@
 F 0 "R?" H 7450 3800 50  0000 L CNN
 F 1 "10k" H 7450 3700 50  0000 L CNN
-F 2 "RespiraWorks_Std:C_0603_1608Metric" V 7680 3750 50  0001 C CNN
+F 2 "RespiraWorks_Std:R_0603_1608Metric" V 7680 3750 50  0001 C CNN
 F 3 "~" H 7750 3750 50  0001 C CNN
 	1    7750 3750
@@
 AR Path="/6041384A/60567D6E/602371E3" Ref="C?"  Part="1"
 F 0 "C?" H 7565 4596 50  0000 L CNN
-F 1 "0.1uF" H 7565 4505 50  0000 L CNN
+F 1 "100nF" H 7565 4505 50  0000 L CNN
 F 2 "RespiraWorks_Std:C_0603_1608Metric" H 7488 4400 50  0001 C CNN
 F 3 "~" H 7450 4550 50  0001 C CNN
@@
 AR Path="/6041384A/60567D6E/60263CF0" Ref="R?"  Part="1"
 F 0 "R?" H 4700 5350 50  0000 L CNN
-F 1 "56.2k" H 4700 5250 50  0000 L CNN
-F 2 "RespiraWorks_Std:C_0603_1608Metric" V 4530 5250 50  0001 C CNN
+F 1 "52.3k" H 4700 5250 50  0000 L CNN
+F 2 "RespiraWorks_Std:R_0603_1608Metric" V 4530 5250 50  0001 C CNN
 F 3 "~" H 4600 5250 50  0001 C CNN
 	1    4600 5250
@@
 AR Path="/6041384A/60567D6E/6025AFE5" Ref="C?"  Part="1"
 F 0 "C?" H 2950 4400 50  0000 L CNN
-F 1 "0.1uF" H 2850 4550 50  0000 L CNN
+F 1 "100nF" H 2850 4550 50  0000 L CNN
 F 2 "RespiraWorks_Std:C_0603_1608Metric" H 3188 4300 50  0001 C CNN
 F 3 "~" H 3150 4450 50  0001 C CNN
@@
 F 0 "R?" H 2300 4850 50  0000 L CNN
 F 1 "6.49k" H 2300 4750 50  0000 L CNN
-F 2 "RespiraWorks_Std:C_0603_1608Metric" V 2480 4950 50  0001 C CNN
+F 2 "RespiraWorks_Std:R_0603_1608Metric" V 2480 4950 50  0001 C CNN
 F 3 "~" H 2550 4950 50  0001 C CNN
 	1    2550 4950
@@
 F 0 "R?" H 1850 4100 50  0000 L CNN
 F 1 "10k" H 1850 4000 50  0000 L CNN
-F 2 "RespiraWorks_Std:C_0603_1608Metric" V 2080 4050 50  0001 C CNN
+F 2 "RespiraWorks_Std:R_0603_1608Metric" V 2080 4050 50  0001 C CNN
 F 3 "~" H 2150 4050 50  0001 C CNN
 	1    2150 4050
@@
 F 0 "R?" H 1850 3850 50  0000 L CNN
 F 1 "10k" H 1850 3750 50  0000 L CNN
-F 2 "RespiraWorks_Std:C_0603_1608Metric" V 2080 3750 50  0001 C CNN
+F 2 "RespiraWorks_Std:R_0603_1608Metric" V 2080 3750 50  0001 C CNN
 F 3 "~" H 2150 3750 50  0001 C CNN
 F 4 "DNP" H 1950 3650 50  0000 C CNN "DNP"
@@
 F 0 "R?" V 4650 2300 50  0000 L CNN
 F 1 "10" V 4650 2700 50  0000 L CNN
-F 2 "RespiraWorks_Std:C_0603_1608Metric" V 4630 2550 50  0001 C CNN
+F 2 "RespiraWorks_Std:R_0603_1608Metric" V 4630 2550 50  0001 C CNN
 F 3 "~" H 4700 2550 50  0001 C CNN
 	1    4700 2550
@@
 F 0 "R?" V 1950 3050 50  0000 L CNN
 F 1 "10k" V 2050 3050 50  0000 L CNN
-F 2 "RespiraWorks_Std:C_0603_1608Metric" V 2080 3100 50  0001 C CNN
+F 2 "RespiraWorks_Std:R_0603_1608Metric" V 2080 3100 50  0001 C CNN
 F 3 "~" H 2150 3100 50  0001 C CNN
 	1    2150 3100
@@
 220nF modulates fsw +/- 5% @ ~~380 Hz
 Text Notes 4500 5550 0    50   ~ 0
-56.2K fine-tunes fsw = 436 kHz nominal
+53.2k fine-tunes fsw = 422 kHz nominal
 Text Notes 3100 4300 0    50   ~ 0
 Soft-start time = 1.2V*100nF/20uA = 6 ms

Commit message: BOM
More BOM consolidation with bulk capacitors + changed tantalum stepper caps to aluminum, added bulk cap to PSol driver
Made stepper's 3.3V power naming consistent with others (3.3V->3V3)
Slightly increased current limit on PSOL/heater driver
Changed 3906 transistors to 2907 to better support +5V_Batt current
Parts:
- removed C?: 2.2uF, RespiraWorks_Std:C_1206_3216Metric, symbol Device:C
- added C? (x2): 1uF, RespiraWorks_Std:C_0603_1608Metric, symbol Device:C
- added R?: 1M, RespiraWorks_Std:R_0603_1608Metric, symbol Device:R
- C? (x6): footprint RespiraWorks_Std:C_0805_2012Metric -> RespiraWorks_Std:C_1210_3225Metric; Dielectric X5R -> X7S; Manufacturer (none) -> Murata; Manufacturer PN (none) -> GRM32EC72A106KE05L; Voltage 35V -> 100V
- C?: value 33pF -> 100pF
- L?: Manufacturer PN (none) -> SPM12565VT-6R8M-D; manufacturer PN SPM12565VT-6R8M-D -> (none)
- NT?: footprint (none) -> RespiraWorks_Std:NetTie-2_SMD_Pad0.5mm
- R?: value 90.9k -> 100k
Connections:
- wire segments 96 -> 102
Other:
- note added: "= 90.9k,\nto reduce BOM"
- note added: "Regulates @ FB = 1.2V;\nNom. 12.1V out"
- moved on the sheet: R?
Changed lines of the file:
@@
 L Device:R R?
 U 1 1 601F467D
-P 7250 2800
+P 7250 2650
 AR Path="/601A64F8/601F467D" Ref="R?"  Part="1"
 AR Path="/601A64F8/60567144/601F467D" Ref="R?"  Part="1"
@@
 AR Path="/6023BF6A/60567D6E/601F467D" Ref="R?"  Part="1"
 AR Path="/6041384A/60567D6E/601F467D" Ref="R?"  Part="1"
-F 0 "R?" H 6950 2850 50  0000 L CNN
-F 1 "90.9k" H 6950 2750 50  0000 L CNN
-F 2 "RespiraWorks_Std:R_0603_1608Metric" V 7180 2800 50  0001 C CNN
-F 3 "~" H 7250 2800 50  0001 C CNN
-	1    7250 2800
+F 0 "R?" H 6950 2700 50  0000 L CNN
+F 1 "100k" H 6950 2600 50  0000 L CNN
+F 2 "RespiraWorks_Std:R_0603_1608Metric" V 7180 2650 50  0001 C CNN
+F 3 "~" H 7250 2650 50  0001 C CNN
+	1    7250 2650
 	1    0    0    -1
 $EndComp
@@
 F 0 "C?" H 8450 1400 50  0000 L CNN
 F 1 "10uF" H 8450 1300 50  0000 L CNN
-F 2 "RespiraWorks_Std:C_0805_2012Metric" H 8438 1350 50  0001 C CNN
+F 2 "RespiraWorks_Std:C_1210_3225Metric" H 8438 1350 50  0001 C CNN
 F 3 "~" H 8400 1500 50  0001 C CNN
-F 4 "35V" H 8450 1200 50  0000 L CNN "Voltage"
-F 5 "X5R" H 8400 1500 50  0001 C CNN "Dielectric"
+F 4 "100V" H 8450 1200 50  0000 L CNN "Voltage"
+F 5 "X7S" H 8400 1500 50  0001 C CNN "Dielectric"
+F 6 "Murata" H 8400 1500 50  0001 C CNN "Manufacturer"
+F 7 "GRM32EC72A106KE05L" H 8400 1500 50  0001 C CNN "Manufacturer PN"
 	1    8400 1500
 	1    0    0    -1
@@
 F 0 "C?" H 8150 1400 50  0000 L CNN
 F 1 "10uF" H 8150 1300 50  0000 L CNN
-F 2 "RespiraWorks_Std:C_0805_2012Metric" H 8138 1350 50  0001 C CNN
+F 2 "RespiraWorks_Std:C_1210_3225Metric" H 8138 1350 50  0001 C CNN
 F 3 "~" H 8100 1500 50  0001 C CNN
-F 4 "35V" H 8150 1200 50  0000 L CNN "Voltage"
-F 5 "X5R" H 8100 1500 50  0001 C CNN "Dielectric"
+F 4 "100V" H 8150 1200 50  0000 L CNN "Voltage"
+F 5 "X7S" H 8100 1500 50  0001 C CNN "Dielectric"
+F 6 "Murata" H 8100 1500 50  0001 C CNN "Manufacturer"
+F 7 "GRM32EC72A106KE05L" H 8100 1500 50  0001 C CNN "Manufacturer PN"
 	1    8100 1500
 	1    0    0    -1
@@
 F 0 "C?" H 7850 1400 50  0000 L CNN
 F 1 "10uF" H 7850 1300 50  0000 L CNN
-F 2 "RespiraWorks_Std:C_0805_2012Metric" H 7838 1350 50  0001 C CNN
+F 2 "RespiraWorks_Std:C_1210_3225Metric" H 7838 1350 50  0001 C CNN
 F 3 "~" H 7800 1500 50  0001 C CNN
-F 4 "35V" H 7850 1200 50  0000 L CNN "Voltage"
-F 5 "X5R" H 7800 1500 50  0001 C CNN "Dielectric"
+F 4 "100V" H 7850 1200 50  0000 L CNN "Voltage"
+F 5 "X7S" H 7800 1500 50  0001 C CNN "Dielectric"
+F 6 "Murata" H 7800 1500 50  0001 C CNN "Manufacturer"
+F 7 "GRM32EC72A106KE05L" H 7800 1500 50  0001 C CNN "Manufacturer PN"
 	1    7800 1500
 	1    0    0    -1
@@
 F 0 "C?" H 7550 1400 50  0000 L CNN
 F 1 "10uF" H 7550 1300 50  0000 L CNN
-F 2 "RespiraWorks_Std:C_0805_2012Metric" H 7538 1350 50  0001 C CNN
+F 2 "RespiraWorks_Std:C_1210_3225Metric" H 7538 1350 50  0001 C CNN
 F 3 "~" H 7500 1500 50  0001 C CNN
-F 4 "35V" H 7550 1200 50  0000 L CNN "Voltage"
-F 5 "X5R" H 7500 1500 50  0001 C CNN "Dielectric"
+F 4 "100V" H 7550 1200 50  0000 L CNN "Voltage"
+F 5 "X7S" H 7500 1500 50  0001 C CNN "Dielectric"
+F 6 "Murata" H 7500 1500 50  0001 C CNN "Manufacturer"
+F 7 "GRM32EC72A106KE05L" H 7500 1500 50  0001 C CNN "Manufacturer PN"
 	1    7500 1500
 	1    0    0    -1
@@
 	7250 1350 7500 1350
 Wire Wire Line
-	7250 1350 7250 2650
+	7250 1350 7250 2500
 Wire Wire Line
 	4200 1550 4200 2750
@@
 AR Path="/6041384A/60567D6E/601ED324" Ref="C?"  Part="1"
 F 0 "C?" V 6600 1700 50  0000 L CNN
-F 1 "33pF" V 6500 1600 50  0000 L CNN
+F 1 "100pF" V 6500 1550 50  0000 L CNN
 F 2 "RespiraWorks_Std:C_0603_1608Metric" H 6788 1500 50  0001 C CNN
 F 3 "~" H 6750 1650 50  0001 C CNN
@@
 F 0 "C?" H 3500 1400 50  0000 L CNN
 F 1 "10uF" H 3500 1300 50  0000 L CNN
-F 2 "RespiraWorks_Std:C_0805_2012Metric" H 3488 1350 50  0001 C CNN
+F 2 "RespiraWorks_Std:C_1210_3225Metric" H 3488 1350 50  0001 C CNN
 F 3 "~" H 3450 1500 50  0001 C CNN
-F 4 "35V" H 3500 1200 50  0000 L CNN "Voltage"
-F 5 "X5R" H 3450 1500 50  0001 C CNN "Dielectric"
+F 4 "100V" H 3500 1200 50  0000 L CNN "Voltage"
+F 5 "X7S" H 3450 1500 50  0001 C CNN "Dielectric"
+F 6 "Murata" H 3450 1500 50  0001 C CNN "Manufacturer"
+F 7 "GRM32EC72A106KE05L" H 3450 1500 50  0001 C CNN "Manufacturer PN"
 	1    3450 1500
 	1    0    0    -1
@@
 F 0 "C?" H 3200 1400 50  0000 L CNN
 F 1 "10uF" H 3200 1300 50  0000 L CNN
-F 2 "RespiraWorks_Std:C_0805_2012Metric" H 3188 1350 50  0001 C CNN
+F 2 "RespiraWorks_Std:C_1210_3225Metric" H 3188 1350 50  0001 C CNN
 F 3 "~" H 3150 1500 50  0001 C CNN
-F 4 "35V" H 3200 1200 50  0000 L CNN "Voltage"
-F 5 "X5R" H 3150 1500 50  0001 C CNN "Dielectric"
+F 4 "100V" H 3200 1200 50  0000 L CNN "Voltage"
+F 5 "X7S" H 3150 1500 50  0001 C CNN "Dielectric"
+F 6 "Murata" H 3150 1500 50  0001 C CNN "Manufacturer"
+F 7 "GRM32EC72A106KE05L" H 3150 1500 50  0001 C CNN "Manufacturer PN"
 	1    3150 1500
 	1    0    0    -1
@@
 F 3 "https://product.tdk.com/info/en/catalog/datasheets/inductor_automotive_power_spm12565vt-d_en.pdf" V 5750 1350 50  0001 C CNN
 F 4 "TDK" H 5750 1350 50  0001 C CNN "Manufacturer"
-F 5 "SPM12565VT-6R8M-D" H 5800 1450 50  0000 C CNN "manufacturer PN"
+F 5 "SPM12565VT-6R8M-D" H 5800 1450 50  0000 C CNN "Manufacturer PN"
 	1    5750 1350
 	1    0    0    -1
@@
 Wire Wire Line
 	6450 4200 8050 4200
-$Comp
-L Device:C C?
-U 1 1 6022668B
-P 8050 4350
-AR Path="/601A64F8/6022668B" Ref="C?"  Part="1"
-AR Path="/601A64F8/60567144/6022668B" Ref="C?"  Part="1"
-AR Path="/601A64F8/60567D6E/6022668B" Ref="C?"  Part="1"
-AR Path="/6023BF6A/60567D6E/6022668B" Ref="C?"  Part="1"
-AR Path="/6041384A/60567D6E/6022668B" Ref="C?"  Part="1"
-F 0 "C?" H 7850 4350 50  0000 L CNN
-F 1 "2.2uF" H 7700 4450 50  0000 L CNN
-F 2 "RespiraWorks_Std:C_1206_3216Metric" H 8088 4200 50  0001 C CNN
-F 3 "~" H 8050 4350 50  0001 C CNN
-	1    8050 4350
-	-1   0    0    1
-$EndComp
-$Comp
-L power:GND #PWR?
-U 1 1 602277DB
-P 8050 4500
-AR Path="/601A64F8/602277DB" Ref="#PWR?"  Part="1"
-AR Path="/601A64F8/60567144/602277DB" Ref="#PWR?"  Part="1"
-AR Path="/601A64F8/60567D6E/602277DB" Ref="#PWR?"  Part="1"
-AR Path="/6023BF6A/60567D6E/602277DB" Ref="#PWR?"  Part="1"
-AR Path="/6041384A/60567D6E/602277DB" Ref="#PWR?"  Part="1"
-F 0 "#PWR?" H 8050 4250 50  0001 C CNN
-F 1 "GND" H 8055 4327 50  0000 C CNN
-F 2 "" H 8050 4500 50  0001 C CNN
-F 3 "" H 8050 4500 50  0001 C CNN
-	1    8050 4500
-	1    0    0    -1
-$EndComp
 $Comp
 L Device:R R?
@@
 F 0 "NT?" V 7150 4900 50  0000 C CNN
 F 1 "Net-Tie_2" H 7100 4850 50  0001 C CNN
-F 2 "" H 7150 4800 50  0001 C CNN
+F 2 "RespiraWorks_Std:NetTie-2_SMD_Pad0.5mm" H 7150 4800 50  0001 C CNN
 F 3 "~" H 7150 4800 50  0001 C CNN
 	1    7150 4800
@@
 Text Notes 3100 4300 0    50   ~ 0
 Soft-start time = 1.2V*100nF/20uA = 6 ms
+$Comp
+L Device:C C?
+U 1 1 6043B4C4
+P 8050 4350
+AR Path="/5FCD4B8E/5FCD4BC5/6043B4C4" Ref="C?"  Part="1"
+AR Path="/5FCD4B8E/5FE27F70/6043B4C4" Ref="C?"  Part="1"
+AR Path="/6041384A/60567D6E/6043B4C4" Ref="C?"  Part="1"
+F 0 "C?" H 7900 4450 50  0000 L CNN
+F 1 "1uF" H 7850 4550 50  0000 L CNN
+F 2 "RespiraWorks_Std:C_0603_1608Metric" H 8088 4200 50  0001 C CNN
+F 3 "~" H 8050 4350 50  0001 C CNN
+F 4 "AVX" H 8050 4350 50  0001 C CNN "Manufacturer"
+	1    8050 4350
+	-1   0    0    1
+$EndComp
+$Comp
+L power:GND #PWR?
+U 1 1 6043B4CA
+P 8050 4500
+AR Path="/5FCD4B8E/5FCD4BC5/6043B4CA" Ref="#PWR?"  Part="1"
+AR Path="/5FCD4B8E/5FE27F70/6043B4CA" Ref="#PWR?"  Part="1"
+AR Path="/6041384A/60567D6E/6043B4CA" Ref="#PWR?"  Part="1"
+F 0 "#PWR?" H 8050 4250 50  0001 C CNN
+F 1 "GND" H 8055 4327 50  0000 C CNN
+F 2 "" H 8050 4500 50  0001 C CNN
+F 3 "" H 8050 4500 50  0001 C CNN
+	1    8050 4500
+	1    0    0    -1
+$EndComp
+$Comp
+L Device:C C?
+U 1 1 60449E4F
+P 8450 4350
+AR Path="/5FCD4B8E/5FCD4BC5/60449E4F" Ref="C?"  Part="1"
+AR Path="/5FCD4B8E/5FE27F70/60449E4F" Ref="C?"  Part="1"
+AR Path="/6041384A/60567D6E/60449E4F" Ref="C?"  Part="1"
+F 0 "C?" H 8300 4450 50  0000 L CNN
+F 1 "1uF" H 8250 4550 50  0000 L CNN
+F 2 "RespiraWorks_Std:C_0603_1608Metric" H 8488 4200 50  0001 C CNN
+F 3 "~" H 8450 4350 50  0001 C CNN
+F 4 "AVX" H 8450 4350 50  0001 C CNN "Manufacturer"
+	1    8450 4350
+	-1   0    0    1
+$EndComp
+$Comp
+L power:GND #PWR?
+U 1 1 60449E55
+P 8450 4500
+AR Path="/5FCD4B8E/5FCD4BC5/60449E55" Ref="#PWR?"  Part="1"
+AR Path="/5FCD4B8E/5FE27F70/60449E55" Ref="#PWR?"  Part="1"
+AR Path="/6041384A/60567D6E/60449E55" Ref="#PWR?"  Part="1"
+F 0 "#PWR?" H 8450 4250 50  0001 C CNN
+F 1 "GND" H 8455 4327 50  0000 C CNN
+F 2 "" H 8450 4500 50  0001 C CNN
+F 3 "" H 8450 4500 50  0001 C CNN
+	1    8450 4500
+	1    0    0    -1
+$EndComp
+Wire Wire Line
+	8050 4200 8450 4200
+Connection ~ 8050 4200
+$Comp
+L Device:R R?
+U 1 1 60564CB5
+P 7450 2650
+AR Path="/601A64F8/60564CB5" Ref="R?"  Part="1"
+AR Path="/601A64F8/60567144/60564CB5" Ref="R?"  Part="1"
+AR Path="/601A64F8/60567D6E/60564CB5" Ref="R?"  Part="1"
+AR Path="/6023BF6A/60567D6E/60564CB5" Ref="R?"  Part="1"
+AR Path="/6041384A/60567D6E/60564CB5" Ref="R?"  Part="1"
+F 0 "R?" H 7250 2700 50  0000 L CNN
+F 1 "1M" H 7250 2600 50  0000 L CNN
+F 2 "RespiraWorks_Std:R_0603_1608Metric" V 7380 2650 50  0001 C CNN
+F 3 "~" H 7450 2650 50  0001 C CNN
+	1    7450 2650
+	-1   0    0    -1
+$EndComp
+Wire Wire Line
+	7450 2500 7250 2500
+Connection ~ 7250 2500
+Wire Wire Line
+	7250 2800 7250 2850
+Wire Wire Line
+	7250 2850 7450 2850
+Wire Wire Line
+	7450 2850 7450 2800
+Connection ~ 7250 2850
+Wire Wire Line
+	7250 2850 7250 2950
+Text Notes 7350 2450 0    50   ~ 0
+= 90.9k,\nto reduce BOM
+Text Notes 7400 3100 0    50   ~ 0
+Regulates @ FB = 1.2V;\nNom. 12.1V out
 $EndSCHEMATC

Commit message: BOM, fixes
Finished assigning parts, footprints except generic resistors
Added series resistors for logic signals received by UI computer to protect against UI computer power-down
Added tolerance notes on main schem
Replaced PSol fuse with PTC
Enlarged PSol driver bypass resistors to 0 ohm
Changed PSol unpopulated current-limiting resistor to divider
Parts:
- C? (x3): Dielectric (none) -> X7R; Manufacturer (none) -> Kemet; Manufacturer PN (none) -> C0603C104K5RACTU; Voltage (none) -> 50V
- C? (x2): Dielectric (none) -> NP0; Manufacturer (none) -> Kemet; Manufacturer PN (none) -> C0603C101J5GACTU; Voltage (none) -> 50V
- C?: Dielectric (none) -> NP0; Manufacturer (none) -> Kemet; Manufacturer PN (none) -> C0603C272J5GACTU; Voltage (none) -> 50V
- C? (x2): footprint RespiraWorks_Std:C_0603_1608Metric -> RespiraWorks_Std:C_0805_2012Metric; Dielectric (none) -> X7R; Manufacturer (none) -> Kemet; Manufacturer PN (none) -> C0805C224K1RACTU; Voltage (none) -> 100V
- C? (x2): Dielectric (none) -> X7R; Manufacturer AVX -> Kemet; Manufacturer PN (none) -> C0805C105K5RACTU; Voltage (none) -> 50V
- D?: Manufacturer (none) -> Nexperia; Manufacturer PN (none) -> BAT54J,115
- Q? (x2): Manufacturer (none) -> Texas Instruments; Manufacturer PN (none) -> CSD17304Q3
- Q?: Manufacturer (none) -> Diodes Inc.; Manufacturer PN (none) -> MMBT3904-7-F
Changed lines of the file:
@@
 F 2 "RespiraWorks_Std:C_0603_1608Metric" H 6788 1500 50  0001 C CNN
 F 3 "~" H 6750 1650 50  0001 C CNN
+F 4 "NP0" H 6750 1650 50  0001 C CNN "Dielectric"
+F 5 "Kemet" H 6750 1650 50  0001 C CNN "Manufacturer"
+F 6 "C0603C101J5GACTU" H 6750 1650 50  0001 C CNN "Manufacturer PN"
+F 7 "50V" H 6750 1650 50  0001 C CNN "Voltage"
 	1    6750 1650
 	0    -1   -1   0
@@
 F 2 "RespiraWorks_Std:VSON-8_3.3x3.3mm_P0.65mm_NexFET" H 4600 1475 50  0001 L CIN
 F 3 "https://www.ti.com/lit/ds/symlink/csd17304q3.pdf?ts=1608773956037" V 4400 1550 50  0001 L CNN
+F 4 "Texas Instruments" H 4400 1550 50  0001 C CNN "Manufacturer"
+F 5 "CSD17304Q3" H 4400 1550 50  0001 C CNN "Manufacturer PN"
 	1    4400 1550
 	1    0    0    -1
@@
 F 2 "RespiraWorks_Std:C_0603_1608Metric" H 4988 1350 50  0001 C CNN
 F 3 "~" H 4950 1500 50  0001 C CNN
+F 4 "X7R" H 4950 1500 50  0001 C CNN "Dielectric"
+F 5 "Kemet" H 4950 1500 50  0001 C CNN "Manufacturer"
+F 6 "C0603C104K5RACTU" H 4950 1500 50  0001 C CNN "Manufacturer PN"
+F 7 "50V" H 4950 1500 50  0001 C CNN "Voltage"
 	1    4950 1500
 	1    0    0    -1
@@
 F 2 "RespiraWorks_Std:VSON-8_3.3x3.3mm_P0.65mm_NexFET" H 4250 1375 50  0001 L CIN
 F 3 "https://www.ti.com/lit/ds/symlink/csd17304q3.pdf?ts=1608773956037" V 4050 1450 50  0001 L CNN
+F 4 "Texas Instruments" H 4050 1450 50  0001 C CNN "Manufacturer"
+F 5 "CSD17304Q3" H 4050 1450 50  0001 C CNN "Manufacturer PN"
 	1    4050 1450
 	0    -1   -1   0
@@
 F 2 "RespiraWorks_Std:C_0603_1608Metric" H 7488 4400 50  0001 C CNN
 F 3 "~" H 7450 4550 50  0001 C CNN
+F 4 "X7R" H 7450 4550 50  0001 C CNN "Dielectric"
+F 5 "Kemet" H 7450 4550 50  0001 C CNN "Manufacturer"
+F 6 "C0603C104K5RACTU" H 7450 4550 50  0001 C CNN "Manufacturer PN"
+F 7 "50V" H 7450 4550 50  0001 C CNN "Voltage"
 	1    7450 4550
 	1    0    0    -1
@@
 F 2 "RespiraWorks_Std:C_0603_1608Metric" H 3188 4300 50  0001 C CNN
 F 3 "~" H 3150 4450 50  0001 C CNN
+F 4 "X7R" H 3150 4450 50  0001 C CNN "Dielectric"
+F 5 "Kemet" H 3150 4450 50  0001 C CNN "Manufacturer"
+F 6 "C0603C104K5RACTU" H 3150 4450 50  0001 C CNN "Manufacturer PN"
+F 7 "50V" H 3150 4450 50  0001 C CNN "Voltage"
 	1    3150 4450
 	-1   0    0    1
@@
 F 2 "RespiraWorks_Std:C_0603_1608Metric" H 2838 4700 50  0001 C CNN
 F 3 "~" H 2800 4850 50  0001 C CNN
+F 4 "NP0" H 2800 4850 50  0001 C CNN "Dielectric"
+F 5 "Kemet" H 2800 4850 50  0001 C CNN "Manufacturer"
+F 6 "C0603C101J5GACTU" H 2800 4850 50  0001 C CNN "Manufacturer PN"
+F 7 "50V" H 2800 4850 50  0001 C CNN "Voltage"
 	1    2800 4850
 	1    0    0    -1
@@
 F 2 "RespiraWorks_Std:C_0603_1608Metric" H 2588 4500 50  0001 C CNN
 F 3 "~" H 2550 4650 50  0001 C CNN
+F 4 "NP0" H 2550 4650 50  0001 C CNN "Dielectric"
+F 5 "Kemet" H 2550 4650 50  0001 C CNN "Manufacturer"
+F 6 "C0603C272J5GACTU" H 2550 4650 50  0001 C CNN "Manufacturer PN"
+F 7 "50V" H 2550 4650 50  0001 C CNN "Voltage"
 	1    2550 4650
 	1    0    0    -1
@@
 F 0 "C?" H 3400 4600 50  0000 L CNN
 F 1 "220nF" H 3300 4750 50  0000 L CNN
-F 2 "RespiraWorks_Std:C_0603_1608Metric" H 3638 4500 50  0001 C CNN
+F 2 "RespiraWorks_Std:C_0805_2012Metric" H 3638 4500 50  0001 C CNN
 F 3 "~" H 3600 4650 50  0001 C CNN
+F 4 "X7R" H 3600 4650 50  0001 C CNN "Dielectric"
+F 5 "Kemet" H 3600 4650 50  0001 C CNN "Manufacturer"
+F 6 "C0805C224K1RACTU" H 3600 4650 50  0001 C CNN "Manufacturer PN"
+F 7 "100V" H 3600 4650 50  0001 C CNN "Voltage"
 	1    3600 4650
 	-1   0    0    1
@@
 F 0 "C?" H 4000 5000 50  0000 L CNN
 F 1 "220nF" H 3900 5150 50  0000 L CNN
-F 2 "RespiraWorks_Std:C_0603_1608Metric" H 4238 4900 50  0001 C CNN
+F 2 "RespiraWorks_Std:C_0805_2012Metric" H 4238 4900 50  0001 C CNN
 F 3 "~" H 4200 5050 50  0001 C CNN
+F 4 "X7R" H 4200 5050 50  0001 C CNN "Dielectric"
+F 5 "Kemet" H 4200 5050 50  0001 C CNN "Manufacturer"
+F 6 "C0805C224K1RACTU" H 4200 5050 50  0001 C CNN "Manufacturer PN"
+F 7 "100V" H 4200 5050 50  0001 C CNN "Voltage"
 	1    4200 5050
 	-1   0    0    1
@@
 F 2 "RespiraWorks_Std:D_SOD-323F" H 5100 1625 50  0001 C CNN
 F 3 "https://assets.nexperia.com/documents/data-sheet/BAT54J.pdf" H 5100 1800 50  0001 C CNN
+F 4 "Nexperia" H 5100 1800 50  0001 C CNN "Manufacturer"
+F 5 "BAT54J,115" H 5100 1800 50  0001 C CNN "Manufacturer PN"
 	1    5100 1800
 	1    0    0    -1
@@
 F 2 "RespiraWorks_Std:SOT-23" H 3100 3025 50  0001 L CIN
 F 3 "https://www.onsemi.com/pub/Collateral/2N3903-D.PDF" H 2900 3100 50  0001 L CNN
+F 4 "Diodes Inc." H 2900 3100 50  0001 C CNN "Manufacturer"
+F 5 "MMBT3904-7-F" H 2900 3100 50  0001 C CNN "Manufacturer PN"
 	1    2900 3100
 	1    0    0    -1
@@
 F 2 "RespiraWorks_Std:C_0603_1608Metric" H 8088 4200 50  0001 C CNN
 F 3 "~" H 8050 4350 50  0001 C CNN
-F 4 "AVX" H 8050 4350 50  0001 C CNN "Manufacturer"
+F 4 "Kemet" H 8050 4350 50  0001 C CNN "Manufacturer"
+F 5 "X7R" H 8050 4350 50  0001 C CNN "Dielectric"
+F 6 "C0805C105K5RACTU" H 8050 4350 50  0001 C CNN "Manufacturer PN"
+F 7 "50V" H 8050 4350 50  0001 C CNN "Voltage"
 	1    8050 4350
 	-1   0    0    1
@@
 F 2 "RespiraWorks_Std:C_0603_1608Metric" H 8488 4200 50  0001 C CNN
 F 3 "~" H 8450 4350 50  0001 C CNN
-F 4 "AVX" H 8450 4350 50  0001 C CNN "Manufacturer"
+F 4 "Kemet" H 8450 4350 50  0001 C CNN "Manufacturer"
+F 5 "X7R" H 8450 4350 50  0001 C CNN "Dielectric"
+F 6 "C0805C105K5RACTU" H 8450 4350 50  0001 C CNN "Manufacturer PN"
+F 7 "50V" H 8450 4350 50  0001 C CNN "Voltage"
 	1    8450 4350
 	-1   0    0    1
