File: pcb/sensors_temp_rtd.sch (KiCad schematic (older format))
At the start: 11 parts

Commit message: BOM
More BOM consolidation with bulk capacitors + changed tantalum stepper caps to aluminum, added bulk cap to PSol driver
Made stepper's 3.3V power naming consistent with others (3.3V->3V3)
Slightly increased current limit on PSOL/heater driver
Changed 3906 transistors to 2907 to better support +5V_Batt current
Parts:
- R? (x7): Part Number RK73H2BTTD1004F -> (none)
Changed lines of the file:
@@
 F 3 "~" H 4100 3450 50  0001 C CNN
 F 4 "KOA Speer" H 4100 3450 50  0001 C CNN "Manufacturer"
-F 5 "RK73H2BTTD1004F" H 4100 3450 50  0001 C CNN "Part Number"
 	1    4100 3450
 	-1   0    0    1
@@
 F 3 "~" H 5350 2700 50  0001 C CNN
 F 4 "" H 5350 2700 50  0001 C CNN "Manufacturer"
-F 5 "" H 5350 2700 50  0001 C CNN "Part Number"
 	1    5350 2700
 	1    0    0    1
@@
 F 3 "~" H 3350 3500 50  0001 C CNN
 F 4 "KOA Speer" H 3350 3500 50  0001 C CNN "Manufacturer"
-F 5 "RK73H2BTTD1004F" H 3350 3500 50  0001 C CNN "Part Number"
 	1    3350 3500
 	-1   0    0    1
@@
 F 3 "~" H 3350 3800 50  0001 C CNN
 F 4 "KOA Speer" H 3350 3800 50  0001 C CNN "Manufacturer"
-F 5 "RK73H2BTTD1004F" H 3350 3800 50  0001 C CNN "Part Number"
 	1    3350 3800
 	-1   0    0    1
@@
 F 3 "~" H 2800 2700 50  0001 C CNN
 F 4 "KOA Speer" H 2800 2700 50  0001 C CNN "Manufacturer"
-F 5 "RK73H2BTTD1004F" H 2800 2700 50  0001 C CNN "Part Number"
 	1    2800 2700
 	-1   0    0    1
@@
 F 3 "~" H 6000 3400 50  0001 C CNN
 F 4 "KOA Speer" H 6000 3400 50  0001 C CNN "Manufacturer"
-F 5 "RK73H2BTTD1004F" H 6000 3400 50  0001 C CNN "Part Number"
 	1    6000 3400
 	0    -1   -1   0
@@
 F 3 "~" H 5550 3650 50  0001 C CNN
 F 4 "KOA Speer" H 5550 3650 50  0001 C CNN "Manufacturer"
-F 5 "RK73H2BTTD1004F" H 5550 3650 50  0001 C CNN "Part Number"
 	1    5550 3650
 	1    0    0    -1
@@
 F 3 "~" H 3100 3200 50  0001 C CNN
 F 4 "KOA Speer" H 3100 3200 50  0001 C CNN "Manufacturer"
-F 5 "RK73H2BTTD1004F" H 3100 3200 50  0001 C CNN "Part Number"
 	1    3100 3200
 	0    -1   -1   0
