File: pcb/cycle_controller.sch (KiCad schematic (older format))
At the start: 45 parts

Commit message: Pinout fixes, TPs
Fixed pinout for stepper motor limit switches
Added testpoints to programmer's serial connection to CC
Parts:
- removed J?: Optical end stop 1, RespiraWorks_Std:Molex_Micro-Fit_3.0_43650-0315_1x03_P3.00mm_Vertical, symbol Connector_Generic:Conn_01x03
- removed J?: Optical end stop 2, RespiraWorks_Std:Molex_Micro-Fit_3.0_43650-0315_1x03_P3.00mm_Vertical, symbol Connector_Generic:Conn_01x03
- added C? (x2): TBD, RespiraWorks_std:C_0603_1608Metric, symbol Device:C
- added J?: Optical end stop 1, RespiraWorks_Std:Molex_Micro-Fit_3.0_43650-0315_1x03_P3.00mm_Vertical, symbol Connector_Generic:Conn_01x03
- added J?: Optical end stop 2, RespiraWorks_Std:Molex_Micro-Fit_3.0_43650-0315_1x03_P3.00mm_Vertical, symbol Connector_Generic:Conn_01x03
- added R? (x2): 0, RespiraWorks_std:R_0603_1608Metric, symbol Device:R
Connections:
- net labels added: Stepper-Lim-Sw1, Stepper-Lim-Sw2
- wire segments 224 -> 225
- no-connect marks 9 -> 7
Changed lines of the file:
@@
 	6400 2500 6700 2500
-Wire Wire Line
-	6400 3400 7150 3400
 Wire Wire Line
 	6400 3500 6700 3500
@@
 Connection ~ 4150 5450
 Wire Wire Line
-	4800 4450 4950 4450
-Wire Wire Line
-	4950 4450 4950 4500
-Wire Wire Line
-	4950 4500 5100 4500
-Wire Wire Line
 	4350 4000 5100 4000
-NoConn ~ 5100 4400
 $Comp
 L power:GNDA #PWR?
@@
 	1    0    0    -1
 $EndComp
-$Comp
-L Connector_Generic:Conn_01x03 J?
-U 1 1 600F2B33
-P 8850 2900
-F 0 "J?" H 8800 3200 50  0000 L CNN
-F 1 "Optical end stop 1" H 8500 3100 50  0000 L CNN
-F 2 "RespiraWorks_Std:Molex_Micro-Fit_3.0_43650-0315_1x03_P3.00mm_Vertical" H 8850 2900 50  0001 C CNN
-F 3 "~" H 8850 2900 50  0001 C CNN
-	1    8850 2900
-	1    0    0    -1
-$EndComp
-$Comp
-L Connector_Generic:Conn_01x03 J?
-U 1 1 600F2BC2
-P 8850 3300
-F 0 "J?" H 8800 3000 50  0000 L CNN
-F 1 "Optical end stop 2" H 8450 2900 50  0000 L CNN
-F 2 "RespiraWorks_Std:Molex_Micro-Fit_3.0_43650-0315_1x03_P3.00mm_Vertical" H 8850 3300 50  0001 C CNN
-F 3 "~" H 8850 3300 50  0001 C CNN
-	1    8850 3300
-	1    0    0    -1
-$EndComp
 NoConn ~ 10500 2250
 Text Label 3850 1600 0    50   ~ 0
@@
 Wire Wire Line
 	10050 2350 10050 2250
-$Comp
-L power:+5V #PWR?
-U 1 1 6020E488
-P 8350 2750
-F 0 "#PWR?" H 8350 2600 50  0001 C CNN
-F 1 "+5V" H 8365 2923 50  0000 C CNN
-F 2 "" H 8350 2750 50  0001 C CNN
-F 3 "" H 8350 2750 50  0001 C CNN
-	1    8350 2750
-	1    0    0    -1
-$EndComp
-Wire Wire Line
-	8650 3200 8350 3200
-Wire Wire Line
-	8650 2800 8350 2800
-$Comp
-L power:GND #PWR?
-U 1 1 60226FFE
-P 8500 3400
-F 0 "#PWR?" H 8500 3150 50  0001 C CNN
-F 1 "GND" H 8505 3227 50  0000 C CNN
-F 2 "" H 8500 3400 50  0001 C CNN
-F 3 "" H 8500 3400 50  0001 C CNN
-	1    8500 3400
-	1    0    0    -1
-$EndComp
-Wire Wire Line
-	8650 3000 8500 3000
-Wire Wire Line
-	8500 3000 8500 3400
-Wire Wire Line
-	8650 3400 8500 3400
-Connection ~ 8500 3400
 Wire Wire Line
 	7350 850  7500 850
@@
 Wire Wire Line
 	3150 6100 3550 6100
-Wire Wire Line
-	8350 2750 8350 2800
-Connection ~ 8350 2800
-Wire Wire Line
-	8350 2800 8350 3200
 Text Notes 9300 1950 0    79   ~ 0
 Arduino headers for expansion
@@
 Text HLabel 4850 4200 0    50   BiDi ~ 0
 PC9
-Text HLabel 4800 4450 0    50   BiDi ~ 0
+Text HLabel 4850 4500 0    50   BiDi ~ 0
 PC12
 Text HLabel 6700 4700 2    50   BiDi ~ 0
@@
 Text HLabel 6700 3500 2    50   BiDi ~ 0
 PB2
-Text HLabel 7200 3400 2    50   BiDi ~ 0
+Text HLabel 6700 3400 2    50   BiDi ~ 0
 PB1
 Text HLabel 6700 3300 2    50   BiDi ~ 0
@@
 Text HLabel 6700 1900 2    50   BiDi ~ 0
 PA3
-Text HLabel 7500 1800 2    50   BiDi ~ 0
+Text HLabel 6700 1800 2    50   BiDi ~ 0
 PA2
 Text HLabel 6700 1700 2    50   BiDi ~ 0
@@
 	6400 1700 6700 1700
 Wire Wire Line
-	7450 1800 7450 2900
-Wire Wire Line
-	7150 3300 7150 3400
-Connection ~ 7150 3400
-Wire Wire Line
-	7150 3400 7200 3400
-Wire Wire Line
-	7450 2900 8650 2900
-Wire Wire Line
-	7150 3300 8650 3300
-Wire Wire Line
 	6400 4300 6700 4300
 Wire Wire Line
@@
 Text Label 10050 6250 0    50   ~ 0
 PB1
-NoConn ~ 5100 4300
-Wire Wire Line
-	7500 1800 7450 1800
-Wire Wire Line
-	6400 1800 7450 1800
-Connection ~ 7450 1800
 Text HLabel 6700 2100 2    50   Output ~ 0
 SPI-SCLK
@@
 Wire Wire Line
 	5200 7100 5200 6800
+Wire Wire Line
+	6400 1800 6700 1800
+Wire Wire Line
+	6700 3400 6400 3400
+Wire Wire Line
+	4850 4500 5100 4500
+$Comp
+L Connector_Generic:Conn_01x03 J?
+U 1 1 604A44BD
+P 1100 1000
+F 0 "J?" H 1050 1300 50  0000 L CNN
+F 1 "Optical end stop 1" H 750 1200 50  0000 L CNN
+F 2 "RespiraWorks_Std:Molex_Micro-Fit_3.0_43650-0315_1x03_P3.00mm_Vertical" H 1100 1000 50  0001 C CNN
+F 3 "~" H 1100 1000 50  0001 C CNN
+	1    1100 1000
+	-1   0    0    -1
+$EndComp
+$Comp
+L Connector_Generic:Conn_01x03 J?
+U 1 1 604A44C3
+P 1100 1600
+F 0 "J?" H 1050 1300 50  0000 L CNN
+F 1 "Optical end stop 2" H 700 1200 50  0000 L CNN
+F 2 "RespiraWorks_Std:Molex_Micro-Fit_3.0_43650-0315_1x03_P3.00mm_Vertical" H 1100 1600 50  0001 C CNN
+F 3 "~" H 1100 1600 50  0001 C CNN
+	1    1100 1600
+	-1   0    0    -1
+$EndComp
+$Comp
+L power:+5V #PWR?
+U 1 1 604A44C9
+P 1600 850
+F 0 "#PWR?" H 1600 700 50  0001 C CNN
+F 1 "+5V" H 1615 1023 50  0000 C CNN
+F 2 "" H 1600 850 50  0001 C CNN
+F 3 "" H 1600 850 50  0001 C CNN
+	1    1600 850
+	-1   0    0    -1
+$EndComp
+Wire Wire Line
+	1300 1500 1600 1500
+Wire Wire Line
+	1300 900  1600 900
+$Comp
+L power:GND #PWR?
+U 1 1 604A44D1
+P 1450 1700
+F 0 "#PWR?" H 1450 1450 50  0001 C CNN
+F 1 "GND" H 1455 1527 50  0000 C CNN
+F 2 "" H 1450 1700 50  0001 C CNN
+F 3 "" H 1450 1700 50  0001 C CNN
+	1    1450 1700
+	-1   0    0    -1
+$EndComp
+Wire Wire Line
+	1300 1100 1450 1100
+Wire Wire Line
+	1300 1700 1450 1700
+Connection ~ 1450 1700
+Wire Wire Line
+	1600 850  1600 900
+Wire Wire Line
+	3000 1600 2150 1600
+$Comp
+L Device:R R?
+U 1 1 604BABA2
+P 1900 1000
+F 0 "R?" V 1800 950 50  0000 C CNN
+F 1 "0" V 1800 1100 50  0000 C CNN
+F 2 "RespiraWorks_std:R_0603_1608Metric" V 1830 1000 50  0001 C CNN
+F 3 "~" H 1900 1000 50  0001 C CNN
+	1    1900 1000
+	0    1    1    0
+$EndComp
+Wire Wire Line
+	1750 1000 1600 1000
+$Comp
+L Device:R R?
+U 1 1 604BB5FA
+P 1900 1600
+F 0 "R?" V 1800 1550 50  0000 C CNN
+F 1 "0" V 1800 1700 50  0000 C CNN
+F 2 "RespiraWorks_std:R_0603_1608Metric" V 1830 1600 50  0001 C CNN
+F 3 "~" H 1900 1600 50  0001 C CNN
+	1    1900 1600
+	0    1    1    0
+$EndComp
+Wire Wire Line
+	1750 1600 1300 1600
+$Comp
+L Device:C C?
+U 1 1 604C1B1C
+P 2150 1750
+F 0 "C?" H 1950 1750 50  0000 L CNN
+F 1 "TBD" H 1900 1850 50  0000 L CNN
+F 2 "RespiraWorks_std:C_0603_1608Metric" H 2188 1600 50  0001 C CNN
+F 3 "~" H 2150 1750 50  0001 C CNN
+F 4 "DNP" H 1950 1950 50  0000 C CNN "DNP"
+	1    2150 1750
+	-1   0    0    1
+$EndComp
+Connection ~ 2150 1600
+Wire Wire Line
+	2150 1600 2050 1600
+$Comp
+L Device:C C?
+U 1 1 604C7BF1
+P 2150 1150
+F 0 "C?" H 1950 1150 50  0000 L CNN
+F 1 "TBD" H 1900 1250 50  0000 L CNN
+F 2 "RespiraWorks_std:C_0603_1608Metric" H 2188 1000 50  0001 C CNN
+F 3 "~" H 2150 1150 50  0001 C CNN
+F 4 "DNP" H 1950 1350 50  0000 C CNN "DNP"
+	1    2150 1150
+	-1   0    0    1
+$EndComp
+$Comp
+L power:GND #PWR?
+U 1 1 604C8205
+P 2150 1900
+F 0 "#PWR?" H 2150 1650 50  0001 C CNN
+F 1 "GND" H 2155 1727 50  0000 C CNN
+F 2 "" H 2150 1900 50  0001 C CNN
+F 3 "" H 2150 1900 50  0001 C CNN
+	1    2150 1900
+	-1   0    0    -1
+$EndComp
+Wire Wire Line
+	2050 1000 2150 1000
+Connection ~ 2150 1000
+Wire Wire Line
+	1450 1100 1450 1700
+Wire Wire Line
+	1600 1000 1600 1500
+Connection ~ 1600 1000
+Wire Wire Line
+	1600 1000 1300 1000
+$Comp
+L power:GND #PWR?
+U 1 1 605037AB
+P 2150 1300
+F 0 "#PWR?" H 2150 1050 50  0001 C CNN
+F 1 "GND" H 2155 1127 50  0000 C CNN
+F 2 "" H 2150 1300 50  0001 C CNN
+F 3 "" H 2150 1300 50  0001 C CNN
+	1    2150 1300
+	-1   0    0    -1
+$EndComp
+Wire Wire Line
+	2150 1000 3000 1000
+Text Label 3000 1000 2    50   ~ 0
+Stepper-Lim-Sw1
+Text Label 3000 1600 2    50   ~ 0
+Stepper-Lim-Sw2
+Text Label 4300 4300 0    50   ~ 0
+Stepper-Lim-Sw1
+Wire Wire Line
+	4300 4400 5100 4400
+Wire Wire Line
+	4300 4300 5100 4300
+Text Label 4300 4400 0    50   ~ 0
+Stepper-Lim-Sw2
 $EndSCHEMATC

Commit message: CC-I2C, BOM
Added missing pull-ups on CC-SDA, CC-SCL
First pass at BOM consolidation
Parts:
- C? (x7): value 0.1uF, 10V -> 100nF; footprint RespiraWorks_std:C_0603_1608Metric -> RespiraWorks_Std:C_0603_1608Metric
- C?: value 4.7uF, 10V -> 4.7uF; footprint RespiraWorks_std:C_0603_1608Metric -> RespiraWorks_Std:C_0603_1608Metric
- C? (x2): value 1uF, 10V -> 1uF; footprint RespiraWorks_std:C_0603_1608Metric -> RespiraWorks_Std:C_0603_1608Metric
- C? (x4): footprint RespiraWorks_std:C_0603_1608Metric -> RespiraWorks_Std:C_0603_1608Metric
- C?: value 1uF, 10V -> 1uF; footprint (none) -> RespiraWorks_Std:C_0603_1608Metric
- C?: value 0.1uF, 10V -> 100nF; footprint (none) -> RespiraWorks_Std:C_0603_1608Metric
- R? (x2): value 10K -> 10k; footprint RespiraWorks_std:R_0603_1608Metric -> RespiraWorks_Std:R_0603_1608Metric
- R?: value 4.7K -> 4.7k; footprint RespiraWorks_std:R_0603_1608Metric -> RespiraWorks_Std:R_0603_1608Metric
- R?: footprint RespiraWorks_std:R_0603_1608Metric -> RespiraWorks_Std:R_0603_1608Metric
- Y?: value 8 MHz -> 8 Mhz
Changed lines of the file:
@@
 P 7500 1000
 F 0 "C?" H 7450 1200 50  0000 L CNN
-F 1 "0.1uF, 10V" H 7350 600 50  0000 L CNN
-F 2 "RespiraWorks_std:C_0603_1608Metric" H 7538 850 50  0001 C CNN
+F 1 "100nF" H 7350 600 50  0000 L CNN
+F 2 "RespiraWorks_Std:C_0603_1608Metric" H 7538 850 50  0001 C CNN
 F 3 "~" H 7500 1000 50  0001 C CNN
 	1    7500 1000
@@
 P 7800 1000
 F 0 "C?" H 7750 1200 50  0000 L CNN
-F 1 "0.1uF, 10V" H 7650 700 50  0000 L CNN
-F 2 "RespiraWorks_std:C_0603_1608Metric" H 7838 850 50  0001 C CNN
+F 1 "100nF" H 7650 700 50  0000 L CNN
+F 2 "RespiraWorks_Std:C_0603_1608Metric" H 7838 850 50  0001 C CNN
 F 3 "~" H 7800 1000 50  0001 C CNN
 	1    7800 1000
@@
 P 8150 1000
 F 0 "C?" H 8100 1200 50  0000 L CNN
-F 1 "0.1uF, 10V" H 7950 600 50  0000 L CNN
-F 2 "RespiraWorks_std:C_0603_1608Metric" H 8188 850 50  0001 C CNN
+F 1 "100nF" H 7950 600 50  0000 L CNN
+F 2 "RespiraWorks_Std:C_0603_1608Metric" H 8188 850 50  0001 C CNN
 F 3 "~" H 8150 1000 50  0001 C CNN
 	1    8150 1000
@@
 P 8450 1000
 F 0 "C?" H 8400 1200 50  0000 L CNN
-F 1 "0.1uF, 10V" H 8250 700 50  0000 L CNN
-F 2 "RespiraWorks_std:C_0603_1608Metric" H 8488 850 50  0001 C CNN
+F 1 "100nF" H 8250 700 50  0000 L CNN
+F 2 "RespiraWorks_Std:C_0603_1608Metric" H 8488 850 50  0001 C CNN
 F 3 "~" H 8450 1000 50  0001 C CNN
 	1    8450 1000
@@
 P 8750 1000
 F 0 "C?" H 8700 1200 50  0000 L CNN
-F 1 "4.7uF, 10V" H 8750 900 50  0000 L CNN
-F 2 "RespiraWorks_std:C_0603_1608Metric" H 8788 850 50  0001 C CNN
+F 1 "4.7uF" H 8750 900 50  0000 L CNN
+F 2 "RespiraWorks_Std:C_0603_1608Metric" H 8788 850 50  0001 C CNN
 F 3 "~" H 8750 1000 50  0001 C CNN
 	1    8750 1000
@@
 P 9550 1050
 F 0 "C?" H 9450 1300 50  0000 L CNN
-F 1 "0.1uF, 10V" H 9300 850 50  0000 L CNN
-F 2 "RespiraWorks_std:C_0603_1608Metric" H 9588 900 50  0001 C CNN
+F 1 "100nF" H 9300 850 50  0000 L CNN
+F 2 "RespiraWorks_Std:C_0603_1608Metric" H 9588 900 50  0001 C CNN
 F 3 "~" H 9550 1050 50  0001 C CNN
 	1    9550 1050
@@
 P 9900 1050
 F 0 "C?" H 9850 1300 50  0000 L CNN
-F 1 "1uF, 10V" H 9950 950 50  0000 L CNN
-F 2 "RespiraWorks_std:C_0603_1608Metric" H 9938 900 50  0001 C CNN
+F 1 "1uF" H 9950 950 50  0000 L CNN
+F 2 "RespiraWorks_Std:C_0603_1608Metric" H 9938 900 50  0001 C CNN
 F 3 "~" H 9900 1050 50  0001 C CNN
 	1    9900 1050
@@
 P 4700 1750
 F 0 "C?" H 4815 1776 50  0000 L CNN
-F 1 "0.1uF, 10V" H 4750 1650 50  0000 L CNN
-F 2 "RespiraWorks_std:C_0603_1608Metric" H 4738 1600 50  0001 C CNN
+F 1 "100nF" H 4750 1650 50  0000 L CNN
+F 2 "RespiraWorks_Std:C_0603_1608Metric" H 4738 1600 50  0001 C CNN
 F 3 "~" H 4700 1750 50  0001 C CNN
 	1    4700 1750
@@
 P 3700 3050
 F 0 "R?" H 3550 3150 50  0000 C CNN
-F 1 "10K" H 3550 3050 50  0000 C CNN
-F 2 "RespiraWorks_std:R_0603_1608Metric" V 3630 3050 50  0001 C CNN
+F 1 "10k" H 3550 3050 50  0000 C CNN
+F 2 "RespiraWorks_Std:R_0603_1608Metric" V 3630 3050 50  0001 C CNN
 F 3 "~" H 3700 3050 50  0001 C CNN
 	1    3700 3050
@@
 P 2850 2950
 F 0 "Y?" V 2804 3081 50  0000 L CNN
-F 1 "8 MHz" V 2895 3081 50  0000 L CNN
+F 1 "8 Mhz" V 2895 3081 50  0000 L CNN
 F 2 "RespiraWorks_Std:Crystal_SMD_HC49-SD" H 2850 2950 50  0001 C CNN
 F 3 "~" H 2850 2950 50  0001 C CNN
@@
 F 0 "C?" V 2600 2750 50  0000 L CNN
 F 1 "20pF" V 2500 2750 50  0000 L CNN
-F 2 "RespiraWorks_std:C_0603_1608Metric" H 2588 2550 50  0001 C CNN
+F 2 "RespiraWorks_Std:C_0603_1608Metric" H 2588 2550 50  0001 C CNN
 F 3 "~" H 2550 2700 50  0001 C CNN
 F 4 "DNP" V 2600 2500 50  0000 L CNN "DNP"
@@
 F 0 "C?" V 2600 3300 50  0000 L CNN
 F 1 "20pF" V 2500 3300 50  0000 L CNN
-F 2 "RespiraWorks_std:C_0603_1608Metric" H 2588 3100 50  0001 C CNN
+F 2 "RespiraWorks_Std:C_0603_1608Metric" H 2588 3100 50  0001 C CNN
 F 3 "~" H 2550 3250 50  0001 C CNN
 F 4 "DNP" V 2600 3050 50  0000 L CNN "DNP"
@@
 P 2200 4200
 F 0 "R?" H 2050 4300 50  0000 C CNN
-F 1 "4.7K" H 2050 4200 50  0000 C CNN
-F 2 "RespiraWorks_std:R_0603_1608Metric" V 2130 4200 50  0001 C CNN
+F 1 "4.7k" H 2050 4200 50  0000 C CNN
+F 2 "RespiraWorks_Std:R_0603_1608Metric" V 2130 4200 50  0001 C CNN
 F 3 "~" H 2200 4200 50  0001 C CNN
 	1    2200 4200
@@
 P 1600 4500
 F 0 "C?" H 1715 4526 50  0000 L CNN
-F 1 "0.1uF, 10V" H 1650 4400 50  0000 L CNN
-F 2 "RespiraWorks_std:C_0603_1608Metric" H 1638 4350 50  0001 C CNN
+F 1 "100nF" H 1650 4400 50  0000 L CNN
+F 2 "RespiraWorks_Std:C_0603_1608Metric" H 1638 4350 50  0001 C CNN
 F 3 "~" H 1600 4500 50  0001 C CNN
 	1    1600 4500
@@
 F 0 "R?" V 1650 4850 50  0000 C CNN
 F 1 "100" V 1650 4650 50  0000 C CNN
-F 2 "RespiraWorks_std:R_0603_1608Metric" V 1730 4750 50  0001 C CNN
+F 2 "RespiraWorks_Std:R_0603_1608Metric" V 1730 4750 50  0001 C CNN
 F 3 "~" H 1800 4750 50  0001 C CNN
 	1    1800 4750
@@
 AR Path="/5FCD4D18/6016938C" Ref="C?"  Part="1"
 F 0 "C?" H 3200 6400 50  0000 L CNN
-F 1 "1uF, 10V" H 2950 6200 50  0000 L CNN
-F 2 "" H 3188 6150 50  0001 C CNN
+F 1 "1uF" H 2950 6200 50  0000 L CNN
+F 2 "RespiraWorks_Std:C_0603_1608Metric" H 3188 6150 50  0001 C CNN
 F 3 "~" H 3150 6300 50  0001 C CNN
 	1    3150 6300
@@
 AR Path="/5FCD4D18/60169393" Ref="C?"  Part="1"
 F 0 "C?" H 3600 6400 50  0000 L CNN
-F 1 "0.1uF, 10V" H 3600 6200 50  0000 L CNN
-F 2 "" H 3588 6150 50  0001 C CNN
+F 1 "100nF" H 3600 6200 50  0000 L CNN
+F 2 "RespiraWorks_Std:C_0603_1608Metric" H 3588 6150 50  0001 C CNN
 F 3 "~" H 3550 6300 50  0001 C CNN
 	1    3550 6300
@@
 AR Path="/5FCD4D18/601693C1" Ref="R?"  Part="1"
 F 0 "R?" H 900 6850 50  0000 L CNN
-F 1 "10K" H 850 6750 50  0000 L CNN
-F 2 "RespiraWorks_std:R_0603_1608Metric" V 980 6800 50  0001 C CNN
+F 1 "10k" H 850 6750 50  0000 L CNN
+F 2 "RespiraWorks_Std:R_0603_1608Metric" V 980 6800 50  0001 C CNN
 F 3 "~" H 1050 6800 50  0001 C CNN
 	1    1050 6800
@@
 P 4600 1100
 F 0 "C?" H 4300 1200 50  0000 L CNN
-F 1 "1uF, 10V" H 4150 1100 50  0000 L CNN
-F 2 "RespiraWorks_std:C_0603_1608Metric" H 4638 950 50  0001 C CNN
+F 1 "1uF" H 4150 1100 50  0000 L CNN
+F 2 "RespiraWorks_Std:C_0603_1608Metric" H 4638 950 50  0001 C CNN
 F 3 "~" H 4600 1100 50  0001 C CNN
 	1    4600 1100
@@
 F 0 "C?" H 1950 1750 50  0000 L CNN
 F 1 "TBD" H 1900 1850 50  0000 L CNN
-F 2 "RespiraWorks_std:C_0603_1608Metric" H 2188 1600 50  0001 C CNN
+F 2 "RespiraWorks_Std:C_0603_1608Metric" H 2188 1600 50  0001 C CNN
 F 3 "~" H 2150 1750 50  0001 C CNN
 F 4 "DNP" H 1950 1950 50  0000 C CNN "DNP"
@@
 F 0 "C?" H 1950 1150 50  0000 L CNN
 F 1 "TBD" H 1900 1250 50  0000 L CNN
-F 2 "RespiraWorks_std:C_0603_1608Metric" H 2188 1000 50  0001 C CNN
+F 2 "RespiraWorks_Std:C_0603_1608Metric" H 2188 1000 50  0001 C CNN
 F 3 "~" H 2150 1150 50  0001 C CNN
 F 4 "DNP" H 1950 1350 50  0000 C CNN "DNP"
