File: pcb/ui_computer.sch (KiCad schematic (older format))
At the start: 9 parts

Commit message: PCB Rev A Floorplanning (#1079)
* annotate schematics

* generate netlist

* define board edges at 150x300mm

* add parts to board (some pending errors)

* fix schem-pcb footprint mismatches and push to PCB

* preliminary packing at 155x300mm board size - marginal

* PCB floor planning

* added fan power and swapped solenoid/touchscreen power to vertical connectors
Parts:
- J9: renamed from J?; footprint RespiraWorks_Std:Molex_Micro-Fit_3.0_43650-0200_1x02_P3.00mm_Horizontal -> RespiraWorks_Std:Molex_Micro-Fit_3.0_43045-0212_2x01_P3.00mm_Vertical; Manufacturer PN 43650-0200 -> 43045-0212
- gave numbers to parts that had none: 8
Changed lines of the file:
@@
 $EndDescr
 $Comp
-L RespiraWorks:ESQ-120-44-L-D J?
+L RespiraWorks:ESQ-120-44-L-D J8
 U 1 1 5FDAF122
 P 5700 3350
-F 0 "J?" H 5725 4625 50  0000 C CNN
+F 0 "J8" H 5725 4625 50  0000 C CNN
 F 1 "Raspberry Pi" H 5725 4534 50  0000 C CNN
 F 2 "RespiraWorks_Std:PinHeader_2x20_P2.54mm_Vertical" H 5100 4450 50  0001 C CNN
@@
 $EndComp
 $Comp
-L RespiraWorks:+3V3_RPi #PWR?
+L RespiraWorks:+3V3_RPi #PWR0121
 U 1 1 5FDB01F4
 P 4750 2250
-F 0 "#PWR?" H 4750 2300 50  0001 C CNN
+F 0 "#PWR0121" H 4750 2300 50  0001 C CNN
 F 1 "+3V3_RPi" H 4735 2423 50  0000 C CNN
 F 2 "" H 4750 2250 50  0001 C CNN
@@
 	4550 2600 5000 2600
 $Comp
-L power:GND #PWR?
+L power:GND #PWR0122
 U 1 1 5FDB0314
 P 4850 4300
-F 0 "#PWR?" H 4850 4050 50  0001 C CNN
+F 0 "#PWR0122" H 4850 4050 50  0001 C CNN
 F 1 "GND" H 4855 4127 50  0000 C CNN
 F 2 "" H 4850 4300 50  0001 C CNN
@@
 	5000 3900 4550 3900
 $Comp
-L Device:R R?
+L Device:R R51
 U 1 1 5FDB08DB
 P 3800 4350
-F 0 "R?" H 3650 4400 50  0000 L CNN
+F 0 "R51" H 3650 4400 50  0000 L CNN
 F 1 "0" H 3650 4300 50  0000 L CNN
 F 2 "RespiraWorks_Std:R_0603_1608Metric" V 3730 4350 50  0001 C CNN
@@
 $EndComp
 $Comp
-L RespiraWorks:+3V3_RPi #PWR?
+L RespiraWorks:+3V3_RPi #PWR0119
 U 1 1 5FDB0BF2
 P 3800 3700
-F 0 "#PWR?" H 3800 3750 50  0001 C CNN
+F 0 "#PWR0119" H 3800 3750 50  0001 C CNN
 F 1 "+3V3_RPi" H 3785 3873 50  0000 C CNN
 F 2 "" H 3800 3700 50  0001 C CNN
@@
 Connection ~ 3800 4100
 $Comp
-L power:GND #PWR?
+L power:GND #PWR0120
 U 1 1 5FDB0EEF
 P 3800 4500
-F 0 "#PWR?" H 3800 4250 50  0001 C CNN
+F 0 "#PWR0120" H 3800 4250 50  0001 C CNN
 F 1 "GND" H 3805 4327 50  0000 C CNN
 F 2 "" H 3800 4500 50  0001 C CNN
@@
 UI_ID1
 $Comp
-L Device:R R?
+L Device:R R50
 U 1 1 5FE66293
 P 3800 3850
-F 0 "R?" H 3650 3900 50  0000 L CNN
+F 0 "R50" H 3650 3900 50  0000 L CNN
 F 1 "0" H 3650 3800 50  0000 L CNN
 F 2 "RespiraWorks_Std:R_0603_1608Metric" V 3730 3850 50  0001 C CNN
@@
 	6650 2500 6450 2500
 $Comp
-L power:GND #PWR?
+L power:GND #PWR0124
 U 1 1 5FE67C8B
 P 6650 4300
-F 0 "#PWR?" H 6650 4050 50  0001 C CNN
+F 0 "#PWR0124" H 6650 4050 50  0001 C CNN
 F 1 "GND" H 6655 4127 50  0000 C CNN
 F 2 "" H 6650 4300 50  0001 C CNN
@@
 UI_ID0
 $Comp
-L Device:R R?
+L Device:R R52
 U 1 1 5FE6BCEC
 P 7950 3000
-F 0 "R?" H 8050 3050 50  0000 L CNN
+F 0 "R52" H 8050 3050 50  0000 L CNN
 F 1 "0" H 8050 2950 50  0000 L CNN
 F 2 "RespiraWorks_Std:R_0603_1608Metric" V 7880 3000 50  0001 C CNN
@@
 $EndComp
 $Comp
-L Device:R R?
+L Device:R R53
 U 1 1 5FE6BE04
 P 7950 3600
-F 0 "R?" H 8050 3650 50  0000 L CNN
+F 0 "R53" H 8050 3650 50  0000 L CNN
 F 1 "0" H 8050 3550 50  0000 L CNN
 F 2 "RespiraWorks_Std:R_0603_1608Metric" V 7880 3600 50  0001 C CNN
@@
 $EndComp
 $Comp
-L power:GND #PWR?
+L power:GND #PWR0126
 U 1 1 5FE6BE44
 P 7950 3750
-F 0 "#PWR?" H 7950 3500 50  0001 C CNN
+F 0 "#PWR0126" H 7950 3500 50  0001 C CNN
 F 1 "GND" H 7955 3577 50  0000 C CNN
 F 2 "" H 7950 3750 50  0001 C CNN
@@
 Connection ~ 7950 3300
 $Comp
-L RespiraWorks:+3V3_RPi #PWR?
+L RespiraWorks:+3V3_RPi #PWR0125
 U 1 1 5FE6C7D6
 P 7950 2850
-F 0 "#PWR?" H 7950 2900 50  0001 C CNN
+F 0 "#PWR0125" H 7950 2900 50  0001 C CNN
 F 1 "+3V3_RPi" H 7935 3023 50  0000 C CNN
 F 2 "" H 7950 2850 50  0001 C CNN
@@
 USB TO UART adapter: https://www.ftdichip.com/Support/Documents/DataSheets/Modules/DS_DB9-USB-RS232.pdf
 $Comp
-L RespiraWorks:RaspberryPi H?
+L RespiraWorks:RaspberryPi H1
 U 1 1 600E005B
 P 5700 5600
-F 0 "H?" H 5700 6300 50  0001 C CNN
+F 0 "H1" H 5700 6300 50  0001 C CNN
 F 1 "RaspberryPi" H 5800 6250 50  0001 C CNN
 F 2 "RespiraWorks:RaspberryPi" H 5700 5600 50  0001 C CNN
@@
 $EndComp
 $Comp
-L power:GND #PWR?
+L power:GND #PWR0123
 U 1 1 600E0077
 P 5800 5700
-F 0 "#PWR?" H 5800 5450 50  0001 C CNN
+F 0 "#PWR0123" H 5800 5450 50  0001 C CNN
 F 1 "GND" H 5805 5527 50  0000 C CNN
 F 2 "" H 5800 5700 50  0001 C CNN
@@
 	4550 4000 5000 4000
 $Comp
-L Device:C C?
+L Device:C C45
 U 1 1 6015F360
 P 7900 1850
-F 0 "C?" H 8015 1896 50  0000 L CNN
+F 0 "C45" H 8015 1896 50  0000 L CNN
 F 1 "100nF" H 8015 1805 50  0000 L CNN
 F 2 "RespiraWorks_Std:C_0603_1608Metric" H 7938 1700 50  0001 C CNN
@@
 $EndComp
 $Comp
-L Device:C C?
+L Device:C C46
 U 1 1 6015F3CE
 P 8350 1850
-F 0 "C?" H 8465 1896 50  0000 L CNN
+F 0 "C46" H 8465 1896 50  0000 L CNN
 F 1 "1uF" H 8465 1805 50  0000 L CNN
 F 2 "RespiraWorks_Std:C_0603_1608Metric" H 8388 1700 50  0001 C CNN
@@
 5V
 $Comp
-L power:GND #PWR?
+L power:GND #PWR0127
 U 1 1 6016DA3F
 P 8150 2100
-F 0 "#PWR?" H 8150 1850 50  0001 C CNN
+F 0 "#PWR0127" H 8150 1850 50  0001 C CNN
 F 1 "GND" H 8155 1927 50  0000 C CNN
 F 2 "" H 8150 2100 50  0001 C CNN
@@
 	8150 2100 8350 2100
 $Comp
-L RespiraWorks_Std:Conn_01x02 J?
+L RespiraWorks_Std:Conn_01x02 J9
 U 1 1 60436098
 P 9850 3650
-F 0 "J?" H 9930 3642 50  0000 L CNN
+F 0 "J9" H 9930 3642 50  0000 L CNN
 F 1 "Touchscreen power" H 9930 3551 50  0000 L CNN
-F 2 "RespiraWorks_Std:Molex_Micro-Fit_3.0_43650-0200_1x02_P3.00mm_Horizontal" H 9850 3650 50  0001 C CNN
+F 2 "RespiraWorks_Std:Molex_Micro-Fit_3.0_43045-0212_2x01_P3.00mm_Vertical" H 9850 3650 50  0001 C CNN
 F 3 "~" H 9850 3650 50  0001 C CNN
 F 4 "Molex" H 9850 3650 50  0001 C CNN "Manufacturer"
-F 5 "43650-0200" H 9850 3650 50  0001 C CNN "Manufacturer PN"
+F 5 "43045-0212" H 9850 3650 50  0001 C CNN "Manufacturer PN"
 	1    9850 3650
 	1    0    0    1
@@
 5V
 $Comp
-L power:GND #PWR?
+L power:GND #PWR0128
 U 1 1 60439316
 P 9650 3650
-F 0 "#PWR?" H 9650 3400 50  0001 C CNN
+F 0 "#PWR0128" H 9650 3400 50  0001 C CNN
 F 1 "GND" H 9655 3477 50  0000 C CNN
 F 2 "" H 9650 3650 50  0001 C CNN
