File: pcb/sensors_temp_ntc.sch (KiCad schematic (older format))
At the start: 5 parts

Commit message: BOM, fixes
Finished assigning parts, footprints except generic resistors
Added series resistors for logic signals received by UI computer to protect against UI computer power-down
Added tolerance notes on main schem
Replaced PSol fuse with PTC
Enlarged PSol driver bypass resistors to 0 ohm
Changed PSol unpopulated current-limiting resistor to divider
Parts:
- J?: Manufacturer (none) -> Molex; Manufacturer PN (none) -> 43650-0215
- R?: Manufacturer (none) -> Susumu; Manufacturer PN (none) -> RG1608P-103-B-T5
- R?: Manufacturer (none) -> Susumu; Manufacturer PN (none) -> RG1608P-221-B-T5
- U?: Manufacturer (none) -> STMicroelectronics; Manufacturer PN (none) -> USBLC6-2SC6
Changed lines of the file:
@@
 F 2 "RespiraWorks_Std:Molex_Micro-Fit_3.0_43650-0215_1x02_P3.00mm_Vertical" H 1550 3200 50  0001 C CNN
 F 3 "~" H 1550 3200 50  0001 C CNN
+F 4 "Molex" H 1550 3200 50  0001 C CNN "Manufacturer"
+F 5 "43650-0215" H 1550 3200 50  0001 C CNN "Manufacturer PN"
 	1    1550 3200
 	-1   0    0    -1
@@
 F 2 "RespiraWorks_Std:R_0603_1608Metric" V 4230 2700 50  0001 C CNN
 F 3 "~" H 4300 2700 50  0001 C CNN
-F 4 "" H 4300 2700 50  0001 C CNN "Manufacturer"
+F 4 "Susumu" H 4300 2700 50  0001 C CNN "Manufacturer"
+F 5 "RG1608P-221-B-T5" H 4300 2700 50  0001 C CNN "Manufacturer PN"
 	1    4300 2700
 	-1   0    0    1
@@
 F 2 "RespiraWorks_Std:R_0603_1608Metric" V 4230 3600 50  0001 C CNN
 F 3 "~" H 4300 3600 50  0001 C CNN
-F 4 "" H 4300 3600 50  0001 C CNN "Manufacturer"
+F 4 "Susumu" H 4300 3600 50  0001 C CNN "Manufacturer"
+F 5 "RG1608P-103-B-T5" H 4300 3600 50  0001 C CNN "Manufacturer PN"
 	1    4300 3600
 	-1   0    0    1
@@
 F 2 "Package_TO_SOT_SMD:SOT-23-6" H 2400 3400 50  0001 C CNN
 F 3 "https://www.st.com/resource/en/datasheet/usblc6-2.pdf" H 2600 4250 50  0001 C CNN
+F 4 "STMicroelectronics" H 2400 3900 50  0001 C CNN "Manufacturer"
+F 5 "USBLC6-2SC6" H 2400 3900 50  0001 C CNN "Manufacturer PN"
 	1    2400 3900
 	0    1    1    0

Commit message: Naming, minor temp sensor changes
Removed outdated "RTD" label on temp sensor connector
Changed "heater" to "PSol2" and "PSol" to "PSol1"
Added leakage error notes on NTC temp sensor page, fixed minor mistake in LPF notes
Put ESD protection for NTC temp sensor on both pins
Parts:
- J?: value Temperature sensor -> Temperature sensor (NTC)
Connections:
- wire segments 15 -> 17
- no-connect marks 2 -> 0
Other:
- note added: "150 nA max. leakage adds << 1 degree error\nacross full temp. range"
- note added: "LPF varies with temp\n(30hz at 150C, 3.1hz at 25C, 2.2hz at 0C)\nOK because of large margin between ADC \nsampling rate and desired sensor bandwidth"
- note removed: "LPF varies with temp\n(30hz at 150C, 1.5hz at 25C, 2.5hz at 0C)\nOK because of large margin between ADC \nsampling rate and desired sensor bandwidth"
- note removed: "PT100 RTD"
Changed lines of the file:
@@
 $Descr A4 11693 8268
 encoding utf-8
-Sheet 25 38
+Sheet 22 38
 Title "NTC Temperature Sensor Input"
 Date ""
@@
 AR Path="/5FCD4EEA/600F723B/6010AD26" Ref="J?"  Part="1"
 F 0 "J?" H 1468 3417 50  0000 C CNN
-F 1 "Temperature sensor" H 1468 3326 50  0000 C CNN
+F 1 "Temperature sensor (NTC)" H 1468 3326 50  0000 C CNN
 F 2 "RespiraWorks_Std:Molex_Micro-Fit_3.0_43650-0215_1x02_P3.00mm_Vertical" H 1550 3200 50  0001 C CNN
 F 3 "~" H 1550 3200 50  0001 C CNN
@@
 	-1   0    0    -1
 $EndComp
-Text Notes 1000 3300 0    50   ~ 0
-PT100 RTD
 $Comp
 L power:GND #PWR?
@@
 $EndComp
 Text Notes 5200 4600 0    50   ~ 0
-LPF varies with temp\n(30hz at 150C, 1.5hz at 25C, 2.5hz at 0C)\nOK because of large margin between ADC \nsampling rate and desired sensor bandwidth
+LPF varies with temp\n(30hz at 150C, 3.1hz at 25C, 2.2hz at 0C)\nOK because of large margin between ADC \nsampling rate and desired sensor bandwidth
 Text Notes 6800 3500 0    50   ~ 0
 for 10k NTC B=3380K:\n@150C: R = 350       Vout = 3.12V   Sensitivity: 2mV/degC\n@100C: R = 1022     Vout = 2.94V   Sensitivity: 6mV/degC\n@25C:  R = 10000   Vout = 1.63V   Sensitivity: 30mV/degC\n@0C:    R = 28255   Vout = 0.86V   Sensitivity: 29mV/degC\n\nTemp (C) = B / ( ln( Vcc*10k/Vout/Rlim - (10k+220)/Rlim )  ) + 273.15\nWhere Rlim = R0*exp(-B/T0) and T0 is in kelvin.
@@
 $EndComp
 Wire Wire Line
-	1750 3300 2300 3300
-Wire Wire Line
 	4300 3300 4300 3450
-Wire Wire Line
-	1750 3200 4300 3200
 Wire Wire Line
 	4300 3200 4300 2850
@@
 L Power_Protection:USBLC6-2SC6 U?
 U 1 1 5FFD5C58
-P 2400 3900
+P 2400 3600
 AR Path="/5FCD4EEA/600F5EF3/5FFD5C58" Ref="U?"  Part="1"
 AR Path="/5FCD4EEA/600F723B/5FFD5C58" Ref="U?"  Part="1"
@@
 AR Path="/5FCD4EEA/600F719E/5FFD5C58" Ref="U?"  Part="1"
 AR Path="/5FCD4EEA/600F71F1/5FFD5C58" Ref="U?"  Part="1"
-F 0 "U?" V 1950 4100 50  0000 L CNN
-F 1 "USBLC6-2SC6" V 2050 4100 50  0000 L CNN
-F 2 "Package_TO_SOT_SMD:SOT-23-6" H 2400 3400 50  0001 C CNN
-F 3 "https://www.st.com/resource/en/datasheet/usblc6-2.pdf" H 2600 4250 50  0001 C CNN
-F 4 "STMicroelectronics" H 2400 3900 50  0001 C CNN "Manufacturer"
-F 5 "USBLC6-2SC6" H 2400 3900 50  0001 C CNN "Manufacturer PN"
-	1    2400 3900
+F 0 "U?" V 1800 3700 50  0000 L CNN
+F 1 "USBLC6-2SC6" V 1900 3550 50  0000 L CNN
+F 2 "Package_TO_SOT_SMD:SOT-23-6" H 2400 3100 50  0001 C CNN
+F 3 "https://www.st.com/resource/en/datasheet/usblc6-2.pdf" H 2600 3950 50  0001 C CNN
+F 4 "STMicroelectronics" H 2400 3600 50  0001 C CNN "Manufacturer"
+F 5 "USBLC6-2SC6" H 2400 3600 50  0001 C CNN "Manufacturer PN"
+	1    2400 3600
 	0    1    1    0
 $EndComp
 Wire Wire Line
-	2500 3500 2500 3300
-Wire Wire Line
-	2500 3300 4300 3300
-Wire Wire Line
-	2300 3500 2300 3300
-NoConn ~ 2300 4300
-NoConn ~ 2500 4300
-Wire Wire Line
-	2800 3900 3100 3900
-Text Label 2850 3900 0    50   ~ 0
-Vcc
-Text Label 4150 2550 0    50   ~ 0
+	2800 3600 3100 3600
+Text Label 3100 3600 2    50   ~ 0
 Vcc
 $Comp
 L power:GND #PWR?
 U 1 1 5FFDA1EB
-P 1800 4050
+P 1900 3650
 AR Path="/5FCD4B8E/5FCD4BC5/5FFDA1EB" Ref="#PWR?"  Part="1"
 AR Path="/5FCD4B8E/5FE27F70/5FFDA1EB" Ref="#PWR?"  Part="1"
@@
 AR Path="/5FCD4EEA/600F71F1/5FFDA1EB" Ref="#PWR?"  Part="1"
 AR Path="/5FCD4EEA/600F723B/5FFDA1EB" Ref="#PWR?"  Part="1"
-F 0 "#PWR?" H 1800 3800 50  0001 C CNN
-F 1 "GND" H 1805 3877 50  0000 C CNN
-F 2 "" H 1800 4050 50  0001 C CNN
-F 3 "" H 1800 4050 50  0001 C CNN
-	1    1800 4050
-	-1   0    0    -1
-$EndComp
-Wire Wire Line
-	2000 3900 1800 3900
-Wire Wire Line
-	1800 3900 1800 4050
+F 0 "#PWR?" H 1900 3400 50  0001 C CNN
+F 1 "GND" H 1905 3477 50  0000 C CNN
+F 2 "" H 1900 3650 50  0001 C CNN
+F 3 "" H 1900 3650 50  0001 C CNN
+	1    1900 3650
+	-1   0    0    -1
+$EndComp
+Wire Wire Line
+	2000 3600 1900 3600
+Wire Wire Line
+	1900 3600 1900 3650
 $Comp
 L Device:C C?
@@
 Wire Wire Line
 	5600 3300 6100 3300
+Text Notes 1650 4250 0    50   ~ 0
+150 nA max. leakage adds << 1 degree error\nacross full temp. range
+Wire Wire Line
+	1750 3300 1750 4000
+Wire Wire Line
+	1750 4000 2300 4000
+Wire Wire Line
+	2500 4000 3450 4000
+Wire Wire Line
+	3450 4000 3450 3300
+Wire Wire Line
+	3450 3300 4300 3300
+Wire Wire Line
+	1750 3200 2300 3200
+Wire Wire Line
+	2500 3200 4300 3200
 $EndSCHEMATC

Commit message: Symbols
Re-assigned transistor symbols to Device:* and RespiraWorks_Std:*
Parts:
- U?: symbol Power_Protection:USBLC6-2SC6 -> RespiraWorks_Std:USBLC6-2SC6
Changed lines of the file:
@@
 	5600 3600 5600 3850
 $Comp
-L Power_Protection:USBLC6-2SC6 U?
+L RespiraWorks_Std:USBLC6-2SC6 U?
 U 1 1 5FFD5C58
 P 2400 3600

Commit message: PCB Rev A Floorplanning (#1079)
* annotate schematics

* generate netlist

* define board edges at 150x300mm

* add parts to board (some pending errors)

* fix schem-pcb footprint mismatches and push to PCB

* preliminary packing at 155x300mm board size - marginal

* PCB floor planning

* added fan power and swapped solenoid/touchscreen power to vertical connectors
Parts:
- gave numbers to parts that had none: 5
Changed lines of the file:
@@
 Vcc
 $Comp
-L Connector_Generic:Conn_01x02 J?
+L Connector_Generic:Conn_01x02 J31
 U 1 1 6010AD26
 P 1550 3200
-AR Path="/5FCD4EEA/600F5EF3/6010AD26" Ref="J?"  Part="1"
-AR Path="/5FCD4EEA/600F7154/6010AD26" Ref="J?"  Part="1"
-AR Path="/5FCD4EEA/600F719E/6010AD26" Ref="J?"  Part="1"
-AR Path="/5FCD4EEA/600F71F1/6010AD26" Ref="J?"  Part="1"
-AR Path="/5FCD4EEA/600F723B/6010AD26" Ref="J?"  Part="1"
-F 0 "J?" H 1468 3417 50  0000 C CNN
+AR Path="/5FCD4EEA/600F5EF3/6010AD26" Ref="J31"  Part="1"
+AR Path="/5FCD4EEA/600F7154/6010AD26" Ref="J32"  Part="1"
+AR Path="/5FCD4EEA/600F719E/6010AD26" Ref="J33"  Part="1"
+AR Path="/5FCD4EEA/600F71F1/6010AD26" Ref="J34"  Part="1"
+AR Path="/5FCD4EEA/600F723B/6010AD26" Ref="J35"  Part="1"
+F 0 "J35" H 1468 3417 50  0000 C CNN
 F 1 "Temperature sensor (NTC)" H 1468 3326 50  0000 C CNN
 F 2 "RespiraWorks_Std:Molex_Micro-Fit_3.0_43650-0215_1x02_P3.00mm_Vertical" H 1550 3200 50  0001 C CNN
@@
 AR Path="/5FCD4E9D/6007E2BB/6010B42D" Ref="#PWR?"  Part="1"
 AR Path="/5FCD4E9D/60073FCF/6010B42D" Ref="#PWR?"  Part="1"
-AR Path="/5FCD4EEA/600F5EF3/6010B42D" Ref="#PWR?"  Part="1"
-AR Path="/5FCD4EEA/600F7154/6010B42D" Ref="#PWR?"  Part="1"
-AR Path="/5FCD4EEA/600F719E/6010B42D" Ref="#PWR?"  Part="1"
-AR Path="/5FCD4EEA/600F71F1/6010B42D" Ref="#PWR?"  Part="1"
-AR Path="/5FCD4EEA/600F723B/6010B42D" Ref="#PWR?"  Part="1"
-F 0 "#PWR?" H 4300 3600 50  0001 C CNN
+AR Path="/5FCD4EEA/600F5EF3/6010B42D" Ref="#PWR0234"  Part="1"
+AR Path="/5FCD4EEA/600F7154/6010B42D" Ref="#PWR0237"  Part="1"
+AR Path="/5FCD4EEA/600F719E/6010B42D" Ref="#PWR0240"  Part="1"
+AR Path="/5FCD4EEA/600F71F1/6010B42D" Ref="#PWR0243"  Part="1"
+AR Path="/5FCD4EEA/600F723B/6010B42D" Ref="#PWR0246"  Part="1"
+F 0 "#PWR0246" H 4300 3600 50  0001 C CNN
 F 1 "GND" H 4305 3677 50  0000 C CNN
 F 2 "" H 4300 3850 50  0001 C CNN
@@
 AR Path="/5FCD4E9D/6007DA64/60117C67" Ref="#PWR?"  Part="1"
 AR Path="/5FCD4E9D/6007BD34/60117C67" Ref="#PWR?"  Part="1"
-AR Path="/5FCD4EEA/600F5EF3/60117C67" Ref="#PWR?"  Part="1"
-AR Path="/5FCD4EEA/600F71F1/60117C67" Ref="#PWR?"  Part="1"
-AR Path="/5FCD4EEA/600F723B/60117C67" Ref="#PWR?"  Part="1"
-AR Path="/5FCD4EEA/600F7154/60117C67" Ref="#PWR?"  Part="1"
-AR Path="/5FCD4EEA/600F719E/60117C67" Ref="#PWR?"  Part="1"
-F 0 "#PWR?" H 5600 3600 50  0001 C CNN
+AR Path="/5FCD4EEA/600F5EF3/60117C67" Ref="#PWR0235"  Part="1"
+AR Path="/5FCD4EEA/600F71F1/60117C67" Ref="#PWR0244"  Part="1"
+AR Path="/5FCD4EEA/600F723B/60117C67" Ref="#PWR0247"  Part="1"
+AR Path="/5FCD4EEA/600F7154/60117C67" Ref="#PWR0238"  Part="1"
+AR Path="/5FCD4EEA/600F719E/60117C67" Ref="#PWR0241"  Part="1"
+F 0 "#PWR0247" H 5600 3600 50  0001 C CNN
 F 1 "GND" H 5605 3677 50  0000 C CNN
 F 2 "" H 5600 3850 50  0001 C CNN
@@
 AR Path="/5FCD4E9D/6007E2BB/60108F2B" Ref="R?"  Part="1"
 AR Path="/5FCD4E9D/60073FCF/60108F2B" Ref="R?"  Part="1"
-AR Path="/5FCD4EEA/600F5EF3/60108F2B" Ref="R?"  Part="1"
-AR Path="/5FCD4EEA/600F7154/60108F2B" Ref="R?"  Part="1"
-AR Path="/5FCD4EEA/600F719E/60108F2B" Ref="R?"  Part="1"
-AR Path="/5FCD4EEA/600F71F1/60108F2B" Ref="R?"  Part="1"
-AR Path="/5FCD4EEA/600F723B/60108F2B" Ref="R?"  Part="1"
-F 0 "R?" H 4150 2700 50  0000 C CNN
+AR Path="/5FCD4EEA/600F5EF3/60108F2B" Ref="R102"  Part="1"
+AR Path="/5FCD4EEA/600F7154/60108F2B" Ref="R104"  Part="1"
+AR Path="/5FCD4EEA/600F719E/60108F2B" Ref="R106"  Part="1"
+AR Path="/5FCD4EEA/600F71F1/60108F2B" Ref="R108"  Part="1"
+AR Path="/5FCD4EEA/600F723B/60108F2B" Ref="R110"  Part="1"
+F 0 "R110" H 4150 2700 50  0000 C CNN
 F 1 "220 0.1%" H 4000 2800 50  0000 C CNN
 F 2 "RespiraWorks_Std:R_0603_1608Metric" V 4230 2700 50  0001 C CNN
@@
 AR Path="/5FCD4E9D/6007E2BB/5FFCC04E" Ref="R?"  Part="1"
 AR Path="/5FCD4E9D/60073FCF/5FFCC04E" Ref="R?"  Part="1"
-AR Path="/5FCD4EEA/600F5EF3/5FFCC04E" Ref="R?"  Part="1"
-AR Path="/5FCD4EEA/600F7154/5FFCC04E" Ref="R?"  Part="1"
-AR Path="/5FCD4EEA/600F719E/5FFCC04E" Ref="R?"  Part="1"
-AR Path="/5FCD4EEA/600F71F1/5FFCC04E" Ref="R?"  Part="1"
-AR Path="/5FCD4EEA/600F723B/5FFCC04E" Ref="R?"  Part="1"
-F 0 "R?" H 4150 3600 50  0000 C CNN
+AR Path="/5FCD4EEA/600F5EF3/5FFCC04E" Ref="R103"  Part="1"
+AR Path="/5FCD4EEA/600F7154/5FFCC04E" Ref="R105"  Part="1"
+AR Path="/5FCD4EEA/600F719E/5FFCC04E" Ref="R107"  Part="1"
+AR Path="/5FCD4EEA/600F71F1/5FFCC04E" Ref="R109"  Part="1"
+AR Path="/5FCD4EEA/600F723B/5FFCC04E" Ref="R111"  Part="1"
+F 0 "R111" H 4150 3600 50  0000 C CNN
 F 1 "10k 0.1%" H 4000 3700 50  0000 C CNN
 F 2 "RespiraWorks_Std:R_0603_1608Metric" V 4230 3600 50  0001 C CNN
@@
 	5600 3600 5600 3850
 $Comp
-L RespiraWorks_Std:USBLC6-2SC6 U?
+L RespiraWorks_Std:USBLC6-2SC6 U11
 U 1 1 5FFD5C58
 P 2400 3600
-AR Path="/5FCD4EEA/600F5EF3/5FFD5C58" Ref="U?"  Part="1"
-AR Path="/5FCD4EEA/600F723B/5FFD5C58" Ref="U?"  Part="1"
-AR Path="/5FCD4EEA/600F7154/5FFD5C58" Ref="U?"  Part="1"
-AR Path="/5FCD4EEA/600F719E/5FFD5C58" Ref="U?"  Part="1"
-AR Path="/5FCD4EEA/600F71F1/5FFD5C58" Ref="U?"  Part="1"
-F 0 "U?" V 1800 3700 50  0000 L CNN
+AR Path="/5FCD4EEA/600F5EF3/5FFD5C58" Ref="U11"  Part="1"
+AR Path="/5FCD4EEA/600F723B/5FFD5C58" Ref="U15"  Part="1"
+AR Path="/5FCD4EEA/600F7154/5FFD5C58" Ref="U12"  Part="1"
+AR Path="/5FCD4EEA/600F719E/5FFD5C58" Ref="U13"  Part="1"
+AR Path="/5FCD4EEA/600F71F1/5FFD5C58" Ref="U14"  Part="1"
+F 0 "U15" V 1800 3700 50  0000 L CNN
 F 1 "USBLC6-2SC6" V 1900 3550 50  0000 L CNN
 F 2 "Package_TO_SOT_SMD:SOT-23-6" H 2400 3100 50  0001 C CNN
@@
 AR Path="/5FCD4E9D/6007E2BB/5FFDA1EB" Ref="#PWR?"  Part="1"
 AR Path="/5FCD4E9D/60073FCF/5FFDA1EB" Ref="#PWR?"  Part="1"
-AR Path="/5FCD4EEA/600F5EF3/5FFDA1EB" Ref="#PWR?"  Part="1"
-AR Path="/5FCD4EEA/600F7154/5FFDA1EB" Ref="#PWR?"  Part="1"
-AR Path="/5FCD4EEA/600F719E/5FFDA1EB" Ref="#PWR?"  Part="1"
-AR Path="/5FCD4EEA/600F71F1/5FFDA1EB" Ref="#PWR?"  Part="1"
-AR Path="/5FCD4EEA/600F723B/5FFDA1EB" Ref="#PWR?"  Part="1"
-F 0 "#PWR?" H 1900 3400 50  0001 C CNN
+AR Path="/5FCD4EEA/600F5EF3/5FFDA1EB" Ref="#PWR0233"  Part="1"
+AR Path="/5FCD4EEA/600F7154/5FFDA1EB" Ref="#PWR0236"  Part="1"
+AR Path="/5FCD4EEA/600F719E/5FFDA1EB" Ref="#PWR0239"  Part="1"
+AR Path="/5FCD4EEA/600F71F1/5FFDA1EB" Ref="#PWR0242"  Part="1"
+AR Path="/5FCD4EEA/600F723B/5FFDA1EB" Ref="#PWR0245"  Part="1"
+F 0 "#PWR0245" H 1900 3400 50  0001 C CNN
 F 1 "GND" H 1905 3477 50  0000 C CNN
 F 2 "" H 1900 3650 50  0001 C CNN
@@
 AR Path="/5FCD4B8E/603C510C/60567144/6071F4E4" Ref="C?"  Part="1"
 AR Path="/6041384A/60567144/6071F4E4" Ref="C?"  Part="1"
-AR Path="/5FCD4EEA/600F71F1/6071F4E4" Ref="C?"  Part="1"
-AR Path="/5FCD4EEA/600F5EF3/6071F4E4" Ref="C?"  Part="1"
-AR Path="/5FCD4EEA/600F7154/6071F4E4" Ref="C?"  Part="1"
-AR Path="/5FCD4EEA/600F719E/6071F4E4" Ref="C?"  Part="1"
-AR Path="/5FCD4EEA/600F723B/6071F4E4" Ref="C?"  Part="1"
-F 0 "C?" H 5650 3350 50  0000 L CNN
+AR Path="/5FCD4EEA/600F71F1/6071F4E4" Ref="C63"  Part="1"
+AR Path="/5FCD4EEA/600F5EF3/6071F4E4" Ref="C60"  Part="1"
+AR Path="/5FCD4EEA/600F7154/6071F4E4" Ref="C61"  Part="1"
+AR Path="/5FCD4EEA/600F719E/6071F4E4" Ref="C62"  Part="1"
+AR Path="/5FCD4EEA/600F723B/6071F4E4" Ref="C64"  Part="1"
+F 0 "C64" H 5650 3350 50  0000 L CNN
 F 1 "10uF" H 5650 3250 50  0000 L CNN
 F 2 "RespiraWorks_Std:C_1210_3225Metric" H 5638 3300 50  0001 C CNN

Commit message: Placement: alarms, solenoid drivers, O2/temp sensors, ST-Link
Initial placements, minor routing for testing route-ability
Fixed incorrect footprint for Raspberry Pi connector
Adjusted schematic positioning of values, references as necessary
Changed lines of the file:
@@
 $Descr A4 11693 8268
 encoding utf-8
-Sheet 22 38
+Sheet 23 38
 Title "NTC Temperature Sensor Input"
 Date ""
@@
 AR Path="/5FCD4EEA/600F71F1/6010AD26" Ref="J34"  Part="1"
 AR Path="/5FCD4EEA/600F723B/6010AD26" Ref="J35"  Part="1"
-F 0 "J35" H 1468 3417 50  0000 C CNN
+F 0 "J32" H 1468 3417 50  0000 C CNN
 F 1 "Temperature sensor (NTC)" H 1468 3326 50  0000 C CNN
 F 2 "RespiraWorks_Std:Molex_Micro-Fit_3.0_43650-0215_1x02_P3.00mm_Vertical" H 1550 3200 50  0001 C CNN
@@
 AR Path="/5FCD4EEA/600F71F1/6010B42D" Ref="#PWR0243"  Part="1"
 AR Path="/5FCD4EEA/600F723B/6010B42D" Ref="#PWR0246"  Part="1"
-F 0 "#PWR0246" H 4300 3600 50  0001 C CNN
+F 0 "#PWR0237" H 4300 3600 50  0001 C CNN
 F 1 "GND" H 4305 3677 50  0000 C CNN
 F 2 "" H 4300 3850 50  0001 C CNN
@@
 AR Path="/5FCD4EEA/600F7154/60117C67" Ref="#PWR0238"  Part="1"
 AR Path="/5FCD4EEA/600F719E/60117C67" Ref="#PWR0241"  Part="1"
-F 0 "#PWR0247" H 5600 3600 50  0001 C CNN
+F 0 "#PWR0238" H 5600 3600 50  0001 C CNN
 F 1 "GND" H 5605 3677 50  0000 C CNN
 F 2 "" H 5600 3850 50  0001 C CNN
@@
 AR Path="/5FCD4EEA/600F71F1/60108F2B" Ref="R108"  Part="1"
 AR Path="/5FCD4EEA/600F723B/60108F2B" Ref="R110"  Part="1"
-F 0 "R110" H 4150 2700 50  0000 C CNN
+F 0 "R104" H 4150 2700 50  0000 C CNN
 F 1 "220 0.1%" H 4000 2800 50  0000 C CNN
 F 2 "RespiraWorks_Std:R_0603_1608Metric" V 4230 2700 50  0001 C CNN
@@
 AR Path="/5FCD4EEA/600F71F1/5FFCC04E" Ref="R109"  Part="1"
 AR Path="/5FCD4EEA/600F723B/5FFCC04E" Ref="R111"  Part="1"
-F 0 "R111" H 4150 3600 50  0000 C CNN
+F 0 "R105" H 4150 3600 50  0000 C CNN
 F 1 "10k 0.1%" H 4000 3700 50  0000 C CNN
 F 2 "RespiraWorks_Std:R_0603_1608Metric" V 4230 3600 50  0001 C CNN
@@
 AR Path="/5FCD4EEA/600F719E/5FFD5C58" Ref="U13"  Part="1"
 AR Path="/5FCD4EEA/600F71F1/5FFD5C58" Ref="U14"  Part="1"
-F 0 "U15" V 1800 3700 50  0000 L CNN
+F 0 "U12" V 1800 3700 50  0000 L CNN
 F 1 "USBLC6-2SC6" V 1900 3550 50  0000 L CNN
 F 2 "Package_TO_SOT_SMD:SOT-23-6" H 2400 3100 50  0001 C CNN
@@
 AR Path="/5FCD4EEA/600F71F1/5FFDA1EB" Ref="#PWR0242"  Part="1"
 AR Path="/5FCD4EEA/600F723B/5FFDA1EB" Ref="#PWR0245"  Part="1"
-F 0 "#PWR0245" H 1900 3400 50  0001 C CNN
+F 0 "#PWR0236" H 1900 3400 50  0001 C CNN
 F 1 "GND" H 1905 3477 50  0000 C CNN
 F 2 "" H 1900 3650 50  0001 C CNN
@@
 AR Path="/5FCD4EEA/600F719E/6071F4E4" Ref="C62"  Part="1"
 AR Path="/5FCD4EEA/600F723B/6071F4E4" Ref="C64"  Part="1"
-F 0 "C64" H 5650 3350 50  0000 L CNN
+F 0 "C61" H 5650 3350 50  0000 L CNN
 F 1 "10uF" H 5650 3250 50  0000 L CNN
 F 2 "RespiraWorks_Std:C_1210_3225Metric" H 5638 3300 50  0001 C CNN

Commit message: KiCAD extras
Auto-update of schematic files based on last-loaded sub-sheet instance (??)
Changed lines of the file:
@@
 AR Path="/5FCD4EEA/600F71F1/6010AD26" Ref="J34"  Part="1"
 AR Path="/5FCD4EEA/600F723B/6010AD26" Ref="J35"  Part="1"
-F 0 "J32" H 1468 3417 50  0000 C CNN
+F 0 "J35" H 1468 3417 50  0000 C CNN
 F 1 "Temperature sensor (NTC)" H 1468 3326 50  0000 C CNN
 F 2 "RespiraWorks_Std:Molex_Micro-Fit_3.0_43650-0215_1x02_P3.00mm_Vertical" H 1550 3200 50  0001 C CNN
@@
 AR Path="/5FCD4EEA/600F71F1/60108F2B" Ref="R108"  Part="1"
 AR Path="/5FCD4EEA/600F723B/60108F2B" Ref="R110"  Part="1"
-F 0 "R104" H 4150 2700 50  0000 C CNN
+F 0 "R110" H 4150 2700 50  0000 C CNN
 F 1 "220 0.1%" H 4000 2800 50  0000 C CNN
 F 2 "RespiraWorks_Std:R_0603_1608Metric" V 4230 2700 50  0001 C CNN
@@
 AR Path="/5FCD4EEA/600F71F1/5FFCC04E" Ref="R109"  Part="1"
 AR Path="/5FCD4EEA/600F723B/5FFCC04E" Ref="R111"  Part="1"
-F 0 "R105" H 4150 3600 50  0000 C CNN
+F 0 "R111" H 4150 3600 50  0000 C CNN
 F 1 "10k 0.1%" H 4000 3700 50  0000 C CNN
 F 2 "RespiraWorks_Std:R_0603_1608Metric" V 4230 3600 50  0001 C CNN
@@
 AR Path="/5FCD4EEA/600F719E/5FFD5C58" Ref="U13"  Part="1"
 AR Path="/5FCD4EEA/600F71F1/5FFD5C58" Ref="U14"  Part="1"
-F 0 "U12" V 1800 3700 50  0000 L CNN
+F 0 "U15" V 1800 3700 50  0000 L CNN
 F 1 "USBLC6-2SC6" V 1900 3550 50  0000 L CNN
 F 2 "Package_TO_SOT_SMD:SOT-23-6" H 2400 3100 50  0001 C CNN
@@
 AR Path="/5FCD4EEA/600F719E/6071F4E4" Ref="C62"  Part="1"
 AR Path="/5FCD4EEA/600F723B/6071F4E4" Ref="C64"  Part="1"
-F 0 "C61" H 5650 3350 50  0000 L CNN
+F 0 "C64" H 5650 3350 50  0000 L CNN
 F 1 "10uF" H 5650 3250 50  0000 L CNN
 F 2 "RespiraWorks_Std:C_1210_3225Metric" H 5638 3300 50  0001 C CNN

Commit message: Current sense resistors
Changed all current sense resistors to 5 mOhms and larger size (2512) to handle current; gave solid plane connections for heatsinking
Fixed input-power planes on solenoid drivers
Updated a few package references which still pointed to KiCAD standard libraries
Fixed misc. reference placement in schematics
Parts:
- U11: footprint Package_TO_SOT_SMD:SOT-23-6 -> RespiraWorks_Std:SOT-23-6
Changed lines of the file:
@@
 F 0 "U15" V 1800 3700 50  0000 L CNN
 F 1 "USBLC6-2SC6" V 1900 3550 50  0000 L CNN
-F 2 "Package_TO_SOT_SMD:SOT-23-6" H 2400 3100 50  0001 C CNN
+F 2 "RespiraWorks_Std:SOT-23-6" H 2400 3100 50  0001 C CNN
 F 3 "https://www.st.com/resource/en/datasheet/usblc6-2.pdf" H 2600 3950 50  0001 C CNN
 F 4 "STMicroelectronics" H 2400 3600 50  0001 C CNN "Manufacturer"
