File: pcb/sensor-daughterboards/pressure_mpxv5004dp/pressure_mpxv5004dp.sch (KiCad schematic (older format))
At the start: 5 parts

Commit message: Daughterboard interface changes
Moved pressure sensor LPF(s) from mainboard to daughterboards
Changed pressure sensor interface to 2x 4-pin headers to accomodate analog and I2C
Added onboard BMP280 for ambient pressure/temp
Added new +5V_Sns power rail for analog sensors, with optional filtering
Parts:
- added C?: 470pF 50V NP0, RespiraWorks_Std:C_0603_1608Metric, symbol Device:C
- added C?: 1uF 10V X7R, RespiraWorks_Std:C_0603_1608Metric, symbol Device:C
- added R?: 2.4K 1%, RespiraWorks_Std:R_0603_1608Metric, symbol Device:R
- added R?: 4.7K 1%, RespiraWorks_Std:R_0603_1608Metric, symbol Device:R
- J? (x2): footprint RespiraWorks_Std:PinSocket_1x03_P2.54mm_Vertical_SMD_Samtec_SSM-103-x-SV-BE -> RespiraWorks_Std:PinSocket_1x04_P2.54mm_Vertical_SMD_Samtec_SSM-104-x-SV-BE; symbol Connector_Generic:Conn_01x03 -> Connector_Generic:Conn_01x04
Connections:
- net GND: now also J?.2 (Pin_2), J?.4 (Pin_4), C?.1, C?.1, R?.1; no longer J?.1 (Pin_1), J?.3 (Pin_3), J?.3 (Pin_3)
- net at U?.4 (Vout): now also C?.2, R?.2; no longer J?.2 (Pin_2)
- net VCC renamed +5V_Sns
- new net: C?.2, J?.1 (Pin_1), R?.1, R?.2
- no-connect marks 0 -> 3
Other:
- note added: "x0.662\nLPF fc = 100 Hz"
- moved on the sheet: C?, U?

Commit message: BOM
More BOM consolidation with bulk capacitors + changed tantalum stepper caps to aluminum, added bulk cap to PSol driver
Made stepper's 3.3V power naming consistent with others (3.3V->3V3)
Slightly increased current limit on PSOL/heater driver
Changed 3906 transistors to 2907 to better support +5V_Batt current
Parts:
- C?: Part Number GRM1885C1H103JA01D -> (none)
- R? (x2): Part Number RK73H2BTTD1004F -> (none)
Changed lines of the file:
@@
 F 3 "~" H 4550 2650 50  0001 C CNN
 F 4 "Murata" H 4550 2650 50  0001 C CNN "Manufacturer"
-F 5 "GRM1885C1H103JA01D" H 4550 2650 50  0001 C CNN "Part Number"
 	1    4550 2650
 	-1   0    0    1
@@
 F 3 "~" H 5150 3600 50  0001 C CNN
 F 4 "KOA Speer" H 5150 3600 50  0001 C CNN "Manufacturer"
-F 5 "RK73H2BTTD1004F" H 5150 3600 50  0001 C CNN "Part Number"
 	1    5150 3600
 	0    1    1    0
@@
 F 3 "~" H 5550 3750 50  0001 C CNN
 F 4 "KOA Speer" H 5550 3750 50  0001 C CNN "Manufacturer"
-F 5 "RK73H2BTTD1004F" H 5550 3750 50  0001 C CNN "Part Number"
 	1    5550 3750
 	-1   0    0    1

Commit message: Pressure sensor daughterboard, misc. layout fixes
Fixed missing connections from +5V to +3.3V_Ctrl regulator, +5V_Sns filter
Finished I2C aux connector routing
Placed components for MPXV5004 daughterboard
Parts:
- added H1, H2, H3, H4: M2.5, MountingHole:MountingHole_2.7mm_M2.5_Pad_Via, symbol Mechanical:MountingHole_Pad
- C1, C4: renamed from C?; value 1uF 10V X7R -> 1uF
- C2: renamed from C?; value 10nF 100V NP0 -> 10nF
- C3: renamed from C?; value 470pF 50V NP0 -> 470pF
- R1: renamed from R?; value 2.4K 1% -> 2.4K
- R2: renamed from R?; value 4.7K 1% -> 4.7K
- gave numbers to parts that had none: 3
Connections:
- no-connect marks 3 -> 7
Changed lines of the file:
@@
 $EndDescr
 $Comp
-L RespiraWorks:MPXV5004DP U?
+L RespiraWorks:MPXV5004DP U1
 U 1 1 5FFA0C0F
 P 3550 3600
-F 0 "U?" H 3222 3621 50  0000 R CNN
+F 0 "U1" H 3222 3621 50  0000 R CNN
 F 1 "MPXV5004DP" H 3222 3530 50  0000 R CNN
 F 2 "RespiraWorks:NXP_MPXV5004DP" H 3550 3750 50  0001 C CNN
@@
 $EndComp
 $Comp
-L Device:C C?
+L Device:C C2
 U 1 1 5FFA6CA1
 P 4550 2650
-AR Path="/5FFA6CA1" Ref="C?"  Part="1"
+AR Path="/5FFA6CA1" Ref="C2"  Part="1"
 AR Path="/5E8AFE9D/5FFA6CA1" Ref="C?"  Part="1"
 AR Path="/5E8FBD97/5FFA6CA1" Ref="C?"  Part="1"
@@
 AR Path="/5FCD4DF5/5FFA6CA1" Ref="C?"  Part="1"
 AR Path="/5FCD4E9D/5FFA6CA1" Ref="C?"  Part="1"
-F 0 "C?" H 4300 2650 50  0000 C CNN
-F 1 "10nF 100V NP0" H 4200 2750 50  0000 C CNN
+F 0 "C2" H 4300 2650 50  0000 C CNN
+F 1 "10nF" H 4350 2750 50  0000 C CNN
 F 2 "RespiraWorks_Std:C_0603_1608Metric" H 4588 2500 50  0001 C CNN
 F 3 "~" H 4550 2650 50  0001 C CNN
@@
 $EndComp
 $Comp
-L power:GND #PWR?
+L power:GND #PWR0101
 U 1 1 5FFA6CA7
 P 4550 2800
-AR Path="/5FFA6CA7" Ref="#PWR?"  Part="1"
+AR Path="/5FFA6CA7" Ref="#PWR0101"  Part="1"
 AR Path="/5E8AFE9D/5FFA6CA7" Ref="#PWR?"  Part="1"
 AR Path="/5E8FBD97/5FFA6CA7" Ref="#PWR?"  Part="1"
@@
 AR Path="/5FCD4DF5/5FFA6CA7" Ref="#PWR?"  Part="1"
 AR Path="/5FCD4E9D/5FFA6CA7" Ref="#PWR?"  Part="1"
-F 0 "#PWR?" H 4550 2550 50  0001 C CNN
+F 0 "#PWR0101" H 4550 2550 50  0001 C CNN
 F 1 "GND" H 4555 2627 50  0000 C CNN
 F 2 "" H 4550 2800 50  0001 C CNN
@@
 AR Path="/5FCD4B8E/606EF10F/5FFA6CAD" Ref="C?"  Part="1"
 AR Path="/5FCD4E9D/5FFA6CAD" Ref="C?"  Part="1"
-F 0 "C?" H 4550 2650 50  0000 L CNN
-F 1 "1uF 10V X7R" H 4350 2750 50  0000 L CNN
+AR Path="/5FFA6CAD" Ref="C1"  Part="1"
+F 0 "C1" H 4450 2650 50  0000 L CNN
+F 1 "1uF" H 4350 2750 50  0000 L CNN
 F 2 "RespiraWorks_Std:C_0603_1608Metric" H 4288 2500 50  0001 C CNN
 F 3 "~" H 4250 2650 50  0001 C CNN
@@
 AR Path="/5FCD4B8E/606EF10F/5FFA6CB3" Ref="#PWR?"  Part="1"
 AR Path="/5FCD4E9D/5FFA6CB3" Ref="#PWR?"  Part="1"
-AR Path="/5FFA6CB3" Ref="#PWR?"  Part="1"
-F 0 "#PWR?" H 4250 2550 50  0001 C CNN
+AR Path="/5FFA6CB3" Ref="#PWR0102"  Part="1"
+F 0 "#PWR0102" H 4250 2550 50  0001 C CNN
 F 1 "GND" H 4255 2627 50  0000 C CNN
 F 2 "" H 4250 2800 50  0001 C CNN
@@
 	4250 2500 4550 2500
 $Comp
-L Connector_Generic:Conn_01x04 J?
+L Connector_Generic:Conn_01x04 J1
 U 1 1 5FFA737A
 P 7200 3700
-F 0 "J?" H 7280 3742 50  0000 L CNN
+F 0 "J1" H 7280 3742 50  0000 L CNN
 F 1 "0.1\" female header, bottom entry" H 7280 3651 50  0000 L CNN
 F 2 "RespiraWorks_Std:PinSocket_1x04_P2.54mm_Vertical_SMD_Samtec_SSM-104-x-SV-BE" H 7200 3700 50  0001 C CNN
@@
 $EndComp
 $Comp
-L Connector_Generic:Conn_01x04 J?
+L Connector_Generic:Conn_01x04 J2
 U 1 1 5FFA26A3
 P 7200 4700
-F 0 "J?" H 7280 4742 50  0000 L CNN
+F 0 "J2" H 7280 4742 50  0000 L CNN
 F 1 "0.1\" female header, bottom entry" H 7280 4651 50  0000 L CNN
 F 2 "RespiraWorks_Std:PinSocket_1x04_P2.54mm_Vertical_SMD_Samtec_SSM-104-x-SV-BE" H 7200 4700 50  0001 C CNN
@@
 AR Path="/5FCD4B8E/606EF10F/5FFA361A" Ref="#PWR?"  Part="1"
 AR Path="/5FCD4E9D/5FFA361A" Ref="#PWR?"  Part="1"
-AR Path="/5FFA361A" Ref="#PWR?"  Part="1"
-F 0 "#PWR?" H 3350 3900 50  0001 C CNN
+AR Path="/5FFA361A" Ref="#PWR0103"  Part="1"
+F 0 "#PWR0103" H 3350 3900 50  0001 C CNN
 F 1 "GND" H 3355 3977 50  0000 C CNN
 F 2 "" H 3350 4150 50  0001 C CNN
@@
 AR Path="/5FCD4B8E/606EF10F/5FFA3C31" Ref="#PWR?"  Part="1"
 AR Path="/5FCD4E9D/5FFA3C31" Ref="#PWR?"  Part="1"
-AR Path="/5FFA3C31" Ref="#PWR?"  Part="1"
-F 0 "#PWR?" H 6900 3750 50  0001 C CNN
+AR Path="/5FFA3C31" Ref="#PWR0104"  Part="1"
+F 0 "#PWR0104" H 6900 3750 50  0001 C CNN
 F 1 "GND" H 6905 3827 50  0000 C CNN
 F 2 "" H 6900 4000 50  0001 C CNN
@@
 AR Path="/5FCD4B8E/606EF10F/5FFA7110" Ref="#PWR?"  Part="1"
 AR Path="/5FCD4E9D/5FFA7110" Ref="#PWR?"  Part="1"
-AR Path="/5FFA7110" Ref="#PWR?"  Part="1"
-F 0 "#PWR?" H 6750 4750 50  0001 C CNN
+AR Path="/5FFA7110" Ref="#PWR0105"  Part="1"
+F 0 "#PWR0105" H 6750 4750 50  0001 C CNN
 F 1 "GND" H 6755 4827 50  0000 C CNN
 F 2 "" H 6750 5000 50  0001 C CNN
@@
 AR Path="/5FCD4E9D/6007DA64/5FFBE46B" Ref="C?"  Part="1"
 AR Path="/5FCD4E9D/6007BD34/5FFBE46B" Ref="C?"  Part="1"
-F 0 "C?" H 4850 3750 50  0000 L CNN
-F 1 "470pF 50V NP0" H 4650 3850 50  0000 L CNN
+AR Path="/5FFBE46B" Ref="C3"  Part="1"
+F 0 "C3" H 4700 3750 50  0000 L CNN
+F 1 "470pF" H 4650 3850 50  0000 L CNN
 F 2 "RespiraWorks_Std:C_0603_1608Metric" H 4588 3600 50  0001 C CNN
 F 3 "~" H 4550 3750 50  0001 C CNN
@@
 AR Path="/5FCD4E9D/6007DA64/5FFBE471" Ref="#PWR?"  Part="1"
 AR Path="/5FCD4E9D/6007BD34/5FFBE471" Ref="#PWR?"  Part="1"
-F 0 "#PWR?" H 4550 3650 50  0001 C CNN
+AR Path="/5FFBE471" Ref="#PWR0106"  Part="1"
+F 0 "#PWR0106" H 4550 3650 50  0001 C CNN
 F 1 "GND" H 4555 3727 50  0000 C CNN
 F 2 "" H 4550 3900 50  0001 C CNN
@@
 AR Path="/5FCD4E9D/6007DA64/5FFBE477" Ref="C?"  Part="1"
 AR Path="/5FCD4E9D/6007BD34/5FFBE477" Ref="C?"  Part="1"
-F 0 "C?" H 6450 3750 50  0000 L CNN
-F 1 "1uF 10V X7R" H 6250 3850 50  0000 L CNN
+AR Path="/5FFBE477" Ref="C4"  Part="1"
+F 0 "C4" H 6300 3750 50  0000 L CNN
+F 1 "1uF" H 6250 3850 50  0000 L CNN
 F 2 "RespiraWorks_Std:C_0603_1608Metric" H 6188 3600 50  0001 C CNN
 F 3 "~" H 6150 3750 50  0001 C CNN
@@
 AR Path="/5FCD4E9D/6007DA64/5FFBE47D" Ref="#PWR?"  Part="1"
 AR Path="/5FCD4E9D/6007BD34/5FFBE47D" Ref="#PWR?"  Part="1"
-F 0 "#PWR?" H 6150 3650 50  0001 C CNN
+AR Path="/5FFBE47D" Ref="#PWR0107"  Part="1"
+F 0 "#PWR0107" H 6150 3650 50  0001 C CNN
 F 1 "GND" H 6155 3727 50  0000 C CNN
 F 2 "" H 6150 3900 50  0001 C CNN
@@
 $EndComp
 $Comp
-L Device:R R?
+L Device:R R1
 U 1 1 5FFBE485
 P 5150 3600
-AR Path="/5FFBE485" Ref="R?"  Part="1"
+AR Path="/5FFBE485" Ref="R1"  Part="1"
 AR Path="/5E8AFE9D/5FFBE485" Ref="R?"  Part="1"
 AR Path="/5E8C8865/5FFBE485" Ref="R?"  Part="1"
@@
 AR Path="/5FCD4E9D/6007DA64/5FFBE485" Ref="R?"  Part="1"
 AR Path="/5FCD4E9D/6007BD34/5FFBE485" Ref="R?"  Part="1"
-F 0 "R?" V 4950 3600 50  0000 C CNN
-F 1 "2.4K 1%" V 5050 3600 50  0000 C CNN
+F 0 "R1" V 4950 3600 50  0000 C CNN
+F 1 "2.4K" V 5050 3600 50  0000 C CNN
 F 2 "RespiraWorks_Std:R_0603_1608Metric" V 5080 3600 50  0001 C CNN
 F 3 "~" H 5150 3600 50  0001 C CNN
@@
 $EndComp
 $Comp
-L Device:R R?
+L Device:R R2
 U 1 1 5FFBE48D
 P 5550 3750
-AR Path="/5FFBE48D" Ref="R?"  Part="1"
+AR Path="/5FFBE48D" Ref="R2"  Part="1"
 AR Path="/5E8AFE9D/5FFBE48D" Ref="R?"  Part="1"
 AR Path="/5E8C8865/5FFBE48D" Ref="R?"  Part="1"
@@
 AR Path="/5FCD4E9D/6007DA64/5FFBE48D" Ref="R?"  Part="1"
 AR Path="/5FCD4E9D/6007BD34/5FFBE48D" Ref="R?"  Part="1"
-F 0 "R?" H 5400 3750 50  0000 C CNN
-F 1 "4.7K 1%" H 5300 3850 50  0000 C CNN
+F 0 "R2" H 5400 3750 50  0000 C CNN
+F 1 "4.7K" H 5400 3850 50  0000 C CNN
 F 2 "RespiraWorks_Std:R_0603_1608Metric" V 5480 3750 50  0001 C CNN
 F 3 "~" H 5550 3750 50  0001 C CNN
@@
 AR Path="/5FCD4E9D/6007DA64/5FFBE498" Ref="#PWR?"  Part="1"
 AR Path="/5FCD4E9D/6007BD34/5FFBE498" Ref="#PWR?"  Part="1"
-F 0 "#PWR?" H 5550 3650 50  0001 C CNN
+AR Path="/5FFBE498" Ref="#PWR0108"  Part="1"
+F 0 "#PWR0108" H 5550 3650 50  0001 C CNN
 F 1 "GND" H 5555 3727 50  0000 C CNN
 F 2 "" H 5550 3900 50  0001 C CNN
@@
 NoConn ~ 7000 3900
 $Comp
-L RespiraWorks:+5V_Sns #PWR?
+L RespiraWorks:+5V_Sns #PWR0109
 U 1 1 5FFD6716
 P 3350 2500
-F 0 "#PWR?" H 3350 2500 50  0001 C CNN
+F 0 "#PWR0109" H 3350 2500 50  0001 C CNN
 F 1 "+5V_Sns" H 3335 2673 50  0000 C CNN
 F 2 "" H 3350 2500 50  0001 C CNN
@@
 Connection ~ 3350 2500
 $Comp
-L RespiraWorks:+5V_Sns #PWR?
+L RespiraWorks:+5V_Sns #PWR0110
 U 1 1 5FFD6C8C
 P 6750 4600
-F 0 "#PWR?" H 6750 4600 50  0001 C CNN
+F 0 "#PWR0110" H 6750 4600 50  0001 C CNN
 F 1 "+5V_Sns" H 6735 4773 50  0000 C CNN
 F 2 "" H 6750 4600 50  0001 C CNN
@@
 	6750 4900 6750 5000
 NoConn ~ 7000 4800
+$Comp
+L Mechanical:MountingHole_Pad H1
+U 1 1 605B378F
+P 8300 1650
+F 0 "H1" H 8400 1699 50  0000 L CNN
+F 1 "M2.5" H 8400 1608 50  0000 L CNN
+F 2 "MountingHole:MountingHole_2.7mm_M2.5_Pad_Via" H 8300 1650 50  0001 C CNN
+F 3 "~" H 8300 1650 50  0001 C CNN
+	1    8300 1650
+	1    0    0    -1
+$EndComp
+$Comp
+L Mechanical:MountingHole_Pad H3
+U 1 1 605B4C2D
+P 8750 1650
+F 0 "H3" H 8850 1699 50  0000 L CNN
+F 1 "M2.5" H 8850 1608 50  0000 L CNN
+F 2 "MountingHole:MountingHole_2.7mm_M2.5_Pad_Via" H 8750 1650 50  0001 C CNN
+F 3 "~" H 8750 1650 50  0001 C CNN
+	1    8750 1650
+	1    0    0    -1
+$EndComp
+NoConn ~ 8300 1750
+NoConn ~ 8750 1750
+$Comp
+L Mechanical:MountingHole_Pad H2
+U 1 1 605B55AD
+P 8300 2000
+F 0 "H2" H 8400 2049 50  0000 L CNN
+F 1 "M2.5" H 8400 1958 50  0000 L CNN
+F 2 "MountingHole:MountingHole_2.7mm_M2.5_Pad_Via" H 8300 2000 50  0001 C CNN
+F 3 "~" H 8300 2000 50  0001 C CNN
+	1    8300 2000
+	1    0    0    -1
+$EndComp
+NoConn ~ 8300 2100
+$Comp
+L Mechanical:MountingHole_Pad H4
+U 1 1 605B582D
+P 8750 2000
+F 0 "H4" H 8850 2049 50  0000 L CNN
+F 1 "M2.5" H 8850 1958 50  0000 L CNN
+F 2 "MountingHole:MountingHole_2.7mm_M2.5_Pad_Via" H 8750 2000 50  0001 C CNN
+F 3 "~" H 8750 2000 50  0001 C CNN
+	1    8750 2000
+	1    0    0    -1
+$EndComp
+NoConn ~ 8750 2100
 $EndSCHEMATC

Commit message: Pressure daughterboard
Library references to RespiraWorks_Std
Removed unnecessary 10nF cap
Parts:
- removed C2: 10nF, RespiraWorks_Std:C_0603_1608Metric, symbol Device:C
- H1, H2, H3, H4: footprint MountingHole:MountingHole_2.7mm_M2.5_Pad_Via -> RespiraWorks_Std:MountingHole_2.7mm_M2.5_Pad_Via; symbol Mechanical:MountingHole_Pad -> RespiraWorks_Std:MountingHole_Pad
- J1, J2: value 0.1\" female header, bottom entry -> Main board connections (bottom entry)
- R1, R2: Manufacturer KOA Speer -> (none)
Connections:
- wire segments 15 -> 14
Other:
- moved on the sheet: C1
Changed lines of the file:
@@
-$EndComp
-$Comp
-L Device:C C2
-U 1 1 5FFA6CA1
-P 4550 2650
-AR Path="/5FFA6CA1" Ref="C2"  Part="1"
-AR Path="/5E8AFE9D/5FFA6CA1" Ref="C?"  Part="1"
-AR Path="/5E8FBD97/5FFA6CA1" Ref="C?"  Part="1"
-AR Path="/5E8E0754/5FFA6CA1" Ref="C?"  Part="1"
-AR Path="/5E8DFCAD/5FFA6CA1" Ref="C?"  Part="1"
-AR Path="/5E8DEDC0/5FFA6CA1" Ref="C?"  Part="1"
-AR Path="/5E8C8865/5FFA6CA1" Ref="C?"  Part="1"
-AR Path="/5E8E1F08/5FFA6CA1" Ref="C?"  Part="1"
-AR Path="/5FCD4DF5/5FFA6CA1" Ref="C?"  Part="1"
-AR Path="/5FCD4E9D/5FFA6CA1" Ref="C?"  Part="1"
-F 0 "C2" H 4300 2650 50  0000 C CNN
-F 1 "10nF" H 4350 2750 50  0000 C CNN
-F 2 "RespiraWorks_Std:C_0603_1608Metric" H 4588 2500 50  0001 C CNN
-F 3 "~" H 4550 2650 50  0001 C CNN
-F 4 "Murata" H 4550 2650 50  0001 C CNN "Manufacturer"
-	1    4550 2650
-	-1   0    0    1
-$EndComp
-$Comp
-L power:GND #PWR0101
-U 1 1 5FFA6CA7
-P 4550 2800
-AR Path="/5FFA6CA7" Ref="#PWR0101"  Part="1"
-AR Path="/5E8AFE9D/5FFA6CA7" Ref="#PWR?"  Part="1"
-AR Path="/5E8FBD97/5FFA6CA7" Ref="#PWR?"  Part="1"
-AR Path="/5E8E0754/5FFA6CA7" Ref="#PWR?"  Part="1"
-AR Path="/5E8DFCAD/5FFA6CA7" Ref="#PWR?"  Part="1"
-AR Path="/5E8DEDC0/5FFA6CA7" Ref="#PWR?"  Part="1"
-AR Path="/5E8C8865/5FFA6CA7" Ref="#PWR?"  Part="1"
-AR Path="/5E8E1F08/5FFA6CA7" Ref="#PWR?"  Part="1"
-AR Path="/5FCD4DF5/5FFA6CA7" Ref="#PWR?"  Part="1"
-AR Path="/5FCD4E9D/5FFA6CA7" Ref="#PWR?"  Part="1"
-F 0 "#PWR0101" H 4550 2550 50  0001 C CNN
-F 1 "GND" H 4555 2627 50  0000 C CNN
-F 2 "" H 4550 2800 50  0001 C CNN
-F 3 "" H 4550 2800 50  0001 C CNN
-	1    4550 2800
-	1    0    0    -1
 $EndComp
 $Comp
 L Device:C C?
 U 1 1 5FFA6CAD
-P 4250 2650
+P 3750 2650
 AR Path="/5FCD4B8E/5FCD4BC5/5FFA6CAD" Ref="C?"  Part="1"
 AR Path="/5FCD4B8E/5FE27F70/5FFA6CAD" Ref="C?"  Part="1"
@@
 AR Path="/5FCD4E9D/5FFA6CAD" Ref="C?"  Part="1"
 AR Path="/5FFA6CAD" Ref="C1"  Part="1"
-F 0 "C1" H 4450 2650 50  0000 L CNN
-F 1 "1uF" H 4350 2750 50  0000 L CNN
-F 2 "RespiraWorks_Std:C_0603_1608Metric" H 4288 2500 50  0001 C CNN
-F 3 "~" H 4250 2650 50  0001 C CNN
-	1    4250 2650
+F 0 "C1" H 3950 2650 50  0000 L CNN
+F 1 "1uF" H 3850 2750 50  0000 L CNN
+F 2 "RespiraWorks_Std:C_0603_1608Metric" H 3788 2500 50  0001 C CNN
+F 3 "~" H 3750 2650 50  0001 C CNN
+	1    3750 2650
 	-1   0    0    1
 $EndComp
@@
 L power:GND #PWR?
 U 1 1 5FFA6CB3
-P 4250 2800
+P 3750 2800
 AR Path="/5FCD4B8E/5FCD4BC5/5FFA6CB3" Ref="#PWR?"  Part="1"
 AR Path="/5FCD4B8E/5FE27F70/5FFA6CB3" Ref="#PWR?"  Part="1"
@@
 AR Path="/5FCD4E9D/5FFA6CB3" Ref="#PWR?"  Part="1"
 AR Path="/5FFA6CB3" Ref="#PWR0102"  Part="1"
-F 0 "#PWR0102" H 4250 2550 50  0001 C CNN
-F 1 "GND" H 4255 2627 50  0000 C CNN
-F 2 "" H 4250 2800 50  0001 C CNN
-F 3 "" H 4250 2800 50  0001 C CNN
-	1    4250 2800
+F 0 "#PWR0102" H 3750 2550 50  0001 C CNN
+F 1 "GND" H 3755 2627 50  0000 C CNN
+F 2 "" H 3750 2800 50  0001 C CNN
+F 3 "" H 3750 2800 50  0001 C CNN
+	1    3750 2800
 	1    0    0    -1
 $EndComp
@@
 	3350 3100 3350 2500
 Wire Wire Line
-	3350 2500 4250 2500
-Connection ~ 4250 2500
-Wire Wire Line
-	4250 2500 4550 2500
+	3350 2500 3750 2500
 $Comp
 L Connector_Generic:Conn_01x04 J1
@@
 P 7200 3700
 F 0 "J1" H 7280 3742 50  0000 L CNN
-F 1 "0.1\" female header, bottom entry" H 7280 3651 50  0000 L CNN
+F 1 "Main board connections (bottom entry)" H 7280 3651 50  0000 L CNN
 F 2 "RespiraWorks_Std:PinSocket_1x04_P2.54mm_Vertical_SMD_Samtec_SSM-104-x-SV-BE" H 7200 3700 50  0001 C CNN
 F 3 "~" H 7200 3700 50  0001 C CNN
@@
 P 7200 4700
 F 0 "J2" H 7280 4742 50  0000 L CNN
-F 1 "0.1\" female header, bottom entry" H 7280 4651 50  0000 L CNN
+F 1 "Main board connections (bottom entry)" H 7280 4651 50  0000 L CNN
 F 2 "RespiraWorks_Std:PinSocket_1x04_P2.54mm_Vertical_SMD_Samtec_SSM-104-x-SV-BE" H 7200 4700 50  0001 C CNN
 F 3 "~" H 7200 4700 50  0001 C CNN
@@
 F 2 "RespiraWorks_Std:R_0603_1608Metric" V 5080 3600 50  0001 C CNN
 F 3 "~" H 5150 3600 50  0001 C CNN
-F 4 "KOA Speer" H 5150 3600 50  0001 C CNN "Manufacturer"
+F 4 "" H 5150 3600 50  0001 C CNN "Manufacturer"
 	1    5150 3600
 	0    1    1    0
@@
 F 2 "RespiraWorks_Std:R_0603_1608Metric" V 5480 3750 50  0001 C CNN
 F 3 "~" H 5550 3750 50  0001 C CNN
-F 4 "KOA Speer" H 5550 3750 50  0001 C CNN "Manufacturer"
+F 4 "" H 5550 3750 50  0001 C CNN "Manufacturer"
 	1    5550 3750
 	-1   0    0    1
@@
 NoConn ~ 7000 4800
 $Comp
-L Mechanical:MountingHole_Pad H1
+L RespiraWorks_Std:MountingHole_Pad H1
 U 1 1 605B378F
 P 8300 1650
 F 0 "H1" H 8400 1699 50  0000 L CNN
 F 1 "M2.5" H 8400 1608 50  0000 L CNN
-F 2 "MountingHole:MountingHole_2.7mm_M2.5_Pad_Via" H 8300 1650 50  0001 C CNN
+F 2 "RespiraWorks_Std:MountingHole_2.7mm_M2.5_Pad_Via" H 8300 1650 50  0001 C CNN
 F 3 "~" H 8300 1650 50  0001 C CNN
 	1    8300 1650
@@
 $EndComp
 $Comp
-L Mechanical:MountingHole_Pad H3
+L RespiraWorks_Std:MountingHole_Pad H3
 U 1 1 605B4C2D
 P 8750 1650
 F 0 "H3" H 8850 1699 50  0000 L CNN
 F 1 "M2.5" H 8850 1608 50  0000 L CNN
-F 2 "MountingHole:MountingHole_2.7mm_M2.5_Pad_Via" H 8750 1650 50  0001 C CNN
+F 2 "RespiraWorks_Std:MountingHole_2.7mm_M2.5_Pad_Via" H 8750 1650 50  0001 C CNN
 F 3 "~" H 8750 1650 50  0001 C CNN
 	1    8750 1650
@@
 NoConn ~ 8750 1750
 $Comp
-L Mechanical:MountingHole_Pad H2
+L RespiraWorks_Std:MountingHole_Pad H2
 U 1 1 605B55AD
 P 8300 2000
 F 0 "H2" H 8400 2049 50  0000 L CNN
 F 1 "M2.5" H 8400 1958 50  0000 L CNN
-F 2 "MountingHole:MountingHole_2.7mm_M2.5_Pad_Via" H 8300 2000 50  0001 C CNN
+F 2 "RespiraWorks_Std:MountingHole_2.7mm_M2.5_Pad_Via" H 8300 2000 50  0001 C CNN
 F 3 "~" H 8300 2000 50  0001 C CNN
 	1    8300 2000
@@
 $EndComp
 NoConn ~ 8300 2100
-$Comp
-L Mechanical:MountingHole_Pad H4
+NoConn ~ 8750 2100
+$Comp
+L RespiraWorks_Std:MountingHole_Pad H4
 U 1 1 605B582D
 P 8750 2000
 F 0 "H4" H 8850 2049 50  0000 L CNN
 F 1 "M2.5" H 8850 1958 50  0000 L CNN
-F 2 "MountingHole:MountingHole_2.7mm_M2.5_Pad_Via" H 8750 2000 50  0001 C CNN
+F 2 "RespiraWorks_Std:MountingHole_2.7mm_M2.5_Pad_Via" H 8750 2000 50  0001 C CNN
 F 3 "~" H 8750 2000 50  0001 C CNN
 	1    8750 2000
 	1    0    0    -1
 $EndComp
-NoConn ~ 8750 2100
 $EndSCHEMATC
