File: pcb/sensor-daughterboards/pressure_mpxv5004dp/pressure_mpxv5004dp.sch (KiCad schematic (older format))
At the start: 12 parts, among them J1 Main board connections (botto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, J2 Main board connections (botto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, U1 MPXV5004DP

Commit message: Fixed 1uF cap with wrong footprint
Changed 1uF filter caps on pressure sensor daughterboards from 0805-size Kemet X7R part to 0603-size Samsung X5R part to match 0603 footprint on boards
Parts:
- C1, C4: Dielectric X7R -> X5R; Manufacturer Kemet -> Samsung; Manufacturer PN C0805C105K5RACTU -> CL10A105KB8NNNC
Changed lines of the file:
@@
 F 3 "~" H 3750 2650 50  0001 C CNN
 F 4 "50V" H 3950 2850 50  0000 C CNN "Voltage"
-F 5 "X7R" H 3750 2650 50  0001 C CNN "Dielectric"
-F 6 "Kemet" H 3750 2650 50  0001 C CNN "Manufacturer"
-F 7 "C0805C105K5RACTU" H 3750 2650 50  0001 C CNN "Manufacturer PN"
+F 5 "X5R" H 3750 2650 50  0001 C CNN "Dielectric"
+F 6 "Samsung" H 3750 2650 50  0001 C CNN "Manufacturer"
+F 7 "CL10A105KB8NNNC" H 3750 2650 50  0001 C CNN "Manufacturer PN"
 F 8 "SMT" H 3750 2650 50  0001 C CNN "Type"
 	1    3750 2650
@@
 F 2 "RespiraWorks_Std:C_0603_1608Metric" H 6188 3600 50  0001 C CNN
 F 3 "~" H 6150 3750 50  0001 C CNN
-F 4 "X7R" H 6150 3750 50  0001 C CNN "Dielectric"
-F 5 "Kemet" H 6150 3750 50  0001 C CNN "Manufacturer"
-F 6 "C0805C105K5RACTU" H 6150 3750 50  0001 C CNN "Manufacturer PN"
+F 4 "X5R" H 6150 3750 50  0001 C CNN "Dielectric"
+F 5 "Samsung" H 6150 3750 50  0001 C CNN "Manufacturer"
+F 6 "CL10A105KB8NNNC" H 6150 3750 50  0001 C CNN "Manufacturer PN"
 F 7 "50V" H 6350 3950 50  0000 C CNN "Voltage"
 F 8 "SMT" H 6150 3750 50  0001 C CNN "Type"
