File: pcb/sensor-daughterboards/pressure_XGZP6897A/pressure_XGZP6897A.kicad_pcb (KiCad board)
At the start: 2 copper layers, 42 x 25 mm, 12 parts, among them J1 Main board connections (botto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, J2 Main board connections (botto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, U1 XGZP6897A005KPDPN

Commit message: adding manufacturing files
Parts:
- U1: value XGZP6897A005KPDPN -> XGZP6897A005KPD
